File: PCB/Devboard/Devboard.kicad_sch (KiCad schematic)
At the start: 0 parts

Commit message: Section 3 Complete
Other:
- added sheet Battery.Charger,Fuel Gauge (schematics/02_Battery/Battery_Charger_FuelGauge.kicad_sch)
- added sheet Power Tree (schematics/03_Power_Tree/03_Power_Tree.kicad_sch)
- sheet Power,Input,Protection ports: added CC1_SYS, CC2_SYS, DM_SYS, DP_SYS, MUX_STATUS, PWR_GOOD, SBU1_SYS, SBU2_SYS, TPD_FLT2; removed none

Commit message: Completed phase 2
Other:
- added sheet DDR4 Memory (schematics/04_Zynq/04b_Zynq_DDR4.kicad_sch)
- added sheet ZYNQ CORE (schematics/04_Zynq/04a_Zynq_Core.kicad_sch)
- sheet Battery.Charger,Fuel Gauge ports: added none; removed +20V_MAIN, +5V_CHG, +VSYS, BATT_CHG, BQ_INT_N, BQ_OTG, CHG_STAT_N, DM_SYS, DP_SYS, FUEL_GPOUT, I2C_SCL, I2C_SDA, RAW_BAT
- sheet Power Tree ports: added none; removed +0V85, +1V2, +1V8, +20V_MAIN, +3V3, +3V3_ANA, +5V_SYS, PWR_GOOD_1V2, PWR_GOOD_1V8, PWR_GOOD_3V3, PWR_GOOD_5V, PWR_GOOD_CORE, PWR_OV_IN, PWR_UV_IN
- sheet Power,Input,Protection ports: added none; removed +20V_MAIN, CC1_SYS, CC2_SYS, DM_SYS, DP_SYS, MUX_STATUS, PWR_CURR_MON, PWR_FAULT_N, PWR_GOOD, SBU1_SYS, SBU2_SYS, TPD_FLT1, TPD_FLT12, TPD_FLT2
