File: PCB/Devboard/schematics/01_Power/Power_Input_Protection.kicad_sch (KiCad schematic)
At the start: 52 parts, among them Q1 IPB180P04P4L-02, U1 TPS2121RUXR, U2 TVS2201DRBR, U3 TPD6S300ARUKR, U4 TPD6S300ARUKR, U5 TPS259470ARPWR

Commit message: Section 3 Complete
Parts:
- R11: renamed from R19; value 150k -> 120k
- R17: renamed from R12; value 10k -> 100k
- R21: renamed from R11; value 100k -> 10k
- renumbered C14 to C1, C13 to C10, C4 to C11, C6 to C12, C11 to C13, C12 to C14, C7 to C15, C16 to C2, C2 to C3, C5 to C4, C15 to C5, C1 to C6, C9 to C7, C10 to C8, C3 to C9, D4 to D1, D3 to D2, D2 to D3, D1 to D4, R24 to R1, R3 to R10, R29 to R12, R28 to R13, R18 to R14, R17 to R15, R14 to R18, R2 to R19, R25 to R2, R15 to R20, R13 to R22, R10 to R23, R26 to R3, R6 to R4, R8 to R6, R23 to R7, R7 to R8, U2 to U1, U3 to U2, U4 to U3, U1 to U4
Connections:
- net GND: now also R21.2; no longer R17.2
- net VIN_DC: now also R17.2; no longer R21.2
- net +3.3V renamed +3V3

Commit message: Completed phase 2
Parts:
- removed R2, R3: 10k, Resistor_SMD:R_0402_1005Metric, symbol Device:R
- removed R4, R5: 5.1k, Resistor_SMD:R_0402_1005Metric, symbol Device:R
- removed R9: 1k, Resistor_SMD:R_0402_1005Metric, symbol Device:R
- removed U3: TPD6S300ARUKR, Devboard_Footprints:WQFN-20_L3.0-W3.0-P0.40-TL-EP1.7, symbol Devboard_Symbols:TPD6S300ARUKR
- added C76, C77, C83: 1uF, Capacitor_SMD:C_1210_3225Metric, symbol Device:C
- added C78: 100nF, Capacitor_SMD:C_1210_3225Metric, symbol Device:C
- added C82: 100nF, Capacitor_SMD:C_0402_1005Metric, symbol Device:C
- added D6: LSMB24CAH, Diode_SMD:D_SMC, symbol Device:D_TVS
- added D7: SMBJ20A, Diode_SMD:D_SMC, symbol Device:D_TVS
- added D8, D9: D_Schottky, Diode_SMD:D_SMC, symbol Device:D_Schottky
- added Q2: IPB180P04P4L-02, Package_TO_SOT_SMD:TO-263-7_TabPin8, symbol Devboard_Symbols:IPB180P04P4L-02
- added R76, R77, R78, R79: 100k, Resistor_SMD:R_0402_1005Metric, symbol Device:R
- added R92: 5.9kΩ, Resistor_SMD:R_0402_1005Metric, symbol Device:R
- added R93: 100kΩ, Resistor_SMD:R_0402_1005Metric, symbol Device:R
- added R94, R95: 5.1kΩ, Resistor_SMD:R_0402_1005Metric, symbol Device:R
- added U3: STUSB4500QTR, Package_DFN_QFN:QFN-24-1EP_4x4mm_P0.5mm_EP2.7x2.7mm, symbol Interface_USB:STUSB4500QTR
- C13, C15: value 0.1uF 25V -> 0.1uF 50V
- C3, C6, C9: value 100uF 25V -> 100uF 35V
- C5: value 0.1uF 50V X7R -> 2.2uF
- D1: value D_Zener -> 15V; footprint (none) -> Diode_SMD:D_SMC
- D2: value SMCJ36CA -> TP7.OSMD24CA-XC
- Q1: footprint Devboard_Footprints:TO-263-7_L10.2-W9.2-P1.27-LS15.0-TL -> Package_TO_SOT_SMD:TO-263-7_TabPin8
- R10: value 2.2k -> 29.8k
- R16: value 10k -> 100Ω
- R17: value 100k -> 442k
- R20: value 10k -> 124k
- R21: value 10k -> 20.5k
- R22: value 100k -> 210k
- R23: value 10k -> 10kΩ
- R7: value 549Ω -> 750Ω
Connections:
- net +3V3: now also R76.2, R77.2, R78.2, R79.2, U3.22 (VSYS); no longer C1.2, U2.10 (VPWR)
- net CC1: now also R95.1
- net CC1_SYS: now also U3.2 (CC1)
- net CC2: now also R94.1
- net CC2_SYS: now also U3.4 (CC2)
- net GND: now also R23.2, U1.9 (EP), U4.3 (CP2), C76.2, C77.2, C78.1, C82.1, C83.2, D6.1 (A1), D7.2 (A2), D9.2 (A), R93.2, R94.2, R95.2, U3.1 (CC1DB), U3.10 (GND), U3.12 (ADDR0), U3.13 (ADDR1), U3.25 (GND), U3.5 (CC2DB), U3.6 (RESET); no longer R16.2, U5.2 (OVLO/OVCSEL)
- net MUX_IN2: now also Q2.2 (S), Q2.3 (S), Q2.5 (S), Q2.6 (S), Q2.7 (S), R92.2; no longer Q1.8 (D)
- net MUX_OUT: now also R20.2, D8.1 (K)
- net VBUS: now also C83.1, D7.1 (A1), U3.18 (VBUS_VS_DISCH), U3.24 (VDD); no longer R20.2, R23.2
- net at D1.2 (A), Q1.1 (G): now also R16.1, R93.1
- net VREG_2V7: now reaches C5.2
- net VREG_2V7: now also C1.2, U2.10 (VPWR), C77.1, C78.2, C82.2, U3.23 (VREG_2V7)
- net +5V_SYS: now reaches C4.2, U2.3 (VBIAS)
- net +20V_MAIN renamed +15V_MAIN
- net +15V_MAIN: now also D8.2 (A), D9.1 (K)
- removed net CP2_MUX: R19.1, R23.1, U4.3 (CP2)
- removed net MUX_PR1: R16.1, R20.1, U4.6 (PR1)
- net PWR_CURR_MON renamed PWR_CURR_MON_eF
- net PWR_FAULT_N renamed PWR_FAULT_N_eF
- net PWR_GOOD renamed PG_01
- net TPD_FLT1: no longer names the net of R1.1, U2.9 (~{FLT})
- new net: R19.1, R20.1, U5.2 (OVLO/OVCSEL)
- new net: R23.1, R92.1, U4.6 (PR1)
- new net: Q2.1 (G), R16.2
- new net: C76.1, U3.21 (VREG_1V2)
- new net MUX_IN2_INT: D6.2 (A2), Q1.8 (D), Q2.8 (D)
- new net PD_ALERT: R78.1, U3.19 (ALERT)
- new net PD_ATTACH: R79.1, U3.11 (ATTACH)
- new net SINK_SCL: R76.1, U3.7 (SCL)
- new net SINK_SDA: R77.1, U3.8 (SDA)
- no-connect marks 20 -> 17
Other:
- moved on the sheet: C1, C4, D1, DC1, Q1, R1, R17, R21, U2
