File: PCB/Devboard/schematics/02_Battery/Battery_Charger_FuelGauge.kicad_sch (KiCad schematic)
At the start: 27 parts, among them U6 BQ25895RTWR, U7 BQ27441DRZR-G1A, U9 XT60

Commit message: Completed phase 2
Parts:
- added C79: 22uF, Capacitor_SMD:C_0805_2012Metric, symbol Device:C
- added C80, C81: 100nF, Capacitor_SMD:C_0402_1005Metric, symbol Device:C
- added C84, C88, C89: 1uF, Capacitor_SMD:C_0805_2012Metric, symbol Device:C
- added C85: 0.1uF, Capacitor_SMD:C_0805_2012Metric, symbol Device:C
- added C86, C87: 10nF, Capacitor_SMD:C_0805_2012Metric, symbol Device:C
- added L8: 2.2uH,5A, Inductor_SMD:L_Bourns_SRP1245A, symbol Device:L
- added R80, R85, R86, R87, R90, R91: 100kΩ, Resistor_SMD:R_0402_1005Metric, symbol Device:R
- added R81: 1k, Resistor_SMD:R_0402_1005Metric, symbol Device:R
- added R82: 100, Resistor_SMD:R_0402_1005Metric, symbol Device:R
- added R83, R89: 10kΩ, Resistor_SMD:R_0402_1005Metric, symbol Device:R
- added R88: 31.6K, Resistor_SMD:R_0402_1005Metric, symbol Device:R
- added R98: 1kΩ, Resistor_SMD:R_0402_1005Metric, symbol Device:R
- added SW1: SW_Push, Button_Switch_SMD:SW_SPST_Omron_B3FS-100xP, symbol Switch:SW_Push
- added U18: DW06, Devboard_Footprints:SOT-23-6_L2.9-W1.6-P0.95-LS2.8-BL, symbol Devboard_Symbols:DW06
- added U19: TPS61088RHLR, Devboard_Footprints:VQFN-20_L4.6-W3.6-P0.50-BL, symbol Devboard_Symbols:TPS61088RHLR
- added U21: LM66100DCK, Package_TO_SOT_SMD:SOT-363_SC-70-6, symbol Power_Management:LM66100DCK
- D5: footprint Capacitor_SMD:C_0603_1608Metric -> LED_SMD:LED_0603_1608Metric
- R24: value 100Ω -> 180Ω
Connections:
- net BQ_OTG is gone; now on net GND: U6.8 (OTG)
- net +VSYS: now also L1.2, L8.1, R80.1, U19.9 (VIN)
- net BATT_CHG: now also C79.1; no longer L1.2
- net GND: now also C79.2, C81.1, C84.1, C86.1, C87.1, C88.1, C89.1, R83.2, R85.1, R88.2, R90.2, R91.1, SW1.2, U19.13 (MODE), U19.20 (AGND), U19.21 (PGND), U21.2 (GND); no longer U6.9 (CE), U9.1 (-)
- net RAW_BAT: now also R98.1
- net at U6.12 (QON): now also C81.2, SW1.1
- net at C23.2, U7.5 (VDD): now also R98.2
- net +3.3V renamed +3V3
- net +5V_CHG renamed +5V_SYS
- net +5V_SYS: now also C89.2, R91.2, U21.3 (~{CE}), U21.6 (VOUT)
- net DM_SYS renamed DN1
- net DP_SYS renamed DP1
- net I2C_SCL renamed FuelGauge_SCL
- net I2C_SDA renamed FuelGauge_SDA
- net U6_REGN renamed REGN
- net U6_TS renamed TS
- net U7_SRN renamed SRN
- net U7_SRP renamed SRP
- new net: R87.1, R88.1, U19.17 (FB)
- new net: R83.1, U21.5 (ST)
- new net: C85.1, L8.2, R86.1, U19.4 (SW), U19.5 (SW), U19.6 (SW), U19.7 (SW)
- new net: C85.2, U19.8 (BOOT)
- new net: R89.1, U19.18 (COMP)
- new net: C87.2, R89.2
- new net: C86.2, U19.10 (SS)
- new net: R82.1, U18.5 (VDD)
- new net: C84.2, U19.1 (VCC)
- new net: R86.2, U19.3 (FSW)
- new net: R81.2, U18.1 (V-)
- new net: R90.1, U19.19 (ILIM)
- new net: R80.2, U19.2 (EN)
- new net +5V_BOOST: C88.2, R87.2, U19.14 (VOUT), U19.15 (VOUT), U19.16 (VOUT), U21.1 (VIN)
- new net CELL_B+: C80.1, R82.2
- new net CELL_B-: C80.2, U18.3 (S2), U18.6 (VSS)
- new net CHG_EN_N: R85.2, U6.9 (CE)
- new net PACK_P-: R81.1, U18.2 (S1), U9.1 (-)
- no-connect marks 4 -> 6
Other:
- moved on the sheet: C23, D5, R25, R28, R29, R30, R31, R32, R33, R35, RT1, U9
