File: PCB/Devboard/schematics/03_Power_Tree/03_Power_Tree.kicad_sch (KiCad schematic)
At the start: 67 parts, among them U10 TPS62822DLCR, U11 TPS62823DLCR, U12 TPS548A20RVER, U13 TPS7A4700RGWR, U14 TPS3700DSET, U15 TPS54824RNVR, U8 TPS62130RGTR

Commit message: Completed phase 2
Parts:
- added C100, C60, C65: 10nF, Capacitor_SMD:C_0402_1005Metric, symbol Device:C
- added C101, C53, C54, C63, C66, C98: 22uf 25v, Capacitor_SMD:C_0805_2012Metric, symbol Device:C
- added C102, C67: 4.7nF 50V, Capacitor_SMD:C_0402_1005Metric, symbol Device:C
- added C103, C59, C68, C73: 100pF, Capacitor_SMD:C_0402_1005Metric, symbol Device:C
- added C104, C58, C69: 22pF, Capacitor_SMD:C_0402_1005Metric, symbol Device:C
- added C105, C107, C109, C75: 0.1uF 25V, Capacitor_SMD:C_0402_1005Metric, symbol Device:C
- added C106, C108, C110, C71, C74, C91, C94: 10uF, Capacitor_SMD:C_0402_1005Metric, symbol Device:C
- added C55, C64, C99: 0.1uF 25v, Capacitor_SMD:C_0402_1005Metric, symbol Device:C
- added C56, C57, C61, C62, C96, C97: 47uF 6.3V, Capacitor_SMD:C_1206_3216Metric, symbol Device:C
- added C70, C90, C93: 47uF, Capacitor_SMD:C_1206_3216Metric, symbol Device:C
- added C72, C92, C95: 1uF, Capacitor_SMD:C_0402_1005Metric, symbol Device:C
- added FB1, FB2, FB3, FB4: 120Ω@100MHz, Inductor_SMD:L_01005_0402Metric, symbol Device:FerriteBead
- added L10, L7, L9: 1uH, Inductor_SMD:L_Bourns_SRP1245A, symbol Device:L
- added R100, R46, R73: 50K, Resistor_SMD:R_0402_1005Metric, symbol Device:R
- added R101, R74: 100k, Resistor_SMD:R_0402_1005Metric, symbol Device:R
- added R64: 120k, Resistor_SMD:R_0402_1005Metric, symbol Device:R
- added R65, R72, R99: 20k, Resistor_SMD:R_0402_1005Metric, symbol Device:R
- added R66, R68, R69, R71, R75, R84, R97: 10kΩ, Resistor_SMD:R_0402_1005Metric, symbol Device:R
- added R67, R70, R96: 249k, Resistor_SMD:R_0402_1005Metric, symbol Device:R
- added TP1, TP2: TestPoint, TestPoint:TestPoint_Pad_D1.0mm, symbol Connector:TestPoint
- added U16, U20, U25: TPS54824RNVR, Custom_Footprints:VQFN-18_L3.5-W3.5-P0.50-BL_TPS54824RNVR, symbol Custom_Symbols:TPS54824RNVR
- added U17, U22, U23: TPS7A4700RGWR, Devboard_Footprints:VQFN-20_L5.0-W5.0-P0.65-TL-EP, symbol Custom_Symbols:TPS7A4700RGWR
- C19, C28, C31, C32, C33, C34, C35, C37, C43, C44, C46, C47, C48, C49, C50: footprint (none) -> Capacitor_SMD:C_0402_1005Metric
- C24, C27, C29, C30, C36, C51, C52: footprint (none) -> Capacitor_SMD:C_0805_2012Metric
- C38, C39, C40, C41, C42: footprint (none) -> Capacitor_SMD:C_1206_3216Metric
- C45: value 0.1uF, 25V -> 4.7nF 50V; footprint (none) -> Capacitor_SMD:C_0402_1005Metric
- L2, L4, L5, L6: footprint (none) -> Inductor_SMD:L_Bourns_SRP1245A
- L3: value 10uH 3A -> 10uH 12A; footprint (none) -> Inductor_SMD:L_Bourns_SRP1245A
- R36, R37, R38, R39, R40, R41, R43, R44, R45, R47, R48, R50, R51, R52, R53, R54, R56, R57, R58, R59, R60, R61, R62, R63: footprint (none) -> Resistor_SMD:R_0402_1005Metric
- R42: value 300kΩ -> 249kΩ; footprint (none) -> Resistor_SMD:R_0402_1005Metric
- R49: value 24.9k -> 24.3kΩ; footprint (none) -> Resistor_SMD:R_0402_1005Metric
- R55: value 100k -> 10k; footprint (none) -> Resistor_SMD:R_0402_1005Metric
Connections:
- net +3.3V is gone; now on net +3V3: R43.2
- net PGND_U15 is gone; now on net GND: C29.1, C30.1
- net PWR_GOOD_1V8 is gone; now on net PS_POR_B: R55.1, U10.8 (PG)
- net PWR_GOOD_3V3 is gone; now on net PS_POR_B: R36.1, U8.4 (PG)
- net PWR_GOOD_5V is gone; now on net PS_POR_B: R43.1, U15.18 (PGOOD)
- net PWR_GOOD_CORE is gone; now on net PS_POR_B: R51.2, U12.2 (PGOOD)
- net +0V85: no longer C45.2
- net +1V2: now also FB3.2
- net +1V8: now also FB4.2, R75.1
- net +3V3: now also R68.1, R69.1, R84.1
- net +3V3_ANA: now also U22.3 (SENSE/FB); no longer U13.10 (0P4V), U13.4 (6P4V2), U13.5 (6P4V1), U13.6 (3P2V), U13.9 (0P8V)
- net +5V_SYS: now also C101.1, C53.1, C54.1, C63.1, C66.1, C71.1, C91.1, C94.1, C98.1, R66.2, R71.2, R97.2, U16.11 (VIN), U16.2 (VIN), U17.13 (EN), U17.15 (IN), U17.16 (IN), U20.11 (VIN), U20.2 (VIN), U22.13 (EN), U22.15 (IN), U22.16 (IN), U23.13 (EN), U23.15 (IN), U23.16 (IN), U25.11 (VIN), U25.2 (VIN)
- net GND: now also C100.2, C101.2, C103.2, C104.2, C105.2, C106.1, C107.2, C108.1, C109.2, C110.1, C53.2, C54.2, C56.2, C57.2, C58.2, C59.2, C60.2, C61.2, C62.2, C63.2, C65.2, C66.2, C68.2, C69.2, C70.2, C71.2, C72.2, C73.1, C74.1, C75.2, C90.2, C91.2, C92.2, C93.2, C94.2, C95.2, C96.2, C97.2, C98.2, R101.2, R64.2, R65.1, R67.2, R70.2, R72.1, R74.2, R96.2, R99.1, U16.10 (PGND), U16.12 (AGND), U16.3 (PGND), U16.4 (PGND), U16.5 (PGND), U16.8 (PGND), U16.9 (PGND), U17.10 (0P4V), U17.21 (EP), U17.7 (GND), U20.10 (PGND), U20.12 (AGND), U20.3 (PGND), U20.4 (PGND), U20.5 (PGND), U20.8 (PGND), U20.9 (PGND), U22.11 (0P2V), U22.12 (0P1V), U22.21 (EP), U22.7 (GND), U22.8 (1P6V), U23.11 (0P2V), U23.12 (0P1V), U23.21 (EP), U23.7 (GND), U23.9 (0P8V), U25.10 (PGND), U25.12 (AGND), U25.3 (PGND), U25.4 (PGND), U25.5 (PGND), U25.8 (PGND), U25.9 (PGND)
- net PWR_OV_IN: now also TP2.1
- net PWR_UV_IN: now also TP1.1
- net at C46.1, R48.1, R49.1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: no longer C45.1
- net +20V_MAIN renamed +15V_MAIN
- net PWR_GOOD_1V2 renamed PS_POR_B
- net PS_POR_B: now also C73.2, R68.2, R69.2, R75.2, R84.2, U16.18 (PGOOD), U20.18 (PGOOD), U25.18 (PGOOD)
- new net: R71.1, U20.17 (EN)
- new net: C92.1, U22.14 (NR)
- new net: C104.1, R100.1, R101.1, U25.14 (FB)
- new net: C58.1, R46.1, R64.1, U16.14 (FB)
- new net: R97.1, U25.17 (EN)
- new net: C69.1, R73.1, R74.1, U20.14 (FB)
- new net: C95.1, U23.14 (NR)
- new net: C65.1, U20.16 (SS/TRK)
- new net: C99.1, L10.2, U25.6 (SW), U25.7 (SW)
- new net: C99.2, U25.1 (BOOT)
- new net: C67.1, R72.2, U20.15 (COMP)
- new net: C67.2, C68.1
- new net: C45.1, R65.2, U16.15 (COMP)
- new net: C45.2, C59.1
- new net: C55.1, L7.2, U16.6 (SW), U16.7 (SW)
- new net: C55.2, U16.1 (BOOT)
- new net: C102.1, R99.2, U25.15 (COMP)
- new net: C72.1, U17.14 (NR)
- new net: C60.1, U16.16 (SS/TRK)
- new net: R67.1, U16.13 (RT/CLK)
- new net: R66.1, U16.17 (EN)
- new net: R96.1, U25.13 (RT/CLK)
- new net: C100.1, U25.16 (SS/TRK)
- new net: C64.1, L9.2, U20.6 (SW), U20.7 (SW)
- new net: C64.2, U20.1 (BOOT)
- new net: R70.1, U20.13 (RT/CLK)
- new net: C102.2, C103.1
- new net +0V85_GTR: C74.2, C75.1, FB1.1
- new net +0V85_PS: C56.1, C57.1, FB1.2, L7.1, R46.2
- new net +0V9_GTR: C105.1, C106.2, FB2.1
- new net +0V9_VCU: C96.1, C97.1, FB2.2, L10.1, R100.2
- new net +0V9_VCU_GT: C61.1, C62.1, L9.1, R73.2
- new net +1V2_GTH: C107.1, C108.2, FB3.1
- new net +1V8_CLEAN: C70.1, U17.1 (OUT), U17.20 (OUT), U17.3 (SENSE/FB)
- new net +1V8_MGTRAVTT: C109.1, C110.2, FB4.1
- new net +2V5: C93.1, U23.1 (OUT), U23.20 (OUT), U23.3 (SENSE/FB)
- new net +3V3_2: C90.1, U22.1 (OUT), U22.20 (OUT)
- no-connect marks 9 -> 43
Other:
- moved on the sheet: C27, C28, C51, L6, R47, R55, R56, R57, R58, U11
