File: PCB/Devboard/schematics/04_Zynq/04a_Zynq_Core.kicad_sch (KiCad schematic)
At the start: 47 parts, among them U24 xczu4evfbvb900pkg

Commit message: Section 3 Sanity check done
Parts:
- added C160: 330uF, Capacitor_SMD:C_0402_1005Metric, symbol Device:C
- added C161, C162, C163, C164, C165, C169, C171: 100uF, Capacitor_SMD:C_0402_1005Metric, symbol Device:C
- added C166, C168, C170, C173: 10uF, Capacitor_SMD:C_0402_1005Metric, symbol Device:C
- added C167, C180, C181, C182: 47 uF, Capacitor_SMD:C_1206_3216Metric, symbol Device:C
- added C172: 22 uF, Capacitor_SMD:C_0805_2012Metric, symbol Device:C
- added C174, C175, C176: 2.2uF, Capacitor_SMD:C_0402_1005Metric, symbol Device:C
- added C177, C178, C179: 1uF, Capacitor_SMD:C_0402_1005Metric, symbol Device:C
Connections:
- net +0V85: now also C160.1, C161.1, C162.1, C163.1, C164.1
- net +0V85_PS: now also C165.1, C166.1
- net +0V9_VCU: now also C171.1, C172.1, C173.1, C174.1, C175.1, C176.1, C177.1, C178.1, C179.1
- net +1V2: now also C169.1, C170.1
- net +1V8: now also C167.1, C168.1, C182.1
- net +3V3: now also C180.1, C181.1
- net GND: now also C160.2, C161.2, C162.2, C163.2, C164.2, C165.2, C166.2, C167.2, C168.2, C169.2, C170.2, C171.2, C172.2, C173.2, C174.2, C175.2, C176.2, C177.2, C178.2, C179.2, C180.2, C181.2, C182.2
Other:
- moved on the sheet: C116, C117, C120, C121, C122, C123, C126, C127, C128, C129, C132, C133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
