File: PCB/schematics/04_Zynq/04a_Zynq_Core.kicad_sch (KiCad schematic)
At the start: 70 parts, among them U24 xczu4evfbvb900pkg

Commit message: Fix Section 1
Parts:
- removed C114, C124, C130, C157: 0.1uF, Capacitor_SMD:C_0402_1005Metric, symbol Device:C
- removed C115, C125, C131, C136, C137, C151, C152, C153, C154, C158, C166, C168, C170, C173: 10uF, Capacitor_SMD:C_0402_1005Metric, symbol Device:C
- removed C116, C117, C118, C119, C120, C121, C122, C123, C126, C127, C134, C135, C140, C141, C167, C180, C181, C182: 47 uF, Capacitor_SMD:C_1206_3216Metric, symbol Device:C
- removed C128, C129, C132, C133, C139, C172: 22 uF, Capacitor_SMD:C_0805_2012Metric, symbol Device:C
- removed C138, C155, C156: 1 uF, Capacitor_SMD:C_0402_1005Metric, symbol Device:C
- removed C142: 1 uF, Capacitor_SMD:C_0805_2012Metric, symbol Device:C
- removed C143, C144, C145, C146, C147, C148, C149, C150: 22uF, Capacitor_SMD:C_0805_2012Metric, symbol Device:C
- removed C159: 2.2 nF, Capacitor_SMD:C_0402_1005Metric, symbol Device:C
- removed C160: 330uF, Capacitor_SMD:C_0402_1005Metric, symbol Device:C
- removed C161, C162, C163, C164, C165, C169, C171: 100uF, Capacitor_SMD:C_0402_1005Metric, symbol Device:C
- removed C174, C175, C176: 2.2uF, Capacitor_SMD:C_0402_1005Metric, symbol Device:C
- removed C177, C178, C179: 1uF, Capacitor_SMD:C_0402_1005Metric, symbol Device:C
- removed U24: xczu4evfbvb900pkg, Devboard_Footprints:XCZU4EVFBVB900PKG, symbol my_zynq:xczu4evfbvb900pkg

Commit message: Zynq Added
Parts:
- added U26: xczu4evfbvb900pkg, Devboard_Footprints:XCZU4EVFBVB900PKG, symbol my_zynq:xczu4evfbvb900pkg
Connections:
- new net: U26.A10 (MGTAVCC_R), U26.C10 (MGTAVCC_R), U26.F8 (MGTAVCC_R), U26.H8 (MGTAVCC_R), U26.M8 (MGTAVCC_R), U26.P8 (MGTAVCC_R)
- new net: U26.A6 (MGTAVTT_R), U26.B8 (MGTAVTT_R), U26.C6 (MGTAVTT_R), U26.D8 (MGTAVTT_R), U26.E6 (MGTAVTT_R), U26.G6 (MGTAVTT_R), U26.J6 (MGTAVTT_R), U26.L6 (MGTAVTT_R), U26.N6 (MGTAVTT_R), U26.R6 (MGTAVTT_R), U26.U6 (MGTAVTT_R)
- new net: U26.AA18 (VCC_PSINTFP), U26.AA20 (VCC_PSINTFP), U26.Y16 (VCC_PSINTFP), U26.Y17 (VCC_PSINTFP), U26.Y18 (VCC_PSINTFP), U26.Y19 (VCC_PSINTFP), U26.Y20 (VCC_PSINTFP)
- new net: U26.AA21 (VCC_PSINTFP_DDR), U26.AA22 (VCC_PSINTFP_DDR), U26.Y22 (VCC_PSINTFP_DDR)
- new net: U26.AA24 (VCCO_PSDDR_504), U26.AB27 (VCCO_PSDDR_504), U26.AC25 (VCCO_PSDDR_504), U26.AD28 (VCCO_PSDDR_504), U26.AE26 (VCCO_PSDDR_504), U26.AG27 (VCCO_PSDDR_504), U26.AK26 (VCCO_PSDDR_504)
- new net: U26.AB18 (VCCINT_VCU), U26.AB19 (VCCINT_VCU), U26.AB20 (VCCINT_VCU), U26.AB21 (VCCINT_VCU)
- new net: U26.B22 (VCCO_PSIO1_501), U26.B27 (VCCO_PSIO2_502), U26.D18 (VCCO_PSIO0_500), U26.D23 (VCCO_PSIO1_501), U26.D28 (VCCO_PSIO2_502), U26.E21 (VCCO_PSIO1_501), U26.E26 (VCCO_PSIO2_502), U26.F19 (VCCO_PSIO0_500), U26.J18 (VCCO_PSIO0_500), U26.N20 (VCCO_PSIO3_503), U26.P18 (VCCO_PSIO3_503)
- new net: U26.E10 (MGTVCCAUX_R), U26.G10 (MGTVCCAUX_R)
- new net: U26.H25 (PS_MGTRAVTT), U26.K25 (PS_MGTRAVTT), U26.L27 (PS_MGTRAVTT)
- new net: U26.J23 (PS_MGTRAVCC), U26.L23 (PS_MGTRAVCC)
- new net: U26.K10 (VCCAUX), U26.L10 (VCCAUX)
- new net: U26.L11 (VCCINT), U26.L13 (VCCINT), U26.L17 (VCCINT), U26.M12 (VCCINT), U26.M14 (VCCINT), U26.M16 (VCCINT), U26.M18 (VCCINT), U26.N11 (VCCINT), U26.N13 (VCCINT), U26.N15 (VCCINT), U26.N17 (VCCINT), U26.P12 (VCCINT), U26.P14 (VCCINT), U26.P16 (VCCINT), U26.R11 (VCCINT), U26.R13 (VCCINT), U26.R17 (VCCINT), U26.T12 (VCCINT), U26.T16 (VCCINT), U26.U11 (VCCINT), U26.U13 (VCCINT), U26.U17 (VCCINT), U26.V12 (VCCINT), U26.V16 (VCCINT), U26.W11 (VCCINT), U26.W13 (VCCINT), U26.W15 (VCCINT), U26.Y12 (VCCINT), U26.Y14 (VCCINT)
- new net: U26.M10 (VCCAUX_IO), U26.N10 (VCCAUX_IO), U26.P10 (VCCAUX_IO)
- new net: U26.R10 (VCCBRAM), U26.T10 (VCCBRAM), U26.U10 (VCCBRAM), U26.V10 (VCCBRAM)
- new net: U26.T18 (VCC_PSPLL), U26.T20 (VCC_PSPLL), U26.T21 (VCC_PSPLL)
- new net: U26.T22 (VCC_PSAUX), U26.U21 (VCC_PSAUX), U26.V21 (VCC_PSAUX), U26.V22 (VCC_PSAUX)
- new net: U26.T9 (VCCINT_IO), U26.U8 (VCCINT_IO), U26.U9 (VCCINT_IO), U26.V8 (VCCINT_IO)
- new net: U26.V17 (VCC_PSINTLP), U26.V18 (VCC_PSINTLP), U26.V19 (VCC_PSINTLP), U26.W17 (VCC_PSINTLP), U26.W19 (VCC_PSINTLP), U26.W20 (VCC_PSINTLP)
- no-connect marks 0 -> 5
Other:
- note added: "1.32V"
- note added: "1.65V"
- note added: "1V"
- note added: "2V"
- note added: "3.630V"

Commit message: Feat: Added zynq decoupling caps
Parts:
- added C117, C120, C121, C122, C123, C124, C125, C126, C127, C128, C129, C130, C131, C132, C133, C134, C135, C136, C137, C138, C139, C140, C141, C142, C143, C144, C145, C146, C147, C148, C150, C151, C152, C153, C154, C155, C156, C157, C158, C159, C160, C161, C162, C163, C164, C165, C166, C167, C168, C169, C170, C171, C172, C173, C174, C175, C176, C177, C178, C179, C180, C181, C182, C184, C185, C186, C187, C188, C189, C190, C191, C192, C193, C194, C195, C196, C197, C198, C199, C200, C201, C202, C203, C204, C205, C206, C207, C208, C209, C210, C211, C212, C213, C214, C215, C216, C217, C218, C219, C220, C221, C222, C223, C224, C225, C226, C227, C228, C229, C230, C231, C232, C233, C234, C235, C236, C237, C238, C239, C240, C241, C242, C243, C244, C245, C246, C247, C248, C249, C250: 0.1uF, Capacitor_SMD:C_0402_1005Metric, symbol Device:C
- added C118: 1uF, Capacitor_SMD:C_0402_1005Metric, symbol Device:C
- added C119, C149, C183: 47uF, Capacitor_SMD:C_1210_3225Metric, symbol Device:C
Connections:
- net GND: now reaches U26.A1 (GND)
- net GND: now also U26.A11 (GND), U26.A2 (GND), U26.A30 (GND), U26.A5 (GND), U26.A9 (GND), U26.AA19 (GND), U26.AA29 (GND), U26.AA9 (GND), U26.AB12 (GND), U26.AB17 (GND), U26.AB2 (GND), U26.AB22 (GND), U26.AB7 (GND), U26.AC10 (GND), U26.AC20 (GND), U26.AC5 (GND), U26.AD13 (GND), U26.AD18 (GND), U26.AD23 (GND), U26.AE16 (GND), U26.AE21 (GND), U26.AE6 (GND), U26.AF19 (GND), U26.AF24 (GND), U26.AF29 (GND), U26.AF4 (GND), U26.AF9 (GND), U26.AG12 (GND), U26.AG2 (GND), U26.AG22 (GND), U26.AH15 (GND), U26.AH20 (GND), U26.AH25 (GND), U26.AH5 (GND), U26.AJ13 (GND), U26.AJ18 (GND), U26.AJ23 (GND), U26.AJ28 (GND), U26.AJ3 (GND), U26.AJ8 (GND), U26.AK1 (GND), U26.AK30 (GND), U26.B11 (GND), U26.B13 (GND), U26.B17 (GND), U26.B3 (GND), U26.B4 (GND), U26.B7 (GND), U26.C1 (GND), U26.C11 (GND), U26.C15 (GND), U26.C2 (GND), U26.C20 (GND), U26.C25 (GND), U26.C30 (GND), U26.C5 (GND), U26.C9 (GND), U26.D11 (GND), U26.D3 (GND), U26.D4 (GND), U26.D7 (GND), U26.E1 (GND), U26.E11 (GND), U26.E2 (GND), U26.E5 (GND), U26.E9 (GND), U26.F11 (GND), U26.F14 (GND), U26.F24 (GND), U26.F25 (GND), U26.F26 (GND), U26.F27 (GND), U26.F28 (GND), U26.F29 (GND), U26.F3 (GND), U26.F30 (GND), U26.F4 (GND), U26.F7 (GND), U26.G1 (GND), U26.G11 (GND), U26.G17 (GND), U26.G2 (GND), U26.G22 (GND), U26.G23 (GND), U26.G24 (GND), U26.G27 (GND), U26.G28 (GND), U26.G5 (GND), U26.G9 (GND), U26.H11 (GND), U26.H20 (GND), U26.H22 (GND), U26.H26 (GND), U26.H29 (GND), U26.H3 (GND), U26.H30 (GND), U26.H4 (GND), U26.H7 (GND), U26.J1 (GND), U26.J10 (GND), U26.J11 (GND), U26.J13 (GND), U26.J2 (GND), U26.J22 (GND), U26.J24 (GND), U26.J27 (GND), U26.J28 (GND), U26.J5 (GND), U26.J9 (GND), U26.K22 (GND), U26.K26 (GND), U26.K29 (GND), U26.K3 (GND), U26.K30 (GND), U26.K4 (GND), U26.K9 (GND), U26.L1 (GND), U26.L12 (GND), U26.L16 (GND), U26.L18 (GND), U26.L2 (GND), U26.L22 (GND), U26.L24 (GND), U26.L28 (GND), U26.L5 (GND), U26.L9 (GND), U26.M11 (GND), U26.M13 (GND), U26.M15 (GND), U26.M17 (GND), U26.M22 (GND), U26.M26 (GND), U26.M29 (GND), U26.M3 (GND), U26.M30 (GND), U26.M4 (GND), U26.M7 (GND), U26.M9 (GND), U26.N1 (GND), U26.N12 (GND), U26.N14 (GND), U26.N16 (GND), U26.N2 (GND), U26.N23 (GND), U26.N24 (GND), U26.N25 (GND), U26.N26 (GND), U26.N27 (GND), U26.N28 (GND), U26.N29 (GND), U26.N30 (GND), U26.N5 (GND), U26.N9 (GND), U26.P11 (GND), U26.P13 (GND), U26.P15 (GND), U26.P17 (GND), U26.P3 (GND), U26.P4 (GND), U26.P7 (GND), U26.P9 (GND), U26.R1 (GND), U26.R12 (GND), U26.R14 (GNDADC), U26.R16 (GND), U26.R2 (GND), U26.R21 (GND), U26.R26 (GND), U26.R5 (GND), U26.R9 (GND), U26.T11 (GND), U26.T13 (GND), U26.T14 (VREFN), U26.T17 (GND), U26.T19 (GND), U26.T24 (GND), U26.T29 (GND), U26.T3 (GND), U26.T4 (GND), U26.T7 (GND), U26.T8 (GND), U26.U1 (GND), U26.U12 (GND), U26.U16 (GND), U26.U2 (GND), U26.U20 (VCC_PSBATT), U26.U22 (GND), U26.U27 (GND), U26.U5 (GND), U26.U7 (GND), U26.V11 (GND), U26.V13 (GND), U26.V20 (GND), U26.V25 (GND), U26.V3 (GND), U26.V4 (GND), U26.V7 (GND), U26.V9 (GND), U26.W1 (GND), U26.W12 (GND), U26.W14 (GND), U26.W16 (GND), U26.W18 (GND), U26.W2 (GND), U26.W21 (GND_PSADC), U26.W23 (GND), U26.W28 (GND), U26.W5 (GND), U26.W6 (GND), U26.Y11 (GND), U26.Y13 (GND), U26.Y15 (GND), U26.Y2 (GND), U26.Y21 (GND), U26.Y26 (GND), U26.Y3 (GND), U26.Y4 (GND), U26.Y5 (GND), C120.1, C121.1, C122.1, C123.1, C124.1, C125.1, C126.1, C127.1, C128.1, C129.1, C130.1, C131.1, C132.1, C133.1, C134.1, C135.2, C136.2, C137.2, C138.2, C139.2, C140.2, C141.2, C142.2, C143.2, C144.2, C145.2, C146.2, C147.2, C148.2, C149.2, C150.1, C151.1, C152.2, C153.2, C154.1, C155.2, C156.1, C157.2, C158.1, C159.2, C160.1, C161.2, C162.1, C163.2, C164.1, C165.2, C166.1, C167.1, C168.2, C169.1, C170.2, C171.1, C172.2, C173.1, C174.1, C175.2, C176.1, C177.2, C178.1, C179.2, C180.1, C181.1, C182.2, C183.2, C184.1, C185.1, C186.2, C187.1, C188.2, C189.1, C190.2, C191.1, C192.2, C193.1, C194.2, C195.1, C196.2, C197.1, C198.1, C199.2, C200.1, C203.1, C204.1, C205.2, C206.1, C207.2, C208.1, C209.2, C210.1, C211.2, C212.1, C213.2, C214.1, C215.2, C216.1, C217.2, C218.1, C219.2, C220.1, C221.2, C222.1, C223.1, C224.2, C225.2, C226.1, C227.1, C228.2, C229.1, C230.2, C231.1, C232.2, C233.1, C234.2, C235.1, C236.2, C237.1, C238.2, C239.1, C240.2, C241.1, C242.2, C243.1, C244.2, C245.1, C246.2, C247.1, C248.2, C249.1, C250.2
- net +0V9_GTR: now reaches U26.A10 (MGTAVCC_R), U26.C10 (MGTAVCC_R), U26.F8 (MGTAVCC_R), U26.H8 (MGTAVCC_R), U26.M8 (MGTAVCC_R), U26.P8 (MGTAVCC_R)
- net +0V9_GTR: now also C206.2, C207.1, C210.2, C211.1
- net +1V2_GTH: now reaches U26.A6 (MGTAVTT_R), U26.B8 (MGTAVTT_R), U26.C6 (MGTAVTT_R), U26.D8 (MGTAVTT_R), U26.E6 (MGTAVTT_R), U26.G6 (MGTAVTT_R), U26.J6 (MGTAVTT_R), U26.L6 (MGTAVTT_R), U26.N6 (MGTAVTT_R), U26.R6 (MGTAVTT_R), U26.U6 (MGTAVTT_R)
- net +1V2_GTH: now also C212.2, C213.1, C220.2, C221.1, C222.2, C225.1
- net +0V85_PS: now reaches U26.AA18 (VCC_PSINTFP), U26.AA20 (VCC_PSINTFP), U26.Y16 (VCC_PSINTFP), U26.Y17 (VCC_PSINTFP), U26.Y18 (VCC_PSINTFP), U26.Y19 (VCC_PSINTFP), U26.Y20 (VCC_PSINTFP)
- net +0V85_PS: now also U26.AA21 (VCC_PSINTFP_DDR), U26.AA22 (VCC_PSINTFP_DDR), U26.V17 (VCC_PSINTLP), U26.V18 (VCC_PSINTLP), U26.V19 (VCC_PSINTLP), U26.W17 (VCC_PSINTLP), U26.W19 (VCC_PSINTLP), U26.W20 (VCC_PSINTLP), U26.Y22 (VCC_PSINTFP_DDR), C167.2, C168.1, C171.2, C172.1, C173.2, C174.2, C175.1, C178.2, C179.1, C180.2, C181.2, C182.1, C183.1
- net +1V2: now reaches U26.AA24 (VCCO_PSDDR_504), U26.AB27 (VCCO_PSDDR_504), U26.AC25 (VCCO_PSDDR_504), U26.AD28 (VCCO_PSDDR_504), U26.AE26 (VCCO_PSDDR_504), U26.AG27 (VCCO_PSDDR_504), U26.AK26 (VCCO_PSDDR_504)
- net +1V2: now also C184.2, C189.2, C190.1, C193.2, C194.1
- net +1V8: now reaches U26.AA4 (VCCO_66)
- net +1V8: now also U26.AC15 (VCCO_64), U26.AD3 (VCCO_66), U26.AD8 (VCCO_66), U26.AE11 (VCCO_65), U26.AF14 (VCCO_64), U26.AG17 (VCCO_64), U26.AG7 (VCCO_65), U26.AH10 (VCCO_65), U26.E10 (MGTVCCAUX_R), U26.G10 (MGTVCCAUX_R), U26.K10 (VCCAUX), U26.L10 (VCCAUX), U26.M10 (VCCAUX_IO), U26.N10 (VCCAUX_IO), U26.P10 (VCCAUX_IO), U26.R15 (VCCADC), U26.T22 (VCC_PSAUX), U26.U21 (VCC_PSAUX), U26.V21 (VCC_PSAUX), U26.V22 (VCC_PSAUX), C162.2, C163.1, C164.2, C165.1, C166.2, C185.2, C186.1, C187.2, C188.1, C223.2, C224.1, C241.2, C242.1, C243.2, C244.1, C245.2, C246.1, C247.2, C248.1, C249.2, C250.1
- net +0V9_VCU: now reaches U26.AB18 (VCCINT_VCU), U26.AB19 (VCCINT_VCU), U26.AB20 (VCCINT_VCU), U26.AB21 (VCCINT_VCU)
- net +0V9_VCU: now also C158.2, C159.1, C160.2, C161.1
- net +3V3: now reaches U26.B22 (VCCO_PSIO1_501), U26.B27 (VCCO_PSIO2_502), U26.D18 (VCCO_PSIO0_500), U26.D23 (VCCO_PSIO1_501), U26.D28 (VCCO_PSIO2_502), U26.E21 (VCCO_PSIO1_501), U26.E26 (VCCO_PSIO2_502), U26.F19 (VCCO_PSIO0_500), U26.J18 (VCCO_PSIO0_500), U26.N20 (VCCO_PSIO3_503), U26.P18 (VCCO_PSIO3_503)
- net +3V3: now also U26.D13 (VCCO_46), U26.E16 (VCCO_45), U26.G12 (VCCO_46), U26.H15 (VCCO_45), C226.2, C227.2, C228.1, C235.2, C236.1, C237.2, C238.1, C239.2, C240.1
- net +1V8_MGTRAVTT: now reaches U26.H25 (PS_MGTRAVTT), U26.K25 (PS_MGTRAVTT), U26.L27 (PS_MGTRAVTT)
- net +1V8_MGTRAVTT: now also C203.2, C204.2, C205.1
- net +0V85_GTR: now reaches U26.J23 (PS_MGTRAVCC), U26.L23 (PS_MGTRAVCC)
- net +0V85_GTR: now also C201.2, C202.1
- net +0V85: now reaches U26.L11 (VCCINT), U26.L13 (VCCINT), U26.L17 (VCCINT), U26.M12 (VCCINT), U26.M14 (VCCINT), U26.M16 (VCCINT), U26.M18 (VCCINT), U26.N11 (VCCINT), U26.N13 (VCCINT), U26.N15 (VCCINT), U26.N17 (VCCINT), U26.P12 (VCCINT), U26.P14 (VCCINT), U26.P16 (VCCINT), U26.R11 (VCCINT), U26.R13 (VCCINT), U26.R17 (VCCINT), U26.T12 (VCCINT), U26.T16 (VCCINT), U26.U11 (VCCINT), U26.U13 (VCCINT), U26.U17 (VCCINT), U26.V12 (VCCINT), U26.V16 (VCCINT), U26.W11 (VCCINT), U26.W13 (VCCINT), U26.W15 (VCCINT), U26.Y12 (VCCINT), U26.Y14 (VCCINT)
- net +0V85: now also U26.R10 (VCCBRAM), U26.T10 (VCCBRAM), U26.T9 (VCCINT_IO), U26.U10 (VCCBRAM), U26.U8 (VCCINT_IO), U26.U9 (VCCINT_IO), U26.V10 (VCCBRAM), U26.V8 (VCCINT_IO), C120.2, C134.2, C135.1, C149.1, C150.2, C151.2, C152.1, C153.1, C154.2, C155.1, C156.2, C157.1
- net +1V8_CLEAN: now reaches U26.T18 (VCC_PSPLL), U26.T20 (VCC_PSPLL), U26.T21 (VCC_PSPLL)
- net +1V8_CLEAN: now also C197.2, C198.2, C199.1
- net +1V2_PS: now reaches U26.U18 (VCC_PSDDR_PLL)
- net +1V2_PS: now also U26.U19 (VCC_PSDDR_PLL), C195.2, C196.1
- net +1V8_VCCADC: now reaches U26.W22 (VCC_PSADC)
- net +1V8_VCCADC: now also C200.2
- new net: C201.1, C202.2
- new net: C123.2, C138.1
- new net: C214.2, C215.1
- new net: C125.2, C140.1
- new net: C126.2, C141.1
- new net: C218.2, C219.1
- new net: C216.2, C217.1
- new net: C130.2, C145.1
- new net: C132.2, C147.1
- new net: C233.2, C234.1
- new net: C169.2, C170.1
- new net: C122.2, C137.1
- new net: C176.2, C177.1
- new net: C121.2, C136.1
- new net: C127.2, C142.1
- new net: C124.2, C139.1
- new net: C229.2, C230.1
- new net: C208.2, C209.1
- new net: C231.2, C232.1
- new net: C131.2, C146.1
- new net: C129.2, C144.1
- new net: C191.2, C192.1
- new net: C133.2, C148.1
- new net: C128.2, C143.1
Other:
- note added: "DECOUPLING CAPACITORS"
- note added: "MGTAVCC"
- note added: "MGTVCCAUX"
- note added: "PS_MGTRAVCC"
- note added: "PS_MGTRAVTT"
- note added: "VCCADC"
- note added: "VCCAUX+IO"
- note added: "VCCBRAM"
- note added: "VCCINT"
- note added: "VCCINT_IO"
- note added: "VCCINT_VCU"
- note added: "VCCO_64+65+66"
- note added: "VCCO_PSDDR_504"
- note added: "VCC_45+46"
- note added: "VCC_PSADC"
- note added: "VCC_PSAUX"
- note added: "VCC_PSDDR_PLL"
- note added: "VCC_PSINTFP + PSINTLP + DDR"
- note added: "VCC_PSIO"
- note added: "VCC_PSPLL"
- note added: "VREFP"
- note removed: "1.32V"
- note removed: "1.65V"
- note removed: "1V"
- note removed: "2V"
- note removed: "3.630V"
- company: (none) -> Hemanth and CO

Commit message: Feat: Completed Zynq Core
Parts:
- removed C117: 0.1uF, Capacitor_SMD:C_0402_1005Metric, symbol Device:C
- removed C118: 1uF, Capacitor_SMD:C_0402_1005Metric, symbol Device:C
- removed C119: 47uF, Capacitor_SMD:C_1210_3225Metric, symbol Device:C
- renumbered C120 to C117, C121 to C118, C122 to C119, C123 to C120, C124 to C121, C125 to C122, C126 to C123, C127 to C124, C128 to C125, C129 to C126, C130 to C127, C131 to C128, C132 to C129, C133 to C130, C134 to C131, C150 to C132, C151 to C133, C154 to C134, C156 to C135, C135 to C136, C136 to C137, C137 to C138, C138 to C139, C139 to C140, C140 to C141, C141 to C142, C142 to C143, C143 to C144, C144 to C145, C145 to C146, C146 to C147, C147 to C148, C148 to C149, C149 to C150, C152 to C151, C153 to C152, C155 to C153, C157 to C154, C167 to C155, C169 to C156, C171 to C157, C174 to C158, C176 to C159, C178 to C160, C181 to C161, C158 to C162, C160 to C163, C162 to C164, C164 to C165, C185 to C166, C187 to C167, C173 to C168, C180 to C169, C183 to C170, C166 to C171, C168 to C172, C170 to C173, C172 to C174, C177 to C176, C179 to C177, C182 to C178, C159 to C179, C161 to C180, C163 to C181, C165 to C182, C186 to C183, C188 to C184, C189 to C185, C191 to C186, C193 to C187, C201 to C188, C198 to C189, C195 to C190, C184 to C191, C197 to C192, C200 to C193, C190 to C194, C192 to C195, C194 to C196, C202 to C197, C199 to C198, C196 to C199, C206 to C200, C208 to C201, C210 to C202, C212 to C203, C214 to C204, C216 to C205, C218 to C206, C220 to C207, C223 to C208, C204 to C209, C222 to C210, C225 to C211, C203 to C212, C207 to C213, C209 to C214, C211 to C215, C213 to C216, C215 to C217, C217 to C218, C221 to C220, C224 to C221, C205 to C222, C237 to C223, C239 to C224, C241 to C225, C243 to C226, C245 to C227, C247 to C228, C227 to C229, C229 to C230, C233 to C232, C235 to C233, C249 to C234, C250 to C235, C226 to C236, C238 to C237, C240 to C238, C242 to C239, C244 to C240, C246 to C241, C248 to C242, C228 to C243, C230 to C244, C232 to C245, C234 to C246, C236 to C247
Connections:
- net SD0_CD: now reaches U26.A18 (PS_MIO24)
- net SD0_D5: now reaches U26.A19 (PS_MIO20)
- net QSPI_IO0: now reaches U26.A20 (PS_MIO1)
- net UART1_RX: now reaches U26.A21 (PS_MIO28)
- net I2C0_SCL: now reaches U26.A22 (PS_MIO31)
- net USB2_NXT: now reaches U26.A23 (PS_MIO54)
- net USB2_CLK: now reaches U26.A24 (PS_MIO52)
- net USB2_D0: now reaches U26.A25 (PS_MIO56)
- net USB2_D1: now reaches U26.A26 (PS_MIO57)
- net USB2_D3: now reaches U26.A27 (PS_MIO59)
- net USB2_D2: now reaches U26.A28 (PS_MIO58)
- net USB2_D7: now reaches U26.A29 (PS_MIO63)
- net EXP_LANE2_RX_N: now reaches U26.A3 (MGTHRXN3_226)
- net EXP_LANE2_RX_P: now reaches U26.A4 (MGTHRXP3_226)
- net EXP_LANE2_TX_N: now reaches U26.A7 (MGTHTXN3_226)
- net EXP_LANE2_TX_P: now reaches U26.A8 (MGTHTXP3_226)
- net PS_DDR_DQ37: now reaches U26.AA23 (PS_DDR_DQ37)
- net PS_DDR_DQ38: now reaches U26.AA25 (PS_DDR_DQ38)
- net PS_DDR_DQ68: now reaches U26.AA26 (PS_DDR_DQ68)
- net PS_DDR_DM8: now reaches U26.AA27 (PS_DDR_DM8)
- net PS_DDR_DQS_N8: now reaches U26.AA28 (PS_DDR_DQS_N8)
- net PS_DDR_DQ65: now reaches U26.AA30 (PS_DDR_DQ65)
- net PS_DDR_ALERT_N: now reaches U26.AB24 (PS_DDR_ALERT_N)
- net PS_DDR_RAM_RST_N: now reaches U26.AB25 (PS_DDR_RAM_RST_N)
- net PS_DDR_PARITY: now reaches U26.AB26 (PS_DDR_PARITY)
- net PS_DDR_CKE1: now reaches U26.AB28 (PS_DDR_CKE1)
- net PS_DDR_DQ64: now reaches U26.AB29 (PS_DDR_DQ64)
- net PS_DDR_ODT0: now reaches U26.AB30 (PS_DDR_ODT0)
- net PS_DDR_DQS_P2: now reaches U26.AC21 (PS_DDR_DQS_P2)
- net PS_DDR_DQ28: now reaches U26.AC22 (PS_DDR_DQ28)
- net PS_DDR_DQ29: now reaches U26.AC23 (PS_DDR_DQ29)
- net PS_DDR_DQ31: now reaches U26.AC24 (PS_DDR_DQ31)
- net PS_DDR_BA1: now reaches U26.AC26 (PS_DDR_BA1)
- net PS_DDR_BG1: now reaches U26.AC27 (PS_DDR_BG1)
- net PS_DDR_BG0: now reaches U26.AC28 (PS_DDR_BG0)
- net PS_DDR_ODT1: now reaches U26.AC29 (PS_DDR_ODT1)
- net PS_DDR_CKE0: now reaches U26.AC30 (PS_DDR_CKE0)
- net PS_DDR_DQ20: now reaches U26.AD20 (PS_DDR_DQ20)
- net PS_DDR_DQS_N2: now reaches U26.AD21 (PS_DDR_DQS_N2)
- net PS_DDR_DQ16: now reaches U26.AD22 (PS_DDR_DQ16)
- net PS_DDR_DQS_P3: now reaches U26.AD24 (PS_DDR_DQS_P3)
- net PS_DDR_DQ30: now reaches U26.AD25 (PS_DDR_DQ30)
- net PS_DDR_ACT_N: now reaches U26.AD26 (PS_DDR_ACT_N)
- net PS_DDR_BA0: now reaches U26.AD27 (PS_DDR_BA0)
- net PS_DDR_CS_N1: now reaches U26.AD29 (PS_DDR_CS_N1)
- net PS_DDR_CS_N0: now reaches U26.AD30 (PS_DDR_CS_N0)
- net PS_DDR_DQ22: now reaches U26.AE20 (PS_DDR_DQ22)
- net PS_DDR_DQ17: now reaches U26.AE22 (PS_DDR_DQ17)
- net PS_DDR_DQ27: now reaches U26.AE23 (PS_DDR_DQ27)
- net PS_DDR_DQS_N3: now reaches U26.AE24 (PS_DDR_DQS_N3)
- net PS_DDR_DM3: now reaches U26.AE25 (PS_DDR_DM3)
- net PS_DDR_A7: now reaches U26.AE27 (PS_DDR_A7)
- net PS_DDR_A11: now reaches U26.AE28 (PS_DDR_A11)
- net PS_DDR_A10: now reaches U26.AE29 (PS_DDR_A10)
- net PS_DDR_CK0: now reaches U26.AE30 (PS_DDR_CK0)
- net PS_DDR_DQ21: now reaches U26.AF20 (PS_DDR_DQ21)
- net PS_DDR_DM2: now reaches U26.AF21 (PS_DDR_DM2)
- net PS_DDR_DQ18: now reaches U26.AF22 (PS_DDR_DQ18)
- net PS_DDR_DQ25: now reaches U26.AF23 (PS_DDR_DQ25)
- net PS_DDR_DQ26: now reaches U26.AF25 (PS_DDR_DQ26)
- net PS_DDR_A8: now reaches U26.AF26 (PS_DDR_A8)
- net PS_DDR_A6: now reaches U26.AF27 (PS_DDR_A6)
- net PS_DDR_CK1: now reaches U26.AF28 (PS_DDR_CK1)
- net PS_DDR_CK_N0: now reaches U26.AF30 (PS_DDR_CK_N0)
- net PS_DDR_DQ23: now reaches U26.AG20 (PS_DDR_DQ23)
- net PS_DDR_DQ19: now reaches U26.AG21 (PS_DDR_DQ19)
- net PS_DDR_DQ24: now reaches U26.AG23 (PS_DDR_DQ24)
- net PS_DDR_DQ10: now reaches U26.AG24 (PS_DDR_DQ10)
- net PS_DDR_DQ14: now reaches U26.AG25 (PS_DDR_DQ14)
- net PS_DDR_A9: now reaches U26.AG26 (PS_DDR_A9)
- net PS_DDR_CK_N1: now reaches U26.AG28 (PS_DDR_CK_N1)
- net PS_DDR_A14: now reaches U26.AG29 (PS_DDR_A14)
- net PS_DDR_A1: now reaches U26.AG30 (PS_DDR_A1)
- net PS_DDR_DQ7: now reaches U26.AH19 (PS_DDR_DQ7)
- net PS_DDR_DQ1: now reaches U26.AH21 (PS_DDR_DQ1)
- net PS_DDR_DQ0: now reaches U26.AH22 (PS_DDR_DQ0)
- net PS_DDR_DQ8: now reaches U26.AH23 (PS_DDR_DQ8)
- net PS_DDR_DQS_P1: now reaches U26.AH24 (PS_DDR_DQS_P1)
- net PS_DDR_DQ15: now reaches U26.AH26 (PS_DDR_DQ15)
- net PS_DDR_A16: now reaches U26.AH27 (PS_DDR_A16)
- net PS_DDR_A13: now reaches U26.AH28 (PS_DDR_A13)
- net PS_DDR_A12: now reaches U26.AH29 (PS_DDR_A12)
- net PS_DDR_A0: now reaches U26.AH30 (PS_DDR_A0)
- net PS_DDR_DQ5: now reaches U26.AJ19 (PS_DDR_DQ5)
- net PS_DDR_DM0: now reaches U26.AJ20 (PS_DDR_DM0)
- net PS_DDR_DQS_P0: now reaches U26.AJ21 (PS_DDR_DQS_P0)
- net PS_DDR_DQ2: now reaches U26.AJ22 (PS_DDR_DQ2)
- net PS_DDR_DQS_N1: now reaches U26.AJ24 (PS_DDR_DQS_N1)
- net PS_DDR_DM1: now reaches U26.AJ25 (PS_DDR_DM1)
- net PS_DDR_DQ12: now reaches U26.AJ26 (PS_DDR_DQ12)
- net PS_DDR_A17: now reaches U26.AJ27 (PS_DDR_A17)
- net PS_DDR_A15: now reaches U26.AJ29 (PS_DDR_A15)
- net PS_DDR_A2: now reaches U26.AJ30 (PS_DDR_A3)
- net PS_DDR_A2: now also U26.AK29 (PS_DDR_A2)
- net PS_DDR_DQ6: now reaches U26.AK19 (PS_DDR_DQ6)
- net PS_DDR_DQ4: now reaches U26.AK20 (PS_DDR_DQ4)
- net PS_DDR_DQS_N0: now reaches U26.AK21 (PS_DDR_DQS_N0)
- net PS_DDR_DQ3: now reaches U26.AK22 (PS_DDR_DQ3)
- net PS_DDR_DQ9: now reaches U26.AK23 (PS_DDR_DQ9)
- net PS_DDR_DQ11: now reaches U26.AK24 (PS_DDR_DQ11)
- net PS_DDR_DQ13: now reaches U26.AK25 (PS_DDR_DQ13)
- net PS_DDR_A5: now reaches U26.AK27 (PS_DDR_A5)
- net PS_DDR_A4: now reaches U26.AK28 (PS_DDR_A4)
- net EXP_LANE1_RX_N: now reaches U26.B1 (MGTHRXN2_226)
- net GTH_REFCLK1_156M_P: now reaches U26.B10 (MGTREFCLK1P_226)
- net SD0_WP: now reaches U26.B18 (PS_MIO25)
- net QSPI_IO1: now reaches U26.B19 (PS_MIO2)
- net EXP_LANE1_RX_P: now reaches U26.B2 (MGTHRXP2_226)
- net UART0_TX: now reaches U26.B20 (PS_MIO26)
- net UART1_TX: now reaches U26.B21 (PS_MIO27)
- net GPIO_PD_IRQ: now reaches U26.B23 (PS_MIO35)
- net GPIO_PD_IRQ: now also U26.G18 (PS_MIO11)
- net GPIO_BMC_IRQ: now reaches U26.B24 (PS_MIO34)
- net USB2_DIR: now reaches U26.B25 (PS_MIO53)
- net USB2_STP: now reaches U26.B26 (PS_MIO55)
- net USB2_D6: now reaches U26.B28 (PS_MIO62)
- net USB2_D5: now reaches U26.B29 (PS_MIO61)
- net GEM_TXC: now reaches U26.B30 (PS_MIO64)
- net EXP_LANE1_TX_N: now reaches U26.B5 (MGTHTXN2_226)
- net EXP_LANE1_TX_P: now reaches U26.B6 (MGTHTXP2_226)
- net GTH_REFCLK1_156M_N: now reaches U26.B9 (MGTREFCLK1N_226)
- net SD0_D2: now reaches U26.C18 (PS_MIO17)
- net QSPI_SS: now reaches U26.C19 (PS_MIO5)
- net I2C1_SCL: now reaches U26.C21 (PS_MIO30)
- net I2C0_SDA: now reaches U26.C22 (PS_MIO33)
- net SD1_CMD: now reaches U26.C24 (PS_MIO40)
- net USB2_D4: now reaches U26.C26 (PS_MIO60)
- net GEM_TXD1: now reaches U26.C27 (PS_MIO66)
- net GEM_TXD2: now reaches U26.C28 (PS_MIO67)
- net GEM_TXD3: now reaches U26.C29 (PS_MIO68)
- net EXP_LANE0_RX_N: now reaches U26.C3 (MGTHRXN1_226)
- net EXP_LANE0_RX_P: now reaches U26.C4 (MGTHRXP1_226)
- net EXP_LANE0_TX_N: now reaches U26.C7 (MGTHTXN1_226)
- net EXP_LANE0_TX_P: now reaches U26.C8 (MGTHTXP1_226)
- net SFP_RX_N: now reaches U26.D1 (MGTHRXN0_226)
- net GTH_REFCLK0_156M_P: now reaches U26.D10 (MGTREFCLK0P_226)
- net QSPI_IO2: now reaches U26.D19 (PS_MIO3)
- net SFP_RX_P: now reaches U26.D2 (MGTHRXP0_226)
- net QSPI_FEEDBACK_CLK: now reaches U26.D20 (PS_MIO6)
- net UART0_RX: now reaches U26.D21 (PS_MIO29)
- net GPIO_SD1_PWR_EN: now reaches U26.D22 (PS_MIO36)
- net SD1_D0: now reaches U26.D24 (PS_MIO41)
- net GEM_TXD0: now reaches U26.D25 (PS_MIO65)
- net GEM_RXC: now reaches U26.D26 (PS_MIO70)
- net GEM_TX_CTL: now reaches U26.D27 (PS_MIO69)
- net GEM_RX_CTL: now reaches U26.D29 (PS_MIO75)
- net GEM_RXD0: now reaches U26.D30 (PS_MIO71)
- net SFP_TX_N: now reaches U26.D5 (MGTHTXN0_226)
- net SFP_TX_P: now reaches U26.D6 (MGTHTXP0_226)
- net GTH_REFCLK0_156M_N: now reaches U26.D9 (MGTREFCLK0N_226)
- net SD0_CMD: now reaches U26.E18 (PS_MIO14)
- net DP_AUX_P: now reaches U26.E19 (PS_MIO7)
- net DP_AUX_N: now reaches U26.E20 (PS_MIO8)
- net SD1_CLK: now reaches U26.E22 (PS_MIO39)
- net SD1_D1: now reaches U26.E23 (PS_MIO42)
- net SD1_D3: now reaches U26.E24 (PS_MIO44)
- net MDIO_MDIO: now reaches U26.E25 (PS_MIO77)
- net GEM_RXD1: now reaches U26.E27 (PS_MIO72)
- net MDIO_MDC: now reaches U26.E28 (PS_MIO76)
- net GEM_RXD3: now reaches U26.E29 (PS_MIO74)
- net GEM_RXD2: now reaches U26.E30 (PS_MIO73)
- net SD0_D7: now reaches U26.F17 (PS_MIO22)
- net GPIO_PHY_RST: now reaches U26.F18 (PS_MIO10)
- net DP_HPD: now reaches U26.F20 (PS_MIO9)
- net GPIO_BOOT_LED: now reaches U26.F21 (PS_MIO37)
- net SD1_D2: now reaches U26.F22 (PS_MIO43)
- net SD1_CD: now reaches U26.F23 (PS_MIO45)
- net SD0_CLK: now reaches U26.G19 (PS_MIO13)
- net I2C1_SDA: now reaches U26.G20 (PS_MIO32)
- net EXP_LANE4_RX_N: now reaches U26.G3 (MGTHRXN1_225)
- net EXP_LANE4_RX_P: now reaches U26.G4 (MGTHRXP1_225)
- net EXP_LANE4_TX_N: now reaches U26.G7 (MGTHTXN1_225)
- net EXP_LANE4_TX_P: now reaches U26.G8 (MGTHTXP1_225)
- net EXP_LANE3_RX_N: now reaches U26.H1 (MGTHRXN0_225)
- net QSPI_SCLK: now reaches U26.H17 (PS_MIO0)
- net SD0_D6: now reaches U26.H19 (PS_MIO21)
- net EXP_LANE3_RX_P: now reaches U26.H2 (MGTHRXP0_225)
- net DP_RX0_P: now reaches U26.H27 (PS_MGTRRXP2_505)
- net DP_RX0_N: now reaches U26.H28 (PS_MGTRRXN2_505)
- net EXP_LANE3_TX_N: now reaches U26.H5 (MGTHTXN0_225)
- net EXP_LANE3_TX_P: now reaches U26.H6 (MGTHTXP0_225)
- net QSPI_IO3: now reaches U26.J17 (PS_MIO4)
- net SD0_D0: now reaches U26.J19 (PS_MIO15)
- net DP_TX0_P: now reaches U26.J25 (PS_MGTRTXP2_505)
- net DP_TX0_N: now reaches U26.J26 (PS_MGTRTXN2_505)
- net PCIE_RX_P: now reaches U26.J29 (PS_MGTRRXP1_505)
- net PCIE_RX_N: now reaches U26.J30 (PS_MGTRRXN1_505)
- net SD0_D4: now reaches U26.K16 (PS_MIO19)
- net SD0_D1: now reaches U26.K17 (PS_MIO16)
- net SD0_D3: now reaches U26.K18 (PS_MIO18)
- net SD0_RST: now reaches U26.K19 (PS_MIO23)
- net GPIO_EXP_RST: now reaches U26.K20 (PS_MIO46)
- net GPIO_ESP_IRQ: now reaches U26.K21 (PS_MIO47)
- net PCIE_TX_P: now reaches U26.K27 (PS_MGTRTXP1_505)
- net PCIE_TX_N: now reaches U26.K28 (PS_MGTRTXN1_505)
- net PS_JTAG_TCK: now reaches U26.L19 (PS_JTAG_TCK)
- net PS_JTAG_TDI: now reaches U26.L20 (PS_JTAG_TDI)
- net PS_JTAG_TMS: now reaches U26.L21 (PS_JTAG_TMS)
- net PS_REFCLK1_27M_P: now reaches U26.L25 (PS_MGTREFCLK1P_505)
- net PS_REFCLK1_27M_N: now reaches U26.L26 (PS_MGTREFCLK1N_505)
- net USB3_RX_P: now reaches U26.L29 (PS_MGTRRXP0_505)
- net USB3_RX_N: now reaches U26.L30 (PS_MGTRRXN0_505)
- net PS_PROG_B: now reaches U26.M19 (PS_PROG_B)
- net PS_JTAG_TDO: now reaches U26.M20 (PS_JTAG_TDO)
- net PS_REFCLK0_100M_P: now reaches U26.M23 (PS_MGTREFCLK0P_505)
- net PS_REFCLK0_100M_N: now reaches U26.M24 (PS_MGTREFCLK0N_505)
- net USB3_TX_P: now reaches U26.M27 (PS_MGTRTXP0_505)
- net USB3_TX_N: now reaches U26.M28 (PS_MGTRTXN0_505)
- net PS_INIT_B: now reaches U26.N18 (PS_INIT_B)
- net PS_POR_B: now reaches U26.N19 (PS_POR_B)
- net PS_DONE: now reaches U26.N22 (PS_DONE)
- net PS_REF_CLK: now reaches U26.P19 (PS_REF_CLK)
- net PS_SRST_B: now reaches U26.P20 (PS_SRST_B)
- net PS_MODE2: now reaches U26.P21 (PS_MODE2)
- net PS_MODE3: now reaches U26.P22 (PS_MODE3)
- net PS_DDR_DQ40: now reaches U26.P23 (PS_DDR_DQ40)
- net PS_DDR_DQ47: now reaches U26.P24 (PS_DDR_DQ47)
- net PS_DDR_DQS_P5: now reaches U26.P25 (PS_DDR_DQS_P5)
- net PS_DDR_DQ43: now reaches U26.P26 (PS_DDR_DQ43)
- net PS_DDR_DQ62: now reaches U26.P27 (PS_DDR_DQ62)
- net PS_DDR_DM7: now reaches U26.P28 (PS_DDR_DM7)
- net PS_DDR_DQ59: now reaches U26.P29 (PS_DDR_DQ59)
- net PS_DDR_DQ58: now reaches U26.P30 (PS_DDR_DQ58)
- net PS_MODE0: now reaches U26.R18 (PS_MODE0)
- net PS_MODE1: now reaches U26.R19 (PS_MODE1)
- net PS_ERROR_STATUS: now reaches U26.R20 (PS_ERROR_STATUS)
- net PS_ERROR_OUT: now reaches U26.R22 (PS_ERROR_OUT)
- net PS_DDR_DQ41: now reaches U26.R23 (PS_DDR_DQ41)
- net PS_DDR_DM5: now reaches U26.R24 (PS_DDR_DM5)
- net PS_DDR_DQS_N5: now reaches U26.R25 (PS_DDR_DQS_N5)
- net PS_DDR_DQ63: now reaches U26.R27 (PS_DDR_DQ63)
- net PS_DDR_DQS_P7: now reaches U26.R28 (PS_DDR_DQS_P7)
- net PS_DDR_DQS_N7: now reaches U26.R29 (PS_DDR_DQS_N7)
- net PS_DDR_DQ56: now reaches U26.R30 (PS_DDR_DQ56)
- net SYSMON_VP: now reaches U26.T15 (VP)
- net PS_DDR_DQ42: now reaches U26.T23 (PS_DDR_DQ42)
- net PS_DDR_DQ44: now reaches U26.T25 (PS_DDR_DQ44)
- net PS_DDR_DQ46: now reaches U26.T26 (PS_DDR_DQ46)
- net PS_DDR_DQ61: now reaches U26.T27 (PS_DDR_DQ61)
- net PS_DDR_DQ60: now reaches U26.T28 (PS_DDR_DQ60)
- net PS_DDR_DQ57: now reaches U26.T30 (PS_DDR_DQ57)
- net SYSMON_VN: now reaches U26.U14 (VN)
- net SYSMON_VREFP: now reaches U26.U15 (VREFP)
- net PS_DDR_DQ45: now reaches U26.U23 (PS_DDR_DQ45)
- net PS_DDR_DQ32: now reaches U26.U24 (PS_DDR_DQ32)
- net PS_DDR_DQ34: now reaches U26.U25 (PS_DDR_DQ34)
- net PS_DDR_DQ48: now reaches U26.U26 (PS_DDR_DQ48)
- net PS_DDR_DQ50: now reaches U26.U28 (PS_DDR_DQ50)
- net PS_DDR_DQS_P6: now reaches U26.U29 (PS_DDR_DQS_P6)
- net PS_DDR_DQ52: now reaches U26.U30 (PS_DDR_DQ52)
- net SYSMON_DXN: now reaches U26.V14 (DXN)
- net SYSMON_DXP: now reaches U26.V15 (DXP)
- net PS_DDR_DQ33: now reaches U26.V23 (PS_DDR_DQ33)
- net PS_DDR_DQ35: now reaches U26.V24 (PS_DDR_DQ35)
- net PS_DDR_DQ49: now reaches U26.V26 (PS_DDR_DQ49)
- net PS_DDR_DQ51: now reaches U26.V27 (PS_DDR_DQ51)
- net PS_DDR_DM6: now reaches U26.V28 (PS_DDR_DM6)
- net PS_DDR_DQS_N6: now reaches U26.V29 (PS_DDR_DQS_N6)
- net PS_DDR_DQ53: now reaches U26.V30 (PS_DDR_DQ53)
- net PS_DDR_DQS_P4: now reaches U26.W24 (PS_DDR_DQS_P4)
- net PS_DDR_DQS_N4: now reaches U26.W25 (PS_DDR_DQS_N4)
- net PS_DDR_DQ71: now reaches U26.W26 (PS_DDR_DQ71)
- net PS_DDR_DQ69: now reaches U26.W27 (PS_DDR_DQ69)
- net PS_DDR_DQ55: now reaches U26.W29 (PS_DDR_DQ55)
- net PS_DDR_DQ54: now reaches U26.W30 (PS_DDR_DQ54)
- net PS_DDR_DQ39: now reaches U26.Y23 (PS_DDR_DQ39)
- net PS_DDR_DM4: now reaches U26.Y24 (PS_DDR_DM4)
- net PS_DDR_DQ36: now reaches U26.Y25 (PS_DDR_DQ36)
- net PS_DDR_DQ70: now reaches U26.Y27 (PS_DDR_DQ70)
- net PS_DDR_DQS_P8: now reaches U26.Y28 (PS_DDR_DQS_P8)
- net PS_DDR_DQ67: now reaches U26.Y29 (PS_DDR_DQ67)
- net PS_DDR_DQ66: now reaches U26.Y30 (PS_DDR_DQ66)
- no-connect marks 5 -> 281
Other:
- note added: "SECTION 04a : Zynq Core"
- moved on the sheet: C117, C118, C119, C120, C121, C122, C123, C124, C125, C126, C127, C128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

Commit message: Feat: DDR4 Memory added
Connections:
- net PS_DDR_A2: no longer U26.AJ30 (PS_DDR_A3)
- new net PS_DDR_A3: U26.AJ30 (PS_DDR_A3)
Changed lines of the file:
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@@
 		)
 	)
-	(global_label "PS_DDR_A2"
+	(global_label "PS_DDR_A3"
 		(shape input)
 		(at 943.61 730.25 0)

Commit message: Feat: Zynq Peripherals added
Connections:
- net +0V85: no longer U26.R10 (VCCBRAM), U26.T9 (VCCINT_IO), U26.V10 (VCCBRAM), U26.V8 (VCCINT_IO)
- net +0V9_VCU: no longer U26.AB18 (VCCINT_VCU), U26.AB21 (VCCINT_VCU)
- net +1V8: no longer U26.T22 (VCC_PSAUX), U26.V22 (VCC_PSAUX)
- net +3V3: no longer U26.D13 (VCCO_46), U26.H15 (VCCO_45)
- net GEM_RST: now reaches U26.C23 (PS_MIO38)
- no-connect marks 281 -> 280

Commit message: Feat : Completed 04d Peripherals
Changed lines of the file:
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@@
 	(generator "eeschema")
 	(generator_version "10.0")
-	(paper "User" 1300 1300)
+	(paper "User" 1300 1500)
 	(title_block
 		(date "2026-10-24")
@@
 		)
 		(stroke
+			(width 0)
+			(type default)
+		)
+	)
+	(wire
+		(pts
+			(xy 1008.38 582.93) (xy 1014.73 582.93)
+		)
+		(stroke

Commit message: Added 04D High Speed Peripherals
Changed lines of the file:
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@@
-	(wire
-		(pts
-			(xy 1008.38 582.93) (xy 1014.73 582.93)
-		)
-		(stroke
-			(width 0)
-			(type default)
-		)
-	)
 	(wire
 		(pts
