File: PCB/schematics/04_Zynq/04a_Zynq_Core.kicad_sch (KiCad schematic)
At the start: 132 parts, among them U26 xczu4evfbvb900pkg

Commit message: High Speed Peripherals added
Parts:
- added R159: 220Ω, Resistor_SMD:R_0402_1005Metric, symbol Device:R
Connections:
- net GND: now also R159.2
- net USB3_VBUS_NET: now reaches U26.G21 (PS_MIO49)
- net at U26.M25 (PS_MGTRREF_505): now also R159.1
- no-connect marks 280 -> 278
Changed lines of the file:
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@@
 	)
 	(no_connect
-		(at 943.61 582.93)
-	)
-	(no_connect
 		(at 293.37 709.93)
 	)
@@
 	)
 	(no_connect
-		(at 943.61 1108.71)
-	)
-	(no_connect
 		(at 293.37 628.65)
 	)
@@
 		)
 	)
+	(global_label "USB3_VBUS_NET"
+		(shape input)
+		(at 943.61 582.93 0)
+		(fields_autoplaced yes)
+		(effects
+			(font
+				(size 1.27 1.27)
+			)
+			(justify left)
+		)
+		(property "Intersheetrefs" "${INTERSHEET_REFS}"
+			(at 961.8956 582.93 0)
+			(hide yes)
+			(show_name no)
+			(do_not_autoplace no)
+			(effects
+				(font
+					(size 1.27 1.27)
+				)
+				(justify left)
+			)
+		)
+	)
 	(global_label "DP_AUX_P"
 		(shape input)
@@
 	)
 	(symbol
+		(lib_id "Device:R")
+		(at 947.42 1108.71 90)
+		(unit 1)
+		(body_style 1)
+		(exclude_from_sim no)
+		(in_bom yes)
+		(on_board yes)
+		(in_pos_files yes)
+		(dnp no)
+		(property "Reference" "R159"
+			(at 947.42 1110.742 90)
+			(show_name no)
+			(do_not_autoplace no)
+			(effects
+				(font
+					(size 1.27 1.27)
+				)
+			)
+		)
+		(property "Value" "220Ω"
+			(at 947.42 1108.71 90)
+			(show_name no)
+			(do_not_autoplace no)
+			(effects
+				(font
+					(size 1 1)
+				)
+			)
+		)
+		(property "Footprint" "Resistor_SMD:R_0402_1005Metric"
+			(at 947.42 1110.488 90)
+			(hide yes)
+			(show_name no)
+			(do_not_autoplace no)
+			(effects
+				(font
+					(size 1.27 1.27)
+				)
+			)
+		)
+		(property "Datasheet" ""
+			(at 947.42 1108.71 0)
+			(hide yes)
+			(show_name no)
+			(do_not_autoplace no)
+			(effects
+				(font
+					(size 1.27 1.27)
+				)
+			)
+		)
+		(property "Description" "Resistor"
+			(at 947.42 1108.71 0)
+			(hide yes)
+			(show_name no)
+			(do_not_autoplace no)
+			(effects
+				(font
+					(size 1.27 1.27)
+				)
+			)
+		)
+		(pin "1"
+		)
+		(pin "2"
+		)
+		(instances
+			(project "Devboard"
+				(path "/f4f7837f-dd80-4f77-b150-4534de1c10d6/b48c92d5-ffe6-40f3-9dff-a09c41a730f7/67e8dda6-f6da-452b-ac2a-efb32270ca28"
+					(reference "R159")
+					(unit 1)
+				)
+			)
+		)
+	)
+	(symbol
 		(lib_id "Device:C")
 		(at 204.47 309.88 0)
@@
 	)
 	(symbol
+		(lib_id "power:GND")
+		(at 951.23 1108.71 90)
+		(unit 1)
+		(body_style 1)
+		(exclude_from_sim no)
+		(in_bom yes)
+		(on_board yes)
+		(in_pos_files yes)
+		(dnp no)
+		(fields_autoplaced yes)
+		(property "Reference" "#PWR0838"
+			(at 957.58 1108.71 0)
+			(hide yes)
+			(show_name no)
+			(do_not_autoplace no)
+			(effects
+				(font
+					(size 1.27 1.27)
+				)
+			)
+		)
+		(property "Value" "GND"
+			(at 955.04 1108.7099 90)
+			(show_name no)
+			(do_not_autoplace no)
+			(effects
+				(font
+					(size 1.27 1.27)
+				)
+				(justify right)
+			)
+		)
+		(property "Footprint" ""
+			(at 951.23 1108.71 0)
+			(hide yes)
+			(show_name no)
+			(do_not_autoplace no)
+			(effects
+				(font
+					(size 1.27 1.27)
+				)
+			)
+		)
+		(property "Datasheet" ""
+			(at 951.23 1108.71 0)
+			(hide yes)
+			(show_name no)
+			(do_not_autoplace no)
+			(effects
+				(font
+					(size 1.27 1.27)
+				)
+			)
+		)
+		(property "Description" "Power symbol creates a global label with name \"GND\" , ground"
+			(at 951.23 1108.71 0)
+			(hide yes)
+			(show_name no)
+			(do_not_autoplace no)
+			(effects
+				(font
+					(size 1.27 1.27)
+				)
+			)
+		)
+		(pin "1"
+		)
+		(instances
+			(project "Devboard"
+				(path "/f4f7837f-dd80-4f77-b150-4534de1c10d6/b48c92d5-ffe6-40f3-9dff-a09c41a730f7/67e8dda6-f6da-452b-ac2a-efb32270ca28"
+					(reference "#PWR0838")
+					(unit 1)
+				)
+			)
+		)
+	)
+	(symbol
 		(lib_id "Device:C")
 		(at 146.05 320.04 0)
@@
 	(symbol
 		(lib_id "power:+3.3V")
-		(at 250.19 292.1 270)
+		(at 250.19 292.1 90)
 		(unit 1)
 		(body_style 1)
@@
 		(dnp no)
 		(property "Reference" "#PWR0477"
-			(at 246.38 292.1 0)
+			(at 254 292.1 0)
 			(hide yes)
 			(show_name no)
@@
 		)
 		(property "Value" "+1V8_VCCADC"
-			(at 252.73 292.1 90)
+			(at 247.65 292.1 90)
 			(show_name no)
 			(do_not_autoplace no)

Commit message: feat: Section 4 Done
Connections:
- net MIO51: now reaches U26.H21 (PS_MIO51)
- net MIO50: now reaches U26.J20 (PS_MIO50)
- no-connect marks 278 -> 276

Commit message: Feat : Schematics Complete
Parts:
- renumbered C117 to C121, C118 to C122, C119 to C123, C120 to C124, C121 to C125, C122 to C126, C123 to C127, C124 to C128, C125 to C129, C126 to C130, C127 to C131, C128 to C132, C129 to C133, C130 to C134, C131 to C135, C132 to C136, C133 to C137, C134 to C138, C135 to C139, C136 to C140, C137 to C141, C138 to C142, C139 to C143, C140 to C144, C141 to C145, C142 to C146, C143 to C147, C144 to C148, C145 to C149, C146 to C150, C147 to C151, C148 to C152, C149 to C153, C150 to C154, C151 to C155, C152 to C156, C153 to C157, C154 to C158, C155 to C159, C156 to C160, C157 to C161, C158 to C162, C159 to C163, C160 to C164, C161 to C165, C162 to C166, C163 to C167, C164 to C168, C165 to C169, C166 to C170, C167 to C171, C168 to C172, C169 to C173, C170 to C174, C171 to C175, C172 to C176, C173 to C177, C174 to C178, C175 to C179, C176 to C180, C177 to C181, C178 to C182, C179 to C183, C180 to C184, C181 to C185, C182 to C186, C183 to C187, C184 to C188, C185 to C189, C186 to C190, C187 to C191, C188 to C192, C189 to C193, C190 to C194, C191 to C195, C192 to C196, C193 to C197, C194 to C198, C195 to C199, C196 to C200, C197 to C201, C198 to C202, C199 to C203, C200 to C204, C201 to C205, C202 to C206, C203 to C207, C204 to C208, C205 to C209, C206 to C210, C207 to C211, C208 to C212, C209 to C213, C210 to C214, C211 to C215, C212 to C216, C213 to C217, C214 to C218, C215 to C219, C216 to C220, C217 to C221, C218 to C222, C219 to C223, C220 to C224, C221 to C225, C222 to C226, C223 to C227, C224 to C228, C225 to C229, C226 to C230, C227 to C231, C228 to C232, C229 to C233, C230 to C234, C231 to C235, C232 to C236, C233 to C237, C234 to C238, C235 to C239, C236 to C240, C237 to C241, C238 to C242, C239 to C243, C240 to C244, C241 to C245, C242 to C246, C243 to C247, C244 to C248, C245 to C249, C246 to C250, C247 to C251, R159 to R103, U26 to U27
Connections:
- net +0V85: now also U27.R10 (VCCBRAM), U27.T9 (VCCINT_IO), U27.V10 (VCCBRAM)
- net +0V9_VCU: now also U27.AB18 (VCCINT_VCU), U27.AB21 (VCCINT_VCU), U27.V8 (VCCINT_IO)
- net +1V2: now also U27.AA4 (VCCO_66), U27.AD3 (VCCO_66), U27.AD8 (VCCO_66)
- net +1V8: now also U27.T22 (VCC_PSAUX), U27.V22 (VCC_PSAUX); no longer U27.AA4 (VCCO_66), U27.AD3 (VCCO_66), U27.AD8 (VCCO_66)
- net +3V3: now also U27.D13 (VCCO_46), U27.H15 (VCCO_45)
- net MIPI_D0_N: now reaches U27.AA11 (IO_L2N_T0L_N3_66)
- net MIPI_D0_P: now reaches U27.AA12 (IO_L2P_T0L_N2_66)
- net MIPI_D3_P: now reaches U27.AB10 (IO_L5P_T0U_N8_AD14P_66)
- net MIPI_CLK_P: now reaches U27.AB11 (IO_L3P_T0L_N4_AD15P_66)
- net MIPI_D3_N: now reaches U27.AB9 (IO_L5N_T0U_N9_AD14N_66)
- net MIPI_CLK_N: now reaches U27.AC11 (IO_L3N_T0L_N5_AD15N_66)
- net MIPI_D1_P: now reaches U27.AC12 (IO_L1P_T0L_N0_DBC_66)
- net MIPI_D2_N: now reaches U27.AD10 (IO_L4N_T0U_N7_DBC_AD7N_66)
- net MIPI_D2_P: now reaches U27.AD11 (IO_L4P_T0U_N6_DBC_AD7P_66)
- net MIPI_D1_N: now reaches U27.AD12 (IO_L1N_T0L_N1_DBC_66)
- net ADC_CLKOUTP: now reaches U27.AE8 (IO_L10N_T1U_N7_QBC_AD4N_65)
- net ADC_CLKOUTM: now reaches U27.AE9 (IO_L10P_T1U_N6_QBC_AD4P_65)
- net ADC_DA10_P: now reaches U27.AF10 (IO_L6P_T0U_N10_AD6P_65)
- net ADC_DB4_M: now reaches U27.AF5 (IO_L18N_T2U_N11_AD2N_65)
- net ADC_DB4_P: now reaches U27.AF6 (IO_L18P_T2U_N10_AD2P_65)
- net ADC_DA12_M: now reaches U27.AF7 (IO_L9N_T1L_N5_AD12N_65)
- net ADC_DA12_P: now reaches U27.AF8 (IO_L9P_T1L_N4_AD12P_65)
- net ADC_DA10_M: now reaches U27.AG10 (IO_L6N_T0U_N11_AD6N_65)
- net ADC_DB10_M: now reaches U27.AG3 (IO_L22N_T3U_N7_DBC_AD0N_65)
- net ADC_DB10_P: now reaches U27.AG4 (IO_L22P_T3U_N6_DBC_AD0P_65)
- net ADC_DB12_M: now reaches U27.AH2 (IO_L21N_T3L_N5_AD8N_65)
- net ADC_DB12_P: now reaches U27.AH3 (IO_L21P_T3L_N4_AD8P_65)
- net ADC_DA8_M: now reaches U27.AH7 (IO_L12P_T1U_N10_GC_65)
- net ADC_DA8_P: now reaches U27.AH8 (IO_L11N_T1U_N9_GC_65)
- net ADC_DA2_P: now reaches U27.AH9 (IO_L8P_T1L_N2_AD5P_65)
- net ADC_DB6_M: now reaches U27.AJ1 (IO_L20N_T3L_N3_AD1N_65)
- net ADC_DA0_P: now reaches U27.AJ10 (IO_L5P_T0U_N8_AD14P_65)
- net ADC_DA4_P: now reaches U27.AJ11 (IO_L4P_T0U_N6_DBC_AD7P_SMBALERT_65)
- net ADC_DB6_P: now reaches U27.AJ2 (IO_L20P_T3L_N2_AD1P_65)
- net ADC_DB2_M: now reaches U27.AJ4 (IO_L17P_T2U_N8_AD10P_65)
- net ADC_DA6_P: now reaches U27.AJ6 (IO_L13N_T2L_N1_GC_QBC_65)
- net ADC_DA6_M: now reaches U27.AJ7 (IO_L12N_T1U_N11_GC_65)
- net ADC_DA2_M: now reaches U27.AJ9 (IO_L8N_T1L_N3_AD5N_65)
- net ADC_DA0_M: now reaches U27.AK10 (IO_L5N_T0U_N9_AD14N_65)
- net ADC_DA4_M: now reaches U27.AK11 (IO_L4N_T0U_N7_DBC_AD7N_65)
- net ADC_DB8_M: now reaches U27.AK2 (IO_L19N_T3L_N1_DBC_AD9N_65)
- net ADC_DB8_P: now reaches U27.AK3 (IO_L19P_T3L_N0_DBC_AD9P_65)
- net ADC_DB2_P: now reaches U27.AK4 (IO_L17N_T2U_N9_AD10N_65)
- net ADC_DB0_P: now reaches U27.AK6 (IO_L15N_T2L_N5_AD11N_65)
- net ADC_DB0_M: now reaches U27.AK7 (IO_L15P_T2L_N4_AD11P_65)
- net ADS_SYNC: now reaches U27.C17 (IO_L10P_AD10P_45)
- net ADS_DRDY: now reaches U27.D16 (IO_L9P_AD11P_45)
- net ADS_DOUT: now reaches U27.E15 (IO_L8P_HDGC_45)
- net ADS_DIN: now reaches U27.E17 (IO_L7P_HDGC_45)
- net ADS_SCLK: now reaches U27.F16 (IO_L6P_HDGC_45)
- net ADS_CS: now reaches U27.G16 (IO_L5P_HDGC_45)
- net CAM_RST_N: now reaches U27.H18 (PS_MIO12)
- net LMX_CSB: now reaches U27.J15 (IO_L3P_AD13P_45)
- net LMS_SCK: now reaches U27.J16 (IO_L4P_AD12P_45)
- net FAN_TACH: now reaches U27.J21 (PS_MIO48)
- net LMX_SDI: now reaches U27.K15 (IO_L2P_AD14P_45)
- net LMX_MUXOUT: now reaches U27.L15 (IO_L1P_AD15P_45)
- net DP_HPD renamed GNSS_PPS
- net GPIO_PHY_RST renamed CAM_PWDN
- no-connect marks 276 -> 224
