File: PCB/schematics/04_Zynq/04b_Zynq_DDR4.kicad_sch (KiCad schematic)
At the start: 0 parts

Commit message: Feat: DDR4 Memory added
Parts:
- added C248, C249, C250, C251, C252, C253, C254, C255, C256, C257, C258, C259, C260, C261, C262, C263, C264, C265, C266, C267, C268, C269, C270, C271, C272, C273, C274, C275, C276, C277, C278, C279, C280, C281, C282, C283, C284, C285, C286, C287, C288, C289, C290, C291, C292, C293, C294, C295, C296, C297, C298, C299, C300, C301, C302, C303, C304, C305, C306, C307, C308, C309, C310, C311, C312, C313, C314, C315, C316, C317, C318, C319, C320, C321, C322, C323, C324, C325, C326, C327, C328, C329, C330, C331, C332, C333, C334, C335, C336: 0.1uF, Capacitor_SMD:C_0402_1005Metric, symbol Device:C
- added R, R3, R4, R5: 240Ω, Resistor_SMD:R_0402_1005Metric, symbol Device:R
- added R107, R108: 1kΩ, Resistor_SMD:R_0402_1005Metric, symbol Device:R
- added U_RAM, U_RAM2, U_RAM3, U_RAM4: MT40A512M16LY-075:E, Devboard_Footprints:FBGA-96_L13.5-W7.5-R16-C6-P0.80-TL, symbol Devboard_Custom:MT40A512M16LY-075_E
Connections:
- new net: R.1, U_RAM.F9 (ZQ)
- new net: R5.1, U_RAM4.F9 (ZQ)
- new net: R4.1, U_RAM3.F9 (ZQ)
- new net: R3.1, U_RAM2.F9 (ZQ)
- new net +1V2: C248.2, C249.2, C250.2, C251.2, C252.2, C253.2, C254.2, C255.2, C256.2, C257.2, C258.1, C259.1, C260.1, C261.1, C262.1, C263.1, C264.1, C265.1, C266.1, C267.1, C268.2, C269.2, C270.2, C271.2, C272.2, C273.2, C274.2, C275.2, C276.2, C277.2, C278.1, C279.1, C280.1, C281.1, C282.1, C283.1, C284.1, C285.1, C286.1, C287.1, C288.2, C289.1, C290.2, C291.1, C292.2, C293.1, C294.2, C295.1, C296.2, C297.1, C298.2, C299.1, C300.2, C301.1, C302.2, C303.1, C304.2, C305.1, C306.2, C307.1, C308.2, C309.1, C310.2, C311.1, C312.2, C313.1, C314.2, C315.1, C316.2, C317.1, C318.2, C319.1, C320.2, C321.1, C322.2, C323.1, C324.2, C325.1, C326.2, C327.1, R107.2, U_RAM.A1 (VDDQ), U_RAM.A9 (VDDQ), U_RAM.B3 (VDD), U_RAM.B9 (VDD), U_RAM.C1 (VDDQ), U_RAM.D1 (VDD), U_RAM.D9 (VDDQ), U_RAM.F2 (VDDQ), U_RAM.F8 (VDDQ), U_RAM.G1 (VDDQ), U_RAM.G7 (VDD), U_RAM.G9 (VDDQ), U_RAM.J1 (VDD), U_RAM.J2 (VDDQ), U_RAM.J8 (VDDQ), U_RAM.J9 (VDD), U_RAM.L1 (VDD), U_RAM.L9 (VDD), U_RAM.R1 (VDD), U_RAM.T9 (VDD), U_RAM2.A1 (VDDQ), U_RAM2.A9 (VDDQ), U_RAM2.B3 (VDD), U_RAM2.B9 (VDD), U_RAM2.C1 (VDDQ), U_RAM2.D1 (VDD), U_RAM2.D9 (VDDQ), U_RAM2.F2 (VDDQ), U_RAM2.F8 (VDDQ), U_RAM2.G1 (VDDQ), U_RAM2.G7 (VDD), U_RAM2.G9 (VDDQ), U_RAM2.J1 (VDD), U_RAM2.J2 (VDDQ), U_RAM2.J8 (VDDQ), U_RAM2.J9 (VDD), U_RAM2.L1 (VDD), U_RAM2.L9 (VDD), U_RAM2.R1 (VDD), U_RAM2.T9 (VDD), U_RAM3.A1 (VDDQ), U_RAM3.A9 (VDDQ), U_RAM3.B3 (VDD), U_RAM3.B9 (VDD), U_RAM3.C1 (VDDQ), U_RAM3.D1 (VDD), U_RAM3.D9 (VDDQ), U_RAM3.F2 (VDDQ), U_RAM3.F8 (VDDQ), U_RAM3.G1 (VDDQ), U_RAM3.G7 (VDD), U_RAM3.G9 (VDDQ), U_RAM3.J1 (VDD), U_RAM3.J2 (VDDQ), U_RAM3.J8 (VDDQ), U_RAM3.J9 (VDD), U_RAM3.L1 (VDD), U_RAM3.L9 (VDD), U_RAM3.R1 (VDD), U_RAM3.T9 (VDD), U_RAM4.A1 (VDDQ), U_RAM4.A9 (VDDQ), U_RAM4.B3 (VDD), U_RAM4.B9 (VDD), U_RAM4.C1 (VDDQ), U_RAM4.D1 (VDD), U_RAM4.D9 (VDDQ), U_RAM4.F2 (VDDQ), U_RAM4.F8 (VDDQ), U_RAM4.G1 (VDDQ), U_RAM4.G7 (VDD), U_RAM4.G9 (VDDQ), U_RAM4.J1 (VDD), U_RAM4.J2 (VDDQ), U_RAM4.J8 (VDDQ), U_RAM4.J9 (VDD), U_RAM4.L1 (VDD), U_RAM4.L9 (VDD), U_RAM4.R1 (VDD), U_RAM4.T9 (VDD)
- new net +2V5: C328.2, C329.1, C330.2, C331.1, C332.2, C333.1, C334.2, C335.1, U_RAM.B1 (VPP), U_RAM.R9 (VPP), U_RAM2.B1 (VPP), U_RAM2.R9 (VPP), U_RAM3.B1 (VPP), U_RAM3.R9 (VPP), U_RAM4.B1 (VPP), U_RAM4.R9 (VPP)
- new net GND: C248.1, C249.1, C250.1, C251.1, C252.1, C253.1, C254.1, C255.1, C256.1, C257.1, C258.2, C259.2, C260.2, C261.2, C262.2, C263.2, C264.2, C265.2, C266.2, C267.2, C268.1, C269.1, C270.1, C271.1, C272.1, C273.1, C274.1, C275.1, C276.1, C277.1, C278.2, C279.2, C280.2, C281.2, C282.2, C283.2, C284.2, C285.2, C286.2, C287.2, C288.1, C289.2, C290.1, C291.2, C292.1, C293.2, C294.1, C295.2, C296.1, C297.2, C298.1, C299.2, C300.1, C301.2, C302.1, C303.2, C304.1, C305.2, C306.1, C307.2, C308.1, C309.2, C310.1, C311.2, C312.1, C313.2, C314.1, C315.2, C316.1, C317.2, C318.1, C319.2, C320.1, C321.2, C322.1, C323.2, C324.1, C325.2, C326.1, C327.2, C328.1, C329.2, C330.1, C331.2, C332.1, C333.2, C334.1, C335.2, C336.2, R.2, R108.2, R3.2, R4.2, R5.2, U_RAM.A2 (VSSQ), U_RAM.A8 (VSSQ), U_RAM.B2 (VSS), U_RAM.C9 (VSSQ), U_RAM.D2 (VSSQ), U_RAM.D8 (VSSQ), U_RAM.E1 (VSS), U_RAM.E3 (VSSQ), U_RAM.E8 (VSSQ), U_RAM.E9 (VSS), U_RAM.F1 (VSSQ), U_RAM.G8 (VSS), U_RAM.H1 (VSSQ), U_RAM.H9 (VSSQ), U_RAM.K1 (VSS), U_RAM.K9 (VSS), U_RAM.M9 (VSS), U_RAM.N1 (VSS), U_RAM.T1 (VSS), U_RAM2.A2 (VSSQ), U_RAM2.A8 (VSSQ), U_RAM2.B2 (VSS), U_RAM2.C9 (VSSQ), U_RAM2.D2 (VSSQ), U_RAM2.D8 (VSSQ), U_RAM2.E1 (VSS), U_RAM2.E3 (VSSQ), U_RAM2.E8 (VSSQ), U_RAM2.E9 (VSS), U_RAM2.F1 (VSSQ), U_RAM2.G8 (VSS), U_RAM2.H1 (VSSQ), U_RAM2.H9 (VSSQ), U_RAM2.K1 (VSS), U_RAM2.K9 (VSS), U_RAM2.M9 (VSS), U_RAM2.N1 (VSS), U_RAM2.T1 (VSS), U_RAM3.A2 (VSSQ), U_RAM3.A8 (VSSQ), U_RAM3.B2 (VSS), U_RAM3.C9 (VSSQ), U_RAM3.D2 (VSSQ), U_RAM3.D8 (VSSQ), U_RAM3.E1 (VSS), U_RAM3.E3 (VSSQ), U_RAM3.E8 (VSSQ), U_RAM3.E9 (VSS), U_RAM3.F1 (VSSQ), U_RAM3.G8 (VSS), U_RAM3.H1 (VSSQ), U_RAM3.H9 (VSSQ), U_RAM3.K1 (VSS), U_RAM3.K9 (VSS), U_RAM3.M9 (VSS), U_RAM3.N1 (VSS), U_RAM3.T1 (VSS), U_RAM4.A2 (VSSQ), U_RAM4.A8 (VSSQ), U_RAM4.B2 (VSS), U_RAM4.C9 (VSSQ), U_RAM4.D2 (VSSQ), U_RAM4.D8 (VSSQ), U_RAM4.E1 (VSS), U_RAM4.E3 (VSSQ), U_RAM4.E8 (VSSQ), U_RAM4.E9 (VSS), U_RAM4.F1 (VSSQ), U_RAM4.G8 (VSS), U_RAM4.H1 (VSSQ), U_RAM4.H9 (VSSQ), U_RAM4.K1 (VSS), U_RAM4.K9 (VSS), U_RAM4.M9 (VSS), U_RAM4.N1 (VSS), U_RAM4.T1 (VSS)
- new net PS_DDR_A0: U_RAM.P3 (A0), U_RAM2.P3 (A0), U_RAM3.P3 (A0), U_RAM4.P3 (A0)
- new net PS_DDR_A1: U_RAM.P7 (A1), U_RAM2.P7 (A1), U_RAM3.P7 (A1), U_RAM4.P7 (A1)
- new net PS_DDR_A10: U_RAM.M3 (A10/AP), U_RAM2.M3 (A10/AP), U_RAM3.M3 (A10/AP), U_RAM4.M3 (A10/AP)
- new net PS_DDR_A11: U_RAM.T2 (A11), U_RAM2.T2 (A11), U_RAM3.T2 (A11), U_RAM4.T2 (A11)
- new net PS_DDR_A12: U_RAM.M7 (A12/BC_n), U_RAM2.M7 (A12/BC_n), U_RAM3.M7 (A12/BC_n), U_RAM4.M7 (A12/BC_n)
- new net PS_DDR_A13: U_RAM.T8 (A13), U_RAM2.T8 (A13), U_RAM3.T8 (A13), U_RAM4.T8 (A13)
- new net PS_DDR_A14: U_RAM.L2 (WE_n/A14), U_RAM2.L2 (WE_n/A14), U_RAM3.L2 (WE_n/A14), U_RAM4.L2 (WE_n/A14)
- new net PS_DDR_A15: U_RAM.M8 (CAS-n/A15), U_RAM2.M8 (CAS-n/A15), U_RAM3.M8 (CAS-n/A15), U_RAM4.M8 (CAS-n/A15)
- new net PS_DDR_A16: U_RAM.L8 (RAS_n/A16), U_RAM2.L8 (RAS_n/A16), U_RAM3.L8 (RAS_n/A16), U_RAM4.L8 (RAS_n/A16)
- new net PS_DDR_A2: U_RAM.R3 (A2), U_RAM2.R3 (A2), U_RAM3.R3 (A2), U_RAM4.R3 (A2)
- new net PS_DDR_A3: U_RAM.N7 (A3), U_RAM2.N7 (A3), U_RAM3.N7 (A3), U_RAM4.N7 (A3)
- new net PS_DDR_A4: U_RAM.N3 (A4), U_RAM2.N3 (A4), U_RAM3.N3 (A4), U_RAM4.N3 (A4)
- new net PS_DDR_A5: U_RAM.P8 (A5), U_RAM2.P8 (A5), U_RAM3.P8 (A5), U_RAM4.P8 (A5)
- new net PS_DDR_A6: U_RAM.P2 (A6), U_RAM2.P2 (A6), U_RAM3.P2 (A6), U_RAM4.P2 (A6)
- new net PS_DDR_A7: U_RAM.R8 (A7), U_RAM2.R8 (A7), U_RAM3.R8 (A7), U_RAM4.R8 (A7)
- new net PS_DDR_A8: U_RAM.R2 (A8), U_RAM2.R2 (A8), U_RAM3.R2 (A8), U_RAM4.R2 (A8)
- new net PS_DDR_A9: U_RAM.R7 (A9), U_RAM2.R7 (A9), U_RAM3.R7 (A9), U_RAM4.R7 (A9)
- new net PS_DDR_ACT_N: U_RAM.L3 (ACT_n), U_RAM2.L3 (ACT_n), U_RAM3.L3 (ACT_n), U_RAM4.L3 (ACT_n)
- new net PS_DDR_ALERT_N: U_RAM.P9 (ALERT_n), U_RAM2.P9 (ALERT_n), U_RAM3.P9 (ALERT_n), U_RAM4.P9 (ALERT_n)
- new net PS_DDR_BA0: U_RAM.N2 (BA0), U_RAM2.N2 (BA0), U_RAM3.N2 (BA0), U_RAM4.N2 (BA0)
- new net PS_DDR_BA1: U_RAM.N8 (BA1), U_RAM2.N8 (BA1), U_RAM3.N8 (BA1), U_RAM4.N8 (BA1)
- new net PS_DDR_BG0: U_RAM.M2 (BG0), U_RAM2.M2 (BG0), U_RAM3.M2 (BG0), U_RAM4.M2 (BG0)
- new net PS_DDR_CK0: U_RAM.K7 (CK_t), U_RAM2.K7 (CK_t), U_RAM3.K7 (CK_t), U_RAM4.K7 (CK_t)
- new net PS_DDR_CKE0: U_RAM.K2 (CKE), U_RAM2.K2 (CKE), U_RAM3.K2 (CKE), U_RAM4.K2 (CKE)
- new net PS_DDR_CK_N0: U_RAM.K8 (CK_c), U_RAM2.K8 (CK_c), U_RAM3.K8 (CK_c), U_RAM4.K8 (CK_c)
- new net PS_DDR_CS_N0: U_RAM.L7 (CS_n), U_RAM2.L7 (CS_n), U_RAM3.L7 (CS_n), U_RAM4.L7 (CS_n)
- new net PS_DDR_DM0: U_RAM.E7 (NF/LDM_n/LDBI_n)
- new net PS_DDR_DM1: U_RAM.E2 (NF/UDM_n/UDBI_n)
- new net PS_DDR_DM2: U_RAM2.E7 (NF/LDM_n/LDBI_n)
- new net PS_DDR_DM3: U_RAM2.E2 (NF/UDM_n/UDBI_n)
- new net PS_DDR_DM4: U_RAM3.E7 (NF/LDM_n/LDBI_n)
- new net PS_DDR_DM5: U_RAM3.E2 (NF/UDM_n/UDBI_n)
- new net PS_DDR_DM6: U_RAM4.E7 (NF/LDM_n/LDBI_n)
- new net PS_DDR_DM7: U_RAM4.E2 (NF/UDM_n/UDBI_n)
- new net PS_DDR_DQ0: U_RAM.G2 (DQ0)
- new net PS_DDR_DQ1: U_RAM.F7 (DQ1)
- new net PS_DDR_DQ10: U_RAM.C3 (DQ10)
- new net PS_DDR_DQ11: U_RAM.C7 (DQ11)
- new net PS_DDR_DQ12: U_RAM.C2 (DQ12)
- new net PS_DDR_DQ13: U_RAM.C8 (DQ13)
- new net PS_DDR_DQ14: U_RAM.D3 (DQ14)
- new net PS_DDR_DQ15: U_RAM.D7 (DQ15)
- new net PS_DDR_DQ16: U_RAM2.G2 (DQ0)
- new net PS_DDR_DQ17: U_RAM2.F7 (DQ1)
- new net PS_DDR_DQ18: U_RAM2.H3 (DQ2)
- new net PS_DDR_DQ19: U_RAM2.H7 (DQ3)
- new net PS_DDR_DQ2: U_RAM.H3 (DQ2)
- new net PS_DDR_DQ20: U_RAM2.H2 (DQ4)
- new net PS_DDR_DQ21: U_RAM2.H8 (DQ5)
- new net PS_DDR_DQ22: U_RAM2.J3 (DQ6)
- new net PS_DDR_DQ23: U_RAM2.J7 (DQ7)
- new net PS_DDR_DQ24: U_RAM2.A3 (DQ8)
- new net PS_DDR_DQ25: U_RAM2.B8 (DQ9)
- new net PS_DDR_DQ26: U_RAM2.C3 (DQ10)
- new net PS_DDR_DQ27: U_RAM2.C7 (DQ11)
- new net PS_DDR_DQ28: U_RAM2.C2 (DQ12)
- new net PS_DDR_DQ29: U_RAM2.C8 (DQ13)
- new net PS_DDR_DQ3: U_RAM.H7 (DQ3)
- new net PS_DDR_DQ30: U_RAM2.D3 (DQ14)
- new net PS_DDR_DQ31: U_RAM2.D7 (DQ15)
- new net PS_DDR_DQ32: U_RAM3.G2 (DQ0)
- new net PS_DDR_DQ33: U_RAM3.F7 (DQ1)
- new net PS_DDR_DQ34: U_RAM3.H3 (DQ2)
- new net PS_DDR_DQ35: U_RAM3.H7 (DQ3)
- new net PS_DDR_DQ36: U_RAM3.H2 (DQ4)
- new net PS_DDR_DQ37: U_RAM3.H8 (DQ5)
- new net PS_DDR_DQ38: U_RAM3.J3 (DQ6)
- new net PS_DDR_DQ39: U_RAM3.J7 (DQ7)
- new net PS_DDR_DQ4: U_RAM.H2 (DQ4)
- new net PS_DDR_DQ40: U_RAM3.A3 (DQ8)
- new net PS_DDR_DQ41: U_RAM3.B8 (DQ9)
- new net PS_DDR_DQ42: U_RAM3.C3 (DQ10)
- new net PS_DDR_DQ43: U_RAM3.C7 (DQ11)
- new net PS_DDR_DQ44: U_RAM3.C2 (DQ12)
- new net PS_DDR_DQ45: U_RAM3.C8 (DQ13)
- new net PS_DDR_DQ46: U_RAM3.D3 (DQ14)
- new net PS_DDR_DQ47: U_RAM3.D7 (DQ15)
- new net PS_DDR_DQ48: U_RAM4.G2 (DQ0)
- new net PS_DDR_DQ49: U_RAM4.F7 (DQ1)
- new net PS_DDR_DQ5: U_RAM.H8 (DQ5)
- new net PS_DDR_DQ50: U_RAM4.H3 (DQ2)
- new net PS_DDR_DQ51: U_RAM4.H7 (DQ3)
- new net PS_DDR_DQ52: U_RAM4.H2 (DQ4)
- new net PS_DDR_DQ53: U_RAM4.H8 (DQ5)
- new net PS_DDR_DQ54: U_RAM4.J3 (DQ6)
- new net PS_DDR_DQ55: U_RAM4.J7 (DQ7)
- new net PS_DDR_DQ56: U_RAM4.A3 (DQ8)
- new net PS_DDR_DQ57: U_RAM4.B8 (DQ9)
- new net PS_DDR_DQ58: U_RAM4.C3 (DQ10)
- new net PS_DDR_DQ59: U_RAM4.C7 (DQ11)
- new net PS_DDR_DQ6: U_RAM.J3 (DQ6)
- new net PS_DDR_DQ60: U_RAM4.C2 (DQ12)
- new net PS_DDR_DQ61: U_RAM4.C8 (DQ13)
- new net PS_DDR_DQ62: U_RAM4.D3 (DQ14)
- new net PS_DDR_DQ63: U_RAM4.D7 (DQ15)
- new net PS_DDR_DQ7: U_RAM.J7 (DQ7)
- new net PS_DDR_DQ8: U_RAM.A3 (DQ8)
- new net PS_DDR_DQ9: U_RAM.B8 (DQ9)
- new net PS_DDR_DQS_N0: U_RAM.F3 (LDQS_c)
- new net PS_DDR_DQS_N1: U_RAM.A7 (UDQS_c)
- new net PS_DDR_DQS_N2: U_RAM2.F3 (LDQS_c)
- new net PS_DDR_DQS_N3: U_RAM2.A7 (UDQS_c)
- new net PS_DDR_DQS_N4: U_RAM3.A7 (UDQS_c)
- new net PS_DDR_DQS_N5: U_RAM3.F3 (LDQS_c)
- new net PS_DDR_DQS_N6: U_RAM4.F3 (LDQS_c)
- new net PS_DDR_DQS_N7: U_RAM4.B7 (UDQS_t)
- new net PS_DDR_DQS_P0: U_RAM.G3 (LDQS_t)
- new net PS_DDR_DQS_P1: U_RAM.B7 (UDQS_t)
- new net PS_DDR_DQS_P2: U_RAM2.G3 (LDQS_t)
- new net PS_DDR_DQS_P3: U_RAM2.B7 (UDQS_t)
- new net PS_DDR_DQS_P4: U_RAM3.G3 (LDQS_t)
- new net PS_DDR_DQS_P5: U_RAM3.B7 (UDQS_t)
- new net PS_DDR_DQS_P6: U_RAM4.G3 (LDQS_t)
- new net PS_DDR_DQS_P7: U_RAM4.A7 (UDQS_c)
- new net PS_DDR_ODT0: U_RAM.K3 (ODT), U_RAM2.K3 (ODT), U_RAM3.K3 (ODT), U_RAM4.K3 (ODT)
- new net PS_DDR_PARITY: U_RAM.T3 (PAR), U_RAM2.T3 (PAR), U_RAM3.T3 (PAR), U_RAM4.T3 (PAR)
- new net PS_DDR_RAM_RST_N: U_RAM.P1 (RESET_n), U_RAM2.P1 (RESET_n), U_RAM3.P1 (RESET_n), U_RAM4.P1 (RESET_n)
- new net VREFCA_DDR4: C336.1, R107.1, R108.1, U_RAM.M1 (VREFCA), U_RAM2.M1 (VREFCA), U_RAM3.M1 (VREFCA), U_RAM4.M1 (VREFCA)
- no-connect marks 0 -> 8
Other:
- note added: "DECOUPLING CAPACITORS"
- note added: "SECTION 04b : DDR4"
- note added: "VDD"
- note added: "VDDQ"
- note added: "VPP"

Commit message: Feat: Zynq Peripherals added
Parts:
- renumbered R to R109, U_RAM to U_RAM5

Commit message: Feat : Completed 04d Peripherals
Changed lines of the file:
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@@
 	(generator "eeschema")
 	(generator_version "10.0")
-	(paper "User" 594 420)
+	(paper "User" 841 800)
 	(rectangle
 		(start 118.745 150.495)
@@
 		)
 		(stroke
+			(width 0)
+			(type default)
+		)
+	)
+	(wire
+		(pts
+			(xy 1008.38 580.39) (xy 1014.73 580.39)
+		)
+		(stroke

Commit message: Feat : Schematics Complete
Parts:
- renumbered C328 to C252, C330 to C253, C332 to C254, C334 to C255, C248 to C256, C249 to C257, C250 to C258, C251 to C259, C252 to C260, C253 to C261, C254 to C262, C255 to C263, C256 to C264, C257 to C265, C288 to C266, C292 to C267, C296 to C268, C300 to C269, C304 to C270, C308 to C271, C312 to C272, C316 to C273, C320 to C274, C324 to C275, C329 to C276, C331 to C277, C333 to C278, C335 to C279, C258 to C280, C259 to C281, C260 to C282, C261 to C283, C262 to C284, C263 to C285, C264 to C286, C265 to C287, C266 to C288, C267 to C289, C289 to C290, C293 to C291, C297 to C292, C301 to C293, C305 to C294, C309 to C295, C313 to C296, C317 to C297, C321 to C298, C325 to C299, C268 to C300, C269 to C301, C270 to C302, C271 to C303, C272 to C304, C273 to C305, C274 to C306, C275 to C307, C276 to C308, C277 to C309, C290 to C310, C294 to C311, C298 to C312, C302 to C313, C306 to C314, C310 to C315, C314 to C316, C318 to C317, C322 to C318, C326 to C319, C278 to C320, C279 to C321, C280 to C322, C281 to C323, C282 to C324, C283 to C325, C284 to C326, C285 to C327, C286 to C328, C287 to C329, C291 to C330, C295 to C331, C299 to C332, C303 to C333, C307 to C334, C311 to C335, C315 to C336, C319 to C337, C323 to C338, C327 to C339, C336 to C340, R107 to R104, R108 to R105, R109 to R106, R3 to R107, R4 to R108, R5 to R109, U_RAM5 to U_RAM1
