File: PCB/schematics/04_Zynq/04c_Zynq_PS_Perhipherals.kicad_sch (KiCad schematic)
At the start: 0 parts

Commit message: Feat: Zynq Peripherals added
Parts:
- added C337, C338, C340, C342, C344, C346, C347, C350, C351, C354, C357, C358, C359, C361, C362, C363, C367, C369, C371, C373, C377, C378: 0.1uF, Capacitor_SMD:C_0402_1005Metric, symbol Device:C
- added C339, C341, C343, C345, C348, C349, C352, C353, C355, C356, C360: 1uF, Capacitor_SMD:C_0402_1005Metric, symbol Device:C
- added C364, C365, C366, C368, C370, C372, C374: 1nF, Capacitor_SMD:C_0402_1005Metric, symbol Device:C
- added C375, C376: 22uF, Capacitor_SMD:C_0402_1005Metric, symbol Device:C
- added Card1: TF-01A, Devboard_Footprints:TF-SMD_TF-01A, symbol Devboard_Custom:TF-01A
- added J1: HR911105A_C12074, Devboard_Footprints:RJ45-TH_HR911105A, symbol Devboard_Custom:HR911105A_C12074
- added R110, R111, R112, R113, R114, R115, R118, R119, R120, R121, R122, R131, R132, R134: 10kΩ, Resistor_SMD:R_0402_1005Metric, symbol Device:R
- added R116, R117, R123, R124, R125, R126, R127, R128, R129, R130, R2: 22Ω, Resistor_SMD:R_0402_1005Metric, symbol Device:R
- added R133, R135: 2.49kΩ, Resistor_SMD:R_0402_1005Metric, symbol Device:R
- added R136: 11kΩ, Resistor_SMD:R_0402_1005Metric, symbol Device:R
- added R137, R138: 470Ω, Resistor_SMD:R_0402_1005Metric, symbol Device:R
- added U28: MT25QU256ABA8ESF-0SIT TR, Devboard_Footprints:SOP-16_L10.3-W7.5-P1.27-LS10.4-BL, symbol Devboard_Custom:MT25QU256ABA8ESF-0SITTR
- added U29: FEMDNN032G-A3A55, Devboard_Footprints:FBGA-153_L13.0-W11.5-P0.50_KLMAG1JETD-B041, symbol Devboard_Custom:FEMDNN032G-A3A55
- added U30: TXS02612RTWR, Devboard_Footprints:WQFN-24_L4.0-W4.0-P0.50-TL-EP2.5, symbol Devboard_Custom:TXS02612RTWR
- added U31: DP83867IRRGZR, Devboard_Footprints:VQFN-48_L7.0-W7.0-P0.50-TL-EP4.1, symbol Devboard_Custom:DP83867IRRGZR
- added U32: USB3320C-EZK-TR, Connector_USB:USB3_A_Plug_Wuerth_692112030100_Horizontal, symbol Devboard_Custom:USB3320C-EZK-TR
- added U34: CP2102N-Axx-xQFN24, Package_DFN_QFN:QFN-24-1EP_4x4mm_P0.5mm_EP2.6x2.6mm, symbol Interface_USB:CP2102N-Axx-xQFN24
- added U35: TXB0108PW, Package_SO:TSSOP-20_4.4x6.5mm_P0.65mm, symbol Logic_LevelTranslator:TXB0108PW
- added U36: TCA9548APWR, Package_SO:TSSOP-24_4.4x7.8mm_P0.65mm, symbol Interface_Expansion:TCA9548APWR
- added U37: PCA9306, Package_SO:VSSOP-8_2.3x2mm_P0.5mm, symbol Interface:PCA9306
- added U38: TPD4E05U06DQA, Package_SON:USON-10_2.5x1.0mm_P0.5mm, symbol Power_Protection:TPD4E05U06DQA
- added USB2: TYPE-C-24P-SMD, easyeda2kicad:USB-C-SMD_TYPE-C-24P-SMD, symbol Devboard_Custom:TYPE-C-24P-SMD
- added Y1: 25 MHz, Crystal:Crystal_SMD_3225-4Pin_3.2x2.5mm, symbol Device:Crystal_GND24
Connections:
- new net: R129.1, U31.34 (RX_D1)
- new net: C378.2, J1.5
- new net: C375.2, U31.14 (X_O), Y1.3
- new net: R136.2, U31.12 (RBIAS)
- new net: C376.2, U31.15 (X_I), Y1.1
- new net: R126.1, U31.25 (TX_D3)
- new net: R125.1, U31.26 (TX_D2)
- new net: R124.1, U31.27 (TX_D1)
- new net: R123.1, U31.28 (TX_D0)
- new net: R130.1, U31.33 (RX_D0)
- new net: R128.1, U31.35 (RX_D2)
- new net: R127.1, U31.36 (RX_D3)
- new net: U38.3 (GND), U38.8 (GND)
- new net: R113.2, U28.3 (~{RESET})
- new net: U34.2 (GND), U34.25 (GND)
- new net: R117.1, U30.19 (CLKB0)
- new net: R2.1, U28.16 (C)
- new net: J1.9, R137.1
- new net: C377.2, J1.4
- new net: R116.1, U29.M6 (CLK)
- new net: C356.2, U29.C2 (VDDI)
- new net: J1.12, R138.1
- new net: Card1.5 (CLK(SCLK)), R117.2
- new net +1V2: C367.2, C368.1, C369.2, C370.1, C371.2, C372.1, C373.2, C374.1, U31.24 (VDD1P0), U31.31 (VDD1P0), U31.42 (VDD1P0), U31.6 (VDD1P0)
- new net +1V8: C337.1, C357.1, C361.2, C362.2, C363.2, C364.1, C365.1, C366.1, R110.1, R111.1, R112.1, R113.1, R114.1, R115.1, R131.1, R132.1, R134.1, U28.2 (VCC), U29.C6 (VCCQ), U29.M4 (VCCQ), U29.N4 (VCCQ), U29.P3 (VCCQ), U29.P5 (VCCQ), U30.5 (VCCA), U31.19 (VDDIO), U31.30 (VDDIO), U31.41 (VDDIO)
- new net +3V3: C338.2, C339.2, C340.2, C341.2, C342.2, C343.2, C344.2, C345.2, C346.2, C347.2, C348.2, C349.2, C350.2, C351.2, C352.2, C353.2, C354.2, C355.2, C358.2, C359.2, C360.1, Card1.4 (VDD), R118.1, R119.1, R120.1, R121.1, R122.1, U29.E6 (VCC), U29.F5 (VCC), U29.J10 (VCC), U29.K9 (VCC), U30.17 (VCCB1), U30.21 (VCCB0)
- new net CMDB0: Card1.3 (CMD(DI)), R118.2, U30.20 (CMDB0)
- new net DAT0B0: Card1.7 (DAT0(D0)), R119.2, U30.18 (DAT0B0)
- new net DAT1B0: Card1.8 (DAT1(RSV)), R120.2, U30.16 (DAT1B0)
- new net DAT2B0: Card1.1 (DAT2(RSV)), R121.2, U30.23 (DAT2B0)
- new net DAT3B0: Card1.2 (CDDAT3(CS)), R122.2, U30.22 (DAT3B0)
- new net GEM_RST: U31.43 (RESET_N)
- new net GEM_RXC: U31.32 (RX_CLK)
- new net GEM_RXD0: R127.2, R132.2, R133.2
- new net GEM_RXD1: R128.2, R134.2, R135.2
- new net GEM_RXD2: R129.2
- new net GEM_RXD3: R130.2
- new net GEM_RX_CTL: U31.38 (RX_CTRL)
- new net GEM_TXC: U31.29 (GTX_CLK)
- new net GEM_TXD0: R123.2
- new net GEM_TXD1: R124.2
- new net GEM_TXD2: R125.2
- new net GEM_TXD3: R126.2
- new net GEM_TX_CTL: U31.37 (TX_CTRL)
- new net GND: C337.2, C338.1, C339.1, C340.1, C341.1, C342.1, C343.1, C344.1, C345.1, C346.1, C347.1, C348.1, C349.1, C350.1, C351.1, C352.1, C353.1, C354.1, C355.1, C356.1, C357.2, C358.1, C359.1, C360.2, C361.1, C362.1, C363.1, C364.2, C365.2, C366.2, C367.1, C368.2, C369.1, C370.2, C371.1, C372.2, C373.1, C374.2, C375.1, C376.1, C377.1, C378.1, Card1.10 (GND), Card1.11 (GND), Card1.12 (GND), Card1.13 (GND), Card1.6 (VSS), J1.10, J1.11, J1.8 (CHSGND), J1.SH1, J1.SH2, R133.1, R135.1, R136.1, U28.10 (VSS), U29.A6 (VSS), U29.C4 (VSSQ), U29.E7 (VSS), U29.G5 (VSS), U29.H10 (VSS), U29.J5 (VSS), U29.K8 (VSS), U29.N2 (VSSQ), U29.N5 (VSSQ), U29.P4 (VSSQ), U30.11 (GND), U30.2 (GND), U30.24 (SEL), U30.25 (EP), U31.49 (GND), Y1.2 (G), Y1.4 (G)
- new net LED_0: R137.2, U31.47 (LED_0)
- new net LED_1: R138.2, U31.46 (LED_1)
- new net MDIO_MDC: U31.16 (MDC)
- new net MDIO_MDIO: R131.2, U31.17 (MDIO)
- new net QSPI_IO0: U28.15 (DQ0)
- new net QSPI_IO1: U28.8 (DQ1)
- new net QSPI_IO2: R110.2, U28.9 (~{W}/DQ2)
- new net QSPI_IO3: R111.2, U28.1 (DQ3/~{HOLD})
- new net QSPI_SCLK: R2.2
- new net QSPI_SS: R112.2, U28.7 (~{S})
- new net SD0_CLK: R116.2
- new net SD0_CMD: R115.2, U29.M5 (CMD)
- new net SD0_D0: R114.2, U29.A3 (DAT0)
- new net SD0_D1: U29.A4 (DAT1)
- new net SD0_D2: U29.A5 (DAT2)
- new net SD0_D3: U29.B2 (DAT3)
- new net SD0_D4: U29.B3 (DAT4)
- new net SD0_D5: U29.B4 (DAT5)
- new net SD0_D6: U29.B5 (DAT6)
- new net SD0_D7: U29.B6 (DAT7)
- new net SD0_RST: U29.K5 (RSTN)
- new net SD1_CD: Card1.9 (CD)
- new net SD1_CLK: U30.9 (CLKA)
- new net SD1_CMD: U30.4 (CMDA)
- new net SD1_D0: U30.6 (DAT0A)
- new net SD1_D1: U30.7 (DAT1A)
- new net SD1_D2: U30.1 (DAT2A)
- new net SD1_D3: U30.3 (DAT3A)
- new net TD_M_A: J1.1 (TD+), U31.2 (TD_M_A)
- new net TD_P_A: J1.2 (TD-), U31.1 (TD_P_A)
- new net TD_P_B: J1.3 (RD+), J1.6 (RD-), U31.4 (TD_P_B), U31.5 (TD_M_B)
- no-connect marks 0 -> 159
Other:
- note added: "Ethernet"
- note added: "PULL-UPS"
- note added: "QSPIO"
- note added: "SD CARD"
- note added: "VCC"
- note added: "VCCA"
- note added: "VCCB0+B1"
- note added: "VDD1P0"
- note added: "VDDIO"
- note added: "eMMC"

Commit message: Feat : Completed 04d Peripherals
Parts:
- removed U38: TPD4E05U06DQA, Package_SON:USON-10_2.5x1.0mm_P0.5mm, symbol Power_Protection:TPD4E05U06DQA
- added C379, C380: 33pF, Capacitor_SMD:C_0402_1005Metric, symbol Device:C
- added C381, C382, C383, C384, C385, C386, C388, C389, C390, C391, C392: 0.1uF, Capacitor_SMD:C_0402_1005Metric, symbol Device:C
- added C387: 1uF, Capacitor_SMD:C_0402_1005Metric, symbol Device:C
- added J10: I2C_7, Connector_PinHeader_2.54mm:PinHeader_1x02_P2.54mm_Vertical, symbol Connector:Conn_01x02_Pin
- added J11: 3.3V_I2C, Connector_PinHeader_2.54mm:PinHeader_1x02_P2.54mm_Vertical, symbol Connector:Conn_01x02_Pin
- added J17: I2C_0, Connector_PinHeader_2.54mm:PinHeader_1x02_P2.54mm_Vertical, symbol Connector:Conn_01x02_Pin
- added J2: USB3_B, Connector_JST:JST_SH_BM09B-SRSS-TB_1x09-1MP_P1.00mm_Vertical, symbol Connector:USB3_B
- added J4: I2C_1, Connector_PinHeader_2.54mm:PinHeader_1x02_P2.54mm_Vertical, symbol Connector:Conn_01x02_Pin
- added J5: I2C_2, Connector_PinHeader_2.54mm:PinHeader_1x02_P2.54mm_Vertical, symbol Connector:Conn_01x02_Pin
- added J6: I2C_3, Connector_PinHeader_2.54mm:PinHeader_1x02_P2.54mm_Vertical, symbol Connector:Conn_01x02_Pin
- added J7: I2C_4, Connector_PinHeader_2.54mm:PinHeader_1x02_P2.54mm_Vertical, symbol Connector:Conn_01x02_Pin
- added J8: I2C_5, Connector_PinHeader_2.54mm:PinHeader_1x02_P2.54mm_Vertical, symbol Connector:Conn_01x02_Pin
- added J9: I2C_6, Connector_PinHeader_2.54mm:PinHeader_1x02_P2.54mm_Vertical, symbol Connector:Conn_01x02_Pin
- added R139, R146: 1kΩ, Resistor_SMD:R_0402_1005Metric, symbol Device:R
- added R140: 8.06kΩ, Resistor_SMD:R_0402_1005Metric, symbol Device:R
- added R141, R149: 10kΩ, Resistor_SMD:R_0402_1005Metric, symbol Device:R
- added R142, R143: 5.1kΩ, Resistor_SMD:R_0402_1005Metric, symbol Device:R
- added R144: 47.5kΩ, Resistor_SMD:R_0402_1005Metric, symbol Device:R
- added R145: 22.1kΩ, Resistor_SMD:R_0402_1005Metric, symbol Device:R
- added R147, R148, R150, R151, R152, R153, R155: 2.2kΩ, Resistor_SMD:R_0402_1005Metric, symbol Device:R
- added R154: 200kΩ, Resistor_SMD:R_0402_1005Metric, symbol Device:R
- added U33: TPD4E05U06DQA, Package_SON:USON-10_2.5x1.0mm_P0.5mm, symbol Power_Protection:TPD4E05U06DQA
- added Y2: 25 MHz, Crystal:Crystal_SMD_3225-4Pin_3.2x2.5mm, symbol Device:Crystal_GND24
- U34: value CP2102N-Axx-xQFN24 -> CP2102N-A02-GQFN24
Connections:
- net +1V8: now also U32.28 (VDD18), U32.30 (VDD18), U32.32 (VDDIO), U34.5 (VIO), U35.2 (V_{CCA}), U36.1 (A0), U36.2 (A1), U36.21 (A2), U36.24 (VCC), U37.2 (VREF1), C381.1, C382.1, C383.1, C386.1, C388.1, C389.1, C391.1, R141.1, R147.1, R148.1, R149.1
- net +3V3: now also U32.21 (VBAT), U34.6 (VDD), U35.19 (V_{CCB}), U37.7 (VREF2), U37.8 (EN), C385.1, C390.1, C392.1, R146.1, R150.1, R151.1, R152.1, R153.1, R154.1, R154.2
- net GND: now also U34.2 (GND), U34.25 (GND), U35.11 (GND), U36.12 (GND), U37.1 (GND), USB2.A1 (GND), USB2.A12 (GND), USB2.B1 (GND), USB2.B12 (GND), C379.1, C380.1, C381.2, C382.2, C383.2, C384.2, C385.2, C386.2, C387.1, C388.2, C389.2, C390.2, C391.2, C392.2, R140.1, R142.2, R143.2, R144.1, R155.2, U33.3 (GND), U33.8 (GND), Y2.2 (G), Y2.4 (G)
- net UART0_RX: now reaches U34.20 (RXD)
- net UART0_TX: now reaches U34.21 (TXD)
- net at U34.3 (D+): now also U33.5 (D2-)
- net at U34.4 (D-): now also U33.4 (D2+)
- net +5V_SYS: now reaches U34.7 (VREGIN)
- net +5V_SYS: now also C387.2
- net at U34.8 (VBUS): now also R144.2, R145.2
- net at U34.9 (~{RST}): now also R146.2
- net I2C1_SCL: now reaches U37.3 (SCL1)
- net I2C1_SCL: now also R152.2
- net I2C1_SDA: now reaches U37.4 (SDA1)
- net I2C1_SDA: now also R153.2
- net at U37.5 (SDA2): now also J11.1 (Pin_1), R151.2
- net at U37.6 (SCL2): now also J11.2 (Pin_2), R150.2
- net VBUS: now reaches USB2.A4 (VBUS)
- net VBUS: now also USB2.A9 (VBUS), USB2.B4 (VBUS), USB2.B9 (VBUS), J2.1 (VBUS), R139.1, R145.1
- net CC1: now reaches USB2.A5 (CC1)
- net CC1: now also R142.1
- net DP1: now reaches USB2.A6 (Dp1)
- net DP1: now also U32.18 (DP), USB2.B6 (Dp2)
- net DN1: now reaches USB2.A7 (Dn1)
- net DN1: now also U32.19 (DM), USB2.B7 (Dn2)
- net CC2: now reaches USB2.B5 (CC2)
- net CC2: now also R143.1
- net at U35.10 (OE): now also R155.1
- net I2C_SDA_3: now reaches U36.10 (SD3)
- net I2C_SDA_3: now also J6.2 (Pin_2)
- net I2C_SCL_3: now reaches U36.11 (SC3)
- net I2C_SCL_3: now also J6.1 (Pin_1)
- net I2C_SDA_4: now reaches U36.13 (SD4)
- net I2C_SDA_4: now also J7.2 (Pin_2)
- net I2C_SCL_4: now reaches U36.14 (SC4)
- net I2C_SCL_4: now also J7.1 (Pin_1)
- net I2C_SDA_5: now reaches U36.15 (SD5)
- net I2C_SDA_5: now also J8.2 (Pin_2)
- net I2C_SCL_5: now reaches U36.16 (SC5)
- net I2C_SCL_5: now also J8.1 (Pin_1)
- net I2C_SDA_6: now reaches U36.17 (SD6)
- net I2C_SDA_6: now also J9.2 (Pin_2)
- net I2C_SCL_6: now reaches U36.18 (SC6)
- net I2C_SCL_6: now also J9.1 (Pin_1)
- net I2C_SDA_7: now reaches U36.19 (SD7)
- net I2C_SDA_7: now also J10.2 (Pin_2)
- net I2C_SCL_7: now reaches U36.20 (SC7)
- net I2C_SCL_7: now also J10.1 (Pin_1)
- net I2C0_SCL: now reaches U36.22 (SCL)
- net I2C0_SDA: now reaches U36.23 (SDA)
- net at U36.3 (~{RESET}): now also R149.2
- net I2C_SDA_0: now reaches U36.4 (SD0)
- net I2C_SDA_0: now also J17.2 (Pin_2), R148.2
- net I2C_SCL_0: now reaches U36.5 (SC0)
- net I2C_SCL_0: now also J17.1 (Pin_1), R147.2
- net I2C_SDA_1: now reaches U36.6 (SD1)
- net I2C_SDA_1: now also J4.2 (Pin_2)
- net I2C_SCL_1: now reaches U36.7 (SC1)
- net I2C_SCL_1: now also J4.1 (Pin_1)
- net I2C_SDA_2: now reaches U36.8 (SD2)
- net I2C_SDA_2: now also J5.2 (Pin_2)
- net I2C_SCL_2: now reaches U36.9 (SC2)
- net I2C_SCL_2: now also J5.1 (Pin_1)
- net USB2_CLK: now reaches U32.1 (CLKOUT)
- net USB2_D6: now reaches U32.10 (DATA6)
- net USB2_D7: now reaches U32.13 (DATA7)
- net USB2_NXT: now reaches U32.2 (NXT)
- net at U32.20 (VDD33): now also C384.1
- net at U32.22 (VBUS): now also R139.2
- net at U32.24 (RBIAS): now also R140.2
- net at U32.25 (XO): now also C380.2, Y2.1
- net at U32.26 (REFCLK): now also C379.2, Y2.3
- net at U32.27 (RESETB): now also R141.2
- net USB2_STP: now reaches U32.29 (STP)
- net USB2_D0: now reaches U32.3 (DATA0)
- net USB2_DIR: now reaches U32.31 (DIR)
- net USB2_D1: now reaches U32.4 (DATA1)
- net USB2_D2: now reaches U32.5 (DATA2)
- net USB2_D3: now reaches U32.6 (DATA3)
- net USB2_D4: now reaches U32.7 (DATA4)
- net USB2_D5: now reaches U32.9 (DATA5)
- new net: J2.2 (D-), U33.1 (D1+)
- new net: J2.3 (D+), U33.2 (D1-)
- no-connect marks 159 -> 198
Other:
- note added: "0x77"
- note added: "I2C_MUX"
- note added: "I2C_TRANSLATOR"
- note added: "UART"
- note added: "USB Phy"
- note added: "VDD18"
- moved on the sheet: C337, C338, C339, C340, C341, C342, C343, C344, C345, C346, C347, C348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

Commit message: Added 04D High Speed Peripherals
Parts:
- USB2: footprint easyeda2kicad:USB-C-SMD_TYPE-C-24P-SMD -> Devboard_Footprints:USB-C-SMD_TYPE-C-24P-SMD
Changed lines of the file:
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@@
 			)
 		)
-		(property "Footprint" "easyeda2kicad:USB-C-SMD_TYPE-C-24P-SMD"
+		(property "Footprint" "Devboard_Footprints:USB-C-SMD_TYPE-C-24P-SMD"
 			(at 716.28 582.93 0)
 			(hide yes)
