File: PCB/schematics/04_Zynq/04d_Zynq_PS_HighSpeed.kicad_sch (KiCad schematic)
At the start: 0 parts

Commit message: Added 04D High Speed Peripherals
Parts:
- added CN1: APCI0120-P001A, easyeda2kicad:CONN-SMD_APCI0120-P001A, symbol Devboard_Custom:APCI0120-P001A
- added L11: DLW21HN900SQ2L-CUTTAPE, easyeda2kicad:FILTER-SMD_4P-L2.0-W1.3-BL_DLW21, symbol Devboard_Custom:DLW21HN900SQ2L-CUTTAPE
- added U38: USB3320C-EZK-TR, Devboard_Footprints:QFN-32_L5.0-W5.0-P0.50-BL-EP3.4, symbol Devboard_Custom:USB3320C-EZK-TR
- added U39: TPD4E05U06DQA, Package_SON:USON-10_2.5x1.0mm_P0.5mm, symbol Power_Protection:TPD4E05U06DQA
- added USB3: TYPE-C-24P-SMD, Devboard_Footprints:USB-C-SMD_TYPE-C-24P-SMD, symbol Devboard_Custom:TYPE-C-24P-SMD
- added USB4: 472720001, Devboard_Footprints:CONN-SMD_472720001, symbol Devboard_Custom:472720001
Connections:
- new net: U39.3 (GND), U39.8 (GND)

Commit message: High Speed Peripherals added
Parts:
- removed U38: USB3320C-EZK-TR, Devboard_Footprints:QFN-32_L5.0-W5.0-P0.50-BL-EP3.4, symbol Devboard_Custom:USB3320C-EZK-TR
- added C396, C397: 100nF, Capacitor_SMD:C_0402_1005Metric, symbol Device:C
- added C398: 1nF, Capacitor_SMD:C_0402_1005Metric, symbol Device:C
- added R160, R161: 5.1kΩ, Resistor_SMD:R_0402_1005Metric, symbol Device:R
- added R162, R163: 100kΩ, Resistor_SMD:R_0402_1005Metric, symbol Device:R
- added R164: 1MΩ, Resistor_SMD:R_0402_1005Metric, symbol Device:R
- L11: footprint easyeda2kicad:FILTER-SMD_4P-L2.0-W1.3-BL_DLW21 -> Devboard_Footprints:FILTER-SMD_4P-L2.0-W1.3-BL_DLW21
Connections:
- net SH: now reaches USB3.25
- net SH: now also USB3.3, USB3.4, C398.2, R164.1
- net GND: now reaches USB3.A1 (GND)
- net GND: now also U39.3 (GND), U39.8 (GND), USB3.A12 (GND), USB3.B1 (GND), USB3.B12 (GND), USB4.21 (GND), USB4.22 (GND), USB4.23 (GND), USB4.24 (GND), C396.2, C397.2, C398.1, R160.2, R161.2, R162.2, R164.2
- net USB3_RX_N: now reaches USB3.A10 (SSRXn2)
- net USB3_RX_N: now also U39.5 (D2-), USB3.B10 (SSRXn1)
- net D1+: now reaches USB3.A2 (SSTXp1)
- net D1+: now also L11.4, U39.1 (D1+), USB3.B2 (SSTXp2)
- net D1-: now reaches USB3.A3 (SSTXn1)
- net D1-: now also L11.3, U39.4 (D2+), USB3.B3 (SSTXn2)
- net USB3_VBUS: now reaches USB3.A4 (VBUS)
- net USB3_VBUS: now also USB3.A9 (VBUS), USB3.B4 (VBUS), USB3.B9 (VBUS), R163.2
- net CC1: now reaches USB3.A5 (CC1)
- net CC1: now also R160.1
- net USBDP_DN2: now reaches USB3.A6 (Dp1)
- net USBDP_DN2: now also USB3.B6 (Dp2)
- net USBDM_DN2: now reaches USB3.A7 (Dn1)
- net USBDM_DN2: now also USB3.B7 (Dn2)
- net CC2: now reaches USB3.B5 (CC2)
- net CC2: now also R161.1
- net USB3_TX_P: now reaches L11.1
- net USB3_TX_P: now also C396.1
- net USB3_TX_N: now reaches L11.2
- net USB3_TX_N: now also C397.1
- net USB3_RX_P: now reaches U39.2 (D1-)
- new net USB3_VBUS_NET: R162.1, R163.1
- no-connect marks 0 -> 3
Other:
- note added: "USB3 Super Speed"
- moved on the sheet: CN1, L11, U39, USB3, USB4

Commit message: feat: Section 4 Done
Parts:
- removed CN1: APCI0120-P001A, easyeda2kicad:CONN-SMD_APCI0120-P001A, symbol Devboard_Custom:APCI0120-P001A
- added C414, C415, C416, C417, C419, C420, C421, C422, C423, C424, C425, C426: 100nF, Capacitor_SMD:C_0402_1005Metric, symbol Device:C
- added C418: 10uF, Capacitor_SMD:C_0805_2012Metric, symbol Device:C
- added CN1: 1-2199230-6, Devboard_Footprints:PCIE-SMD_1-2199230-6, symbol Devboard_Custom:1-2199230-6
- added R166, R174, R175, R176: 10kΩ, Resistor_SMD:R_0402_1005Metric, symbol Device:R
- added R167, R168: 33Ω, Resistor_SMD:R_0402_1005Metric, symbol Device:R
- added R172, R173: 50Ω, Resistor_SMD:R_0402_1005Metric, symbol Device:R
- added U: TXS0102DQE, Package_SON:X2SON-8_1.4x1mm_P0.35mm, symbol Logic_LevelTranslator:TXS0102DQE
- added Y3: SiT9365AI-4B2-33E100.0000000, Oscillator:Oscillator_SMD_SiTime_PQFD-6L_3.2x2.5mm, symbol Oscillator:SiT9365xx-xBx-xxE
Connections:
- net GND: now also USB4.11, USB4.13, USB4.14, USB4.16, USB4.19, USB4.2, USB4.5, USB4.8, C414.1, C417.1, C418.1, CN1.1, CN1.15, CN1.21, CN1.27, CN1.3, CN1.33, CN1.39, CN1.45, CN1.51, CN1.57, CN1.71, CN1.73, CN1.75, CN1.9, R172.2, R173.2, U.4 (GND), Y3.3 (GND)
- net USB3_RX_P: now also USB3.A11 (SSRXp2), USB3.B11 (SSRXp1)
- net at USB4.1: now also C422.2
- net DP_AUX_P: now reaches USB4.15
- net DP_AUX_N: now reaches USB4.17
- net DP_HPD: now reaches USB4.18
- net +3V3: now reaches USB4.20
- net +3V3: now also C414.2, C417.2, C418.2, CN1.12, CN1.14, CN1.16, CN1.18, CN1.2, CN1.4, CN1.70, CN1.72, CN1.74, R166.1, R174.1, R175.1, R176.1, Y3.6 (VDD)
- net at USB4.3: now also C426.2
- new net: R168.1, Y3.5 (OUT-)
- new net: C416.2, R168.2, R173.1
- new net: C423.2, C424.1
- new net: C420.2, C421.1
- new net: C421.2, C422.1
- new net: C419.2, C420.1
- new net: C424.2, C425.1
- new net: R166.2, Y3.1 (OE)
- new net: R167.1, Y3.4 (OUT+)
- new net: C425.2, C426.1
- new net: C415.2, R167.2, R172.1
- new net CLKREQ#: CN1.52, R175.2, U.3 (A2)
- new net DP_TX0_N: C423.1
- new net DP_TX0_P: C419.1
- new net MIO50: U.7 (B1)
- new net MIO51: U.6 (B2)
- new net PCIE_RX_N: CN1.29
- new net PCIE_RX_P: CN1.31
- new net PCIE_TX_N: CN1.35
- new net PCIE_TX_P: CN1.37
- new net PERST#: CN1.50, R176.2, U.2 (A1)
- new net PEWAKE#: CN1.54, R174.2
- new net REFCLK_N_TERM: C416.1, CN1.53
- new net REFCLK_P_TERM: C415.1, CN1.55
- no-connect marks 3 -> 39
Other:
- note added: "DisplayPort"
- note added: "PCIE"
- note added: "SECTION 04d : High Speed Peripherals"
- moved on the sheet: C396, C397, C398, L11, R160, R161, R162, R163, R164, U39, USB3, USB4

Commit message: Feat : Schematics Complete
Parts:
- added C424, C429: 10uF, Capacitor_SMD:C_0805_2012Metric, symbol Device:C
- added C426, C428: 100nF, Capacitor_SMD:C_0402_1005Metric, symbol Device:C
- added FB10: 120Ω@100MHz, Inductor_SMD:L_01005_0402Metric, symbol Device:FerriteBead
- added J12: SFP+, Connector:Connector_SFP_and_Cage, symbol Interface_Optical:SFP+
- added R194: 10kΩ, Resistor_SMD:R_0402_1005Metric, symbol Device:R
- renumbered C419 to C412, C420 to C413, C421 to C414, C422 to C415, C423 to C416, C424 to C417, C425 to C418, C426 to C419, C396 to C420, C397 to C421, C398 to C422, C414 to C423, C415 to C425, C416 to C427, C417 to C430, C418 to C431, R160 to R163, R161 to R164, R162 to R165, R163 to R166, R164 to R167, R172 to R168, R167 to R169, R166 to R170, R168 to R171, R174 to R172, R175 to R173, R176 to R174, R173 to R175, U to U40, Y3 to Y4
Connections:
- net +3V3: now also U40.1 (VCCA), U40.8 (VCCB), C424.2, C426.2, FB10.2, R194.1
- net GND: now also C424.1, C426.1, C428.1, C429.1, J12.1 (VeeT), J12.10 (VeeR), J12.11 (VeeR), J12.14 (VeeR), J12.17 (VeeT), J12.20 (VeeT), J12.CAGE
- net at U40.5 (OE): now also R194.2
- new net: C428.2, C429.2, FB10.1, J12.15 (VccR), J12.16 (VccT)
- new net I2C_SCL_2_T: J12.5 (SCL)
- new net I2C_SDA_2_T: J12.4 (SDA)
- new net SFP_RX_N: J12.12 (RD-)
- new net SFP_RX_P: J12.13 (RD+)
- new net SFP_TX_N: J12.19 (TD-)
- new net SFP_TX_P: J12.18 (TD+)
- no-connect marks 39 -> 51
Other:
- note added: "SEF CAGE"
- moved on the sheet: C423, C425, C427, C430, C431, CN1, R168, R169, R170, R171, R172, R173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
