File: PCB/Devboard.kicad_pcb (KiCad board)
At the start: 2 copper layers, 353 parts, among them J1 Conn_01x02_Pin, J2 Conn_01x03_Pin, J3 Conn_01x03_Pin, J4 Conn_01x03_Pin, J5 Conn_01x03_Pin, J6 Conn_01x03_Pin, J7 Conn_01x03_Pin, J8 Conn_ARM_JTAG_SWD_10, Q1 IPB180P04P4L-02, U1 TVS2201DRBR, U10 TPS62822DLCR, U11 TPS62823DLCR, U12 TPS548A20RVER, U13 TPS7A4700RGWR, U14 TPS3700DSET, U15 TPS54824RNVR, U16 TPS54824RNVR, U17 TPS7A4700RGWR, U2 TPD6S300ARUKR, U20 TPS54824RNVR, U3 xczu4evfbvb900pkg, U4 TPS2121RUXR, U5 TPS259470ARPWR, U6 BQ25895RTWR, U7 BQ27441DRZR-G1A, U8 TPS62130RGTR, U9 XT60, Y1 ASE-33.333MHz, Y2 32.768 kHz

Commit message: Journal Update
Routing:
- net +0V9_VCU_GT: track 0.00 -> 14.9 mm
- net +1V8: track 0.00 -> 4.83 mm, vias 0 -> 2
- net unconnected-(U3-GND-PadR9): track 0.00 -> 0.67 mm
Changed lines of the file:
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@@
 				(font
 					(size 1.27 1.27)
+					(thickness 0.15)
 				)
 			)
@@
 		)
 		(embedded_fonts no)
-		(model "${EASYEDA2KICAD}/easyeda2kicad.3dshapes/VSON-8_L2.0-W1.5-H1.0-P0.50-BL.wrl"
+		(model "${KIPRJMOD}/libraries/3dmodels/VSON-8_L2.0-W1.5-H1.0-P0.50-BL.step"
 			(offset
 				(xyz 0 0 0)
@@
 				(font
 					(size 1.27 1.27)
+					(thickness 0.15)
 				)
 			)
@@
 		)
 		(embedded_fonts no)
-		(model "${EASYEDA2KICAD}/easyeda2kicad.3dshapes/SON-12_L4.0-W2.5-H1-P0.40-BL-EP.wrl"
+		(model "${KIPRJMOD}/libraries/3dmodels/SON-12_L4.0-W2.5-H1-P0.40-BL-EP.step"
 			(offset
 				(xyz 0 0 0)
@@
 				(font
 					(size 1.27 1.27)
+					(thickness 0.15)
 				)
 			)
@@
 		)
 		(embedded_fonts no)
-		(model "${EASYEDA2KICAD}/easyeda2kicad.3dshapes/WSON-6_L1.5-W1.5-H0.8-P0.50-TL.wrl"
+		(model "${KIPRJMOD}/libraries/3dmodels/WSON-6_L1.5-W1.5-H0.8-P0.50-TL.step"
 			(offset
 				(xyz 0 0 0)
@@
 				(font
 					(size 1.27 1.27)
+					(thickness 0.15)
 				)
 			)
@@
 		)
 		(embedded_fonts no)
-		(model "${EASYEDA2KICAD}/easyeda2kicad.3dshapes/VSON-8_L2.0-W1.5-H1.0-P0.50-BL.wrl"
+		(model "${KIPRJMOD}/libraries/3dmodels/VSON-8_L2.0-W1.5-H1.0-P0.50-BL.step"
 			(offset
 				(xyz 0 0 0)
@@
 				(font
 					(size 1.27 1.27)
+					(thickness 0.15)
 				)
 			)
@@
 		)
 		(embedded_fonts no)
-		(model "${EASYEDA2KICAD}/easyeda2kicad.3dshapes/VQFN-20_L5.0-W5.0-H1.0-P0.65.wrl"
+		(model "${KIPRJMOD}/libraries/3dmodels/VQFN-20_L5.0-W5.0-H1.0-P0.65.step"
 			(offset
 				(xyz 0 0 0)
@@
 				(font
 					(size 1.27 1.27)
+					(thickness 0.15)
 				)
 			)
@@
 		)
 		(embedded_fonts no)
-		(model "${EASYEDA2KICAD}/easyeda2kicad.3dshapes/TO-263-7_L10.2-W9.2-P1.27-LS15.4.wrl"
+		(model "${KIPRJMOD}/libraries/3dmodels/TO-263-7_L10.2-W9.2-P1.27-LS15.4.step"
 			(offset
 				(xyz 0 0 0)
@@
 				(font
 					(size 1.27 1.27)
+					(thickness 0.15)
 				)
 			)
@@
 		)
 		(embedded_fonts no)
-		(model "${EASYEDA2KICAD}/easyeda2kicad.3dshapes/VQFN-HR-12_L2.5-W2.0-H1.0-P0.50-BL.wrl"
+		(model "${KIPRJMOD}/libraries/3dmodels/VQFN-HR-12_L2.5-W2.0-H1.0-P0.50-BL.step"
 			(offset
 				(xyz 0 0 0)
@@
 			)
 		)
-		(attr)
 		(duplicate_pad_numbers_are_jumpers no)
 		(fp_circle
@@
 				(font
 					(size 1.27 1.27)
+					(thickness 0.15)
 				)
 			)
@@
 		)
 		(embedded_fonts no)
-		(model "${EASYEDA2KICAD}/easyeda2kicad.3dshapes/QFN-16_L3.0-W3.0-P0.50-EP1.7.wrl"
+		(model "${KIPRJMOD}/libraries/3dmodels/QFN-16_L3.0-W3.0-P0.50-EP1.7.step"
 			(offset
 				(xyz 0 0 0)
@@
 			)
 		)
-		(attr)
 		(duplicate_pad_numbers_are_jumpers no)
 		(fp_circle
@@
 			)
 		)
-		(attr)
 		(duplicate_pad_numbers_are_jumpers no)
 		(fp_circle
@@
 			)
 		)
-		(attr)
 		(duplicate_pad_numbers_are_jumpers no)
 		(fp_circle
@@
 			)
 		)
-		(attr)
 		(duplicate_pad_numbers_are_jumpers no)
 		(fp_circle
@@
 				(font
 					(size 1.27 1.27)
+					(thickness 0.15)
 				)
 			)
@@
 		)
 		(embedded_fonts no)
-		(model "${EASYEDA2KICAD}/easyeda2kicad.3dshapes/VQFN-10_L2.0-W2.0-P0.45-TL.wrl"
+		(model "${KIPRJMOD}/libraries/3dmodels/VQFN-10_L2.0-W2.0-P0.45-TL.step"
 			(offset
 				(xyz 0 0 0)
@@
 				(font
 					(size 1.27 1.27)
+					(thickness 0.15)
 				)
 			)
@@
 				(font
 					(size 1.27 1.27)
+					(thickness 0.15)
 				)
 			)
@@
 		)
 		(embedded_fonts no)
-		(model "${EASYEDA2KICAD}/easyeda2kicad.3dshapes/WQFN-20_L3.0-W3.0-H0.8-P0.40-TL-EP1.7.wrl"
+		(model "${KIPRJMOD}/libraries/3dmodels/WQFN-20_L3.0-W3.0-H0.8-P0.40-TL-EP1.7.step"
 			(offset
 				(xyz 0 0 0)
@@
 			)
 		)
-		(attr)
 		(duplicate_pad_numbers_are_jumpers no)
 		(fp_circle
@@
 				(font
 					(size 1.27 1.27)
+					(thickness 0.15)
 				)
 			)
@@
 		)
 		(embedded_fonts no)
-		(model "${EASYEDA2KICAD}/easyeda2kicad.3dshapes/DC-IN-TH_PJ-102AH.wrl"
+		(model "${KIPRJMOD}/libraries/3dmodels/DC-IN-TH_PJ-102AH.step"
 			(offset
 				(xyz 0 0 0)
@@
 				(font
 					(size 1.27 1.27)
+					(thickness 0.15)
 				)
 			)
@@
 		)
 		(embedded_fonts no)
-		(model "${EASYEDA2KICAD}/easyeda2kicad.3dshapes/VQFN-CLIP-28_L4.5-W3.5-H0.9-P0.40-BL-EP.wrl"
+		(model "${KIPRJMOD}/libraries/3dmodels/VQFN-CLIP-28_L4.5-W3.5-H0.9-P0.40-BL-EP.step"
 			(offset
 				(xyz 0 0 0)
@@
 				(font
 					(size 1.27 1.27)
+					(thickness 0.15)
 				)
 			)
@@
 				(font
 					(size 1.27 1.27)
+					(thickness 0.15)
 				)
 			)
@@
 		)
 		(embedded_fonts no)
-		(model "${EASYEDA2KICAD}/easyeda2kicad.3dshapes/VSON-8_L3.0-W3.0-H0.9-P0.65.wrl"
+		(model "${KIPRJMOD}/libraries/3dmodels/VSON-8_L3.0-W3.0-H0.9-P0.65.step"
 			(offset
 				(xyz 0 0 0)
@@
 				(font
 					(size 1.27 1.27)
+					(thickness 0.15)
 				)
 			)
@@
 		)
 		(embedded_fonts no)
-		(model "${EASYEDA2KICAD}/easyeda2kicad.3dshapes/VQFN-20_L5.0-W5.0-H1.0-P0.65.wrl"
+		(model "${KIPRJMOD}/libraries/3dmodels/VQFN-20_L5.0-W5.0-H1.0-P0.65.step"
 			(offset
 				(xyz 0 0 0)
@@
 				(font
 					(size 1.27 1.27)
+					(thickness 0.15)
 				)
 			)
@@
 		)
 		(embedded_fonts no)
-		(model "${EASYEDA2KICAD}/easyeda2kicad.3dshapes/QFN-24_L4.0-W4.0-P0.50-TL-EP2.7.wrl"
+		(model "${KIPRJMOD}/libraries/3dmodels/QFN-24_L4.0-W4.0-P0.50-TL-EP2.7.step"
 			(offset
 				(xyz 0 0 0)
@@
 				(font
 					(size 1.27 1.27)
+					(thickness 0.15)
 				)
 			)
@@
 				(font
 					(size 1.27 1.27)
+					(thickness 0.15)
 				)
 			)
@@
 				(font
 					(size 1.27 1.27)
+					(thickness 0.15)
 				)
 			)
@@
 		)
 		(embedded_fonts no)
-		(model "${EASYEDA2KICAD}/easyeda2kicad.3dshapes/USB-C-SMD_TYPE-C-24P-SMD.wrl"
+		(model "${KIPRJMOD}/libraries/3dmodels/USB-C-SMD_TYPE-C-24P-SMD.step"
 			(offset
 				(xyz 0 0 0)
@@
 		)
 	)
+	(segment
+		(start 16.55 11.55)
+		(end 19.55 11.55)
+		(width 0.2)
+		(layer "F.Cu")
+		(net "+0V9_VCU_GT")
+	)
+	(segment
+		(start 13.55 15.55)
+		(end 16.55 12.55)
+		(width 0.2)
+		(layer "F.Cu")
+		(net "+0V9_VCU_GT")
+	)
+	(segment
+		(start 18.55 9.55)
+		(end 19.55 9.55)
+		(width 0.2)
+		(layer "F.Cu")
+		(net "+0V9_VCU_GT")
+	)
+	(segment
+		(start 12.55 12.55)
+		(end 14.55 14.55)
+		(width 0.2)
+		(layer "F.Cu")
+		(net "+0V9_VCU_GT")
+	)
+	(segment
+		(start 17.55 10.55)
+		(end 18.55 10.55)
+		(width 0.2)
+		(layer "F.Cu")
+		(net "+0V9_VCU_GT")
+	)
+	(segment
+		(start 12.55 14.55)
+		(end 14.55 12.55)
+		(width 0.2)
+		(layer "F.Cu")
+		(net "+0V9_VCU_GT")
+	)
+	(segment
+		(start 14.55 21.55)
+		(end 14.54 21.54)
+		(width 0.2)
+		(layer "F.Cu")
+		(net "+1V8")
+	)
+	(via
+		(at 10.55 19.55)
+		(size 0.6)
+		(drill 0.3)
+		(layers "F.Cu" "B.Cu")
+		(net "+1V8")
+	)
+	(via
+		(at 14.54 21.54)
+		(size 0.6)
+		(drill 0.3)
+		(layers "F.Cu" "B.Cu")
+		(net "+1V8")
+	)
+	(segment
+		(start 12.55 19.55)
+		(end 10.55 19.55)
+		(width 0.2)
+		(layer "B.Cu")
+		(net "+1V8")
+	)
+	(segment
+		(start 14.54 21.54)
+		(end 12.55 19.55)
+		(width 0.2)
+		(layer "B.Cu")
+		(net "+1V8")
+	)
+	(segment
+		(start 16.92 10.92)
+		(end 17.07 10.92)
+		(width 0.2)
+		(layer "F.Cu")
+		(net "unconnected-(U3-GND-PadR9)")
+	)
+	(segment
+		(start 16.55 10.55)
+		(end 16.92 10.92)
+		(width 0.2)
+		(layer "F.Cu")
+		(net "unconnected-(U3-GND-PadR9)")
+	)
 	(group ""

Commit message: Feat: Zynq Peripherals added
Parts:
- removed J1: Conn_01x02_Pin, Connector_PinHeader_2.54mm:PinHeader_1x02_P2.54mm_Vertical
- removed J2, J3, J4, J5, J6, J7: Conn_01x03_Pin, Connector_PinSocket_2.54mm:PinSocket_1x03_P2.54mm_Vertical
- removed J8: Conn_ARM_JTAG_SWD_10, Connector_PinHeader_1.27mm:PinHeader_2x05_P1.27mm_Vertical
- removed TP3: RST Probe, TestPoint:TestPoint_Pad_D2.0mm
- removed TP4, TP5, TP6: TestPoint, TestPoint:TestPoint_Pad_D2.0mm
- added C209: 0.1uF, Capacitor_SMD:C_0402_1005Metric, F.Cu at (96.9, 118.5)
- added C210: 0.1uF, Capacitor_SMD:C_0402_1005Metric, F.Cu at (99.8, 94.9)
- added C211: 0.1uF, Capacitor_SMD:C_0402_1005Metric, F.Cu at (99.8, 96.9)
- added C212: 0.1uF, Capacitor_SMD:C_0402_1005Metric, F.Cu at (99.8, 98.8)
- added C213: 0.1uF, Capacitor_SMD:C_0402_1005Metric, F.Cu at (99.8, 100.8)
- added C214: 0.1uF, Capacitor_SMD:C_0402_1005Metric, F.Cu at (99.8, 102.8)
- added C215: 0.1uF, Capacitor_SMD:C_0402_1005Metric, F.Cu at (99.8, 104.7)
- added C216: 0.1uF, Capacitor_SMD:C_0402_1005Metric, F.Cu at (99.8, 106.7)
- added C217: 0.1uF, Capacitor_SMD:C_0402_1005Metric, F.Cu at (99.8, 108.7)
- added C218: 0.1uF, Capacitor_SMD:C_0402_1005Metric, F.Cu at (99.8, 110.7)
- added C219: 0.1uF, Capacitor_SMD:C_0402_1005Metric, F.Cu at (99.8, 112.6)
- added C220: 0.1uF, Capacitor_SMD:C_0402_1005Metric, F.Cu at (99.8, 114.6)
- added C221: 0.1uF, Capacitor_SMD:C_0402_1005Metric, F.Cu at (99.8, 116.6)
- added C222: 0.1uF, Capacitor_SMD:C_0402_1005Metric, F.Cu at (99.8, 118.5)
- added C223: 0.1uF, Capacitor_SMD:C_0402_1005Metric, F.Cu at (102.7, 94.9)
- added C224: 0.1uF, Capacitor_SMD:C_0402_1005Metric, F.Cu at (102.7, 96.9)
- added C225: 0.1uF, Capacitor_SMD:C_0402_1005Metric, F.Cu at (102.7, 98.8)
- added C226: 0.1uF, Capacitor_SMD:C_0402_1005Metric, F.Cu at (102.7, 100.8)
- added C227: 0.1uF, Capacitor_SMD:C_0402_1005Metric, F.Cu at (102.7, 102.8)
- added C228: 0.1uF, Capacitor_SMD:C_0402_1005Metric, F.Cu at (102.7, 104.7)
- added C229: 0.1uF, Capacitor_SMD:C_0402_1005Metric, F.Cu at (102.7, 106.7)
- added C230: 0.1uF, Capacitor_SMD:C_0402_1005Metric, F.Cu at (102.7, 108.7)
- added C231: 0.1uF, Capacitor_SMD:C_0402_1005Metric, F.Cu at (102.7, 110.7)
- added C232: 0.1uF, Capacitor_SMD:C_0402_1005Metric, F.Cu at (102.7, 112.6)
- added C233: 0.1uF, Capacitor_SMD:C_0402_1005Metric, F.Cu at (102.7, 114.6)
- added C234: 0.1uF, Capacitor_SMD:C_0402_1005Metric, F.Cu at (102.7, 116.6)
- added C235: 0.1uF, Capacitor_SMD:C_0402_1005Metric, F.Cu at (102.7, 118.5)
- added C236: 0.1uF, Capacitor_SMD:C_0402_1005Metric, F.Cu at (105.5, 94.9)
- added C237: 0.1uF, Capacitor_SMD:C_0402_1005Metric, F.Cu at (105.5, 96.9)
- added C238: 0.1uF, Capacitor_SMD:C_0402_1005Metric, F.Cu at (105.5, 98.8)
- added C239: 0.1uF, Capacitor_SMD:C_0402_1005Metric, F.Cu at (105.5, 100.8)
- added C240: 0.1uF, Capacitor_SMD:C_0402_1005Metric, F.Cu at (105.5, 102.8)
- added C241: 0.1uF, Capacitor_SMD:C_0402_1005Metric, F.Cu at (105.5, 104.7)
- added C242: 0.1uF, Capacitor_SMD:C_0402_1005Metric, F.Cu at (105.5, 106.7)
- added C243: 0.1uF, Capacitor_SMD:C_0402_1005Metric, F.Cu at (105.5, 108.7)
- added C244: 0.1uF, Capacitor_SMD:C_0402_1005Metric, F.Cu at (105.5, 110.7)
- added C245: 0.1uF, Capacitor_SMD:C_0402_1005Metric, F.Cu at (105.5, 112.6)
- added C246: 0.1uF, Capacitor_SMD:C_0402_1005Metric, F.Cu at (105.5, 114.6)
- added C247: 0.1uF, Capacitor_SMD:C_0402_1005Metric, F.Cu at (105.5, 116.6)
- added C248: 0.1uF, Capacitor_SMD:C_0402_1005Metric, F.Cu at (0.94, 74.5)
- added C249: 0.1uF, Capacitor_SMD:C_0402_1005Metric, F.Cu at (0.94, 76.5)
- added C250: 0.1uF, Capacitor_SMD:C_0402_1005Metric, F.Cu at (0.94, 78.5)
- added C251: 0.1uF, Capacitor_SMD:C_0402_1005Metric, F.Cu at (0.94, 80.5)
- added C252: 0.1uF, Capacitor_SMD:C_0402_1005Metric, F.Cu at (0.94, 82.4)
- added C253: 0.1uF, Capacitor_SMD:C_0402_1005Metric, F.Cu at (0.94, 84.4)
- added C254: 0.1uF, Capacitor_SMD:C_0402_1005Metric, F.Cu at (0.94, 86.4)
- added C255: 0.1uF, Capacitor_SMD:C_0402_1005Metric, F.Cu at (0.94, 88.3)
- added C256: 0.1uF, Capacitor_SMD:C_0402_1005Metric, F.Cu at (0.94, 90.3)
- added C257: 0.1uF, Capacitor_SMD:C_0402_1005Metric, F.Cu at (0.94, 92.3)
- added C258: 0.1uF, Capacitor_SMD:C_0402_1005Metric, F.Cu at (0.94, 94.2)
- added C259: 0.1uF, Capacitor_SMD:C_0402_1005Metric, F.Cu at (0.94, 96.2)
- added C260: 0.1uF, Capacitor_SMD:C_0402_1005Metric, F.Cu at (0.94, 98.2)
- added C261: 0.1uF, Capacitor_SMD:C_0402_1005Metric, F.Cu at (3.81, 74.5)
- added C262: 0.1uF, Capacitor_SMD:C_0402_1005Metric, F.Cu at (3.81, 76.5)
- added C263: 0.1uF, Capacitor_SMD:C_0402_1005Metric, F.Cu at (3.81, 78.5)
- added C264: 0.1uF, Capacitor_SMD:C_0402_1005Metric, F.Cu at (3.81, 80.5)
- added C265: 0.1uF, Capacitor_SMD:C_0402_1005Metric, F.Cu at (3.81, 82.4)
- added C266: 0.1uF, Capacitor_SMD:C_0402_1005Metric, F.Cu at (3.81, 84.4)
- added C267: 0.1uF, Capacitor_SMD:C_0402_1005Metric, F.Cu at (3.81, 86.4)
- added C268: 0.1uF, Capacitor_SMD:C_0402_1005Metric, F.Cu at (3.81, 88.3)
- added C269: 0.1uF, Capacitor_SMD:C_0402_1005Metric, F.Cu at (3.81, 90.3)
- added C270: 0.1uF, Capacitor_SMD:C_0402_1005Metric, F.Cu at (3.81, 92.3)
- added C271: 0.1uF, Capacitor_SMD:C_0402_1005Metric, F.Cu at (3.81, 94.2)
- added C272: 0.1uF, Capacitor_SMD:C_0402_1005Metric, F.Cu at (3.81, 96.2)
- added C273: 0.1uF, Capacitor_SMD:C_0402_1005Metric, F.Cu at (3.81, 98.2)
- added C274: 0.1uF, Capacitor_SMD:C_0402_1005Metric, F.Cu at (6.67, 74.5)
- added C275: 0.1uF, Capacitor_SMD:C_0402_1005Metric, F.Cu at (6.67, 76.5)
- added C276: 0.1uF, Capacitor_SMD:C_0402_1005Metric, F.Cu at (6.67, 78.5)
- added C277: 0.1uF, Capacitor_SMD:C_0402_1005Metric, F.Cu at (6.67, 80.5)
- added C278: 0.1uF, Capacitor_SMD:C_0402_1005Metric, F.Cu at (6.67, 82.4)
- added C279: 0.1uF, Capacitor_SMD:C_0402_1005Metric, F.Cu at (6.67, 84.4)
- added C280: 0.1uF, Capacitor_SMD:C_0402_1005Metric, F.Cu at (6.67, 86.4)
- added C281: 0.1uF, Capacitor_SMD:C_0402_1005Metric, F.Cu at (6.67, 88.3)
- added C282: 0.1uF, Capacitor_SMD:C_0402_1005Metric, F.Cu at (6.67, 90.3)
- added C283: 0.1uF, Capacitor_SMD:C_0402_1005Metric, F.Cu at (6.67, 92.3)
- added C284: 0.1uF, Capacitor_SMD:C_0402_1005Metric, F.Cu at (6.67, 94.2)
- added C285: 0.1uF, Capacitor_SMD:C_0402_1005Metric, F.Cu at (6.67, 96.2)
- added C286: 0.1uF, Capacitor_SMD:C_0402_1005Metric, F.Cu at (6.67, 98.2)
- added C287: 0.1uF, Capacitor_SMD:C_0402_1005Metric, F.Cu at (9.54, 74.5)
- added C288: 0.1uF, Capacitor_SMD:C_0402_1005Metric, F.Cu at (9.54, 76.5)
- added C289: 0.1uF, Capacitor_SMD:C_0402_1005Metric, F.Cu at (9.54, 78.5)
- added C290: 0.1uF, Capacitor_SMD:C_0402_1005Metric, F.Cu at (9.54, 80.5)
- added C291: 0.1uF, Capacitor_SMD:C_0402_1005Metric, F.Cu at (9.54, 82.4)
- added C292: 0.1uF, Capacitor_SMD:C_0402_1005Metric, F.Cu at (9.54, 84.4)
- added C293: 0.1uF, Capacitor_SMD:C_0402_1005Metric, F.Cu at (9.54, 86.4)
- added C294: 0.1uF, Capacitor_SMD:C_0402_1005Metric, F.Cu at (9.54, 88.3)
- added C295: 0.1uF, Capacitor_SMD:C_0402_1005Metric, F.Cu at (9.54, 90.3)
- added C296: 0.1uF, Capacitor_SMD:C_0402_1005Metric, F.Cu at (9.54, 92.3)
- added C297: 0.1uF, Capacitor_SMD:C_0402_1005Metric, F.Cu at (9.54, 94.2)
- added C298: 0.1uF, Capacitor_SMD:C_0402_1005Metric, F.Cu at (9.54, 96.2)
- added C299: 0.1uF, Capacitor_SMD:C_0402_1005Metric, F.Cu at (9.54, 98.2)
- added C300: 0.1uF, Capacitor_SMD:C_0402_1005Metric, F.Cu at (12.4, 74.5)
- added C301: 0.1uF, Capacitor_SMD:C_0402_1005Metric, F.Cu at (12.4, 76.5)
- added C302: 0.1uF, Capacitor_SMD:C_0402_1005Metric, F.Cu at (12.4, 78.5)
- added C303: 0.1uF, Capacitor_SMD:C_0402_1005Metric, F.Cu at (12.4, 80.5)
- added C304: 0.1uF, Capacitor_SMD:C_0402_1005Metric, F.Cu at (12.4, 82.4)
- added C305: 0.1uF, Capacitor_SMD:C_0402_1005Metric, F.Cu at (12.4, 84.4)
- added C306: 0.1uF, Capacitor_SMD:C_0402_1005Metric, F.Cu at (12.4, 86.4)
- added C307: 0.1uF, Capacitor_SMD:C_0402_1005Metric, F.Cu at (12.4, 88.3)
- added C308: 0.1uF, Capacitor_SMD:C_0402_1005Metric, F.Cu at (12.4, 90.3)
- added C309: 0.1uF, Capacitor_SMD:C_0402_1005Metric, F.Cu at (12.4, 92.3)
- added C310: 0.1uF, Capacitor_SMD:C_0402_1005Metric, F.Cu at (12.4, 94.2)
- added C311: 0.1uF, Capacitor_SMD:C_0402_1005Metric, F.Cu at (12.4, 96.2)
- added C312: 0.1uF, Capacitor_SMD:C_0402_1005Metric, F.Cu at (12.4, 98.2)
- added C313: 0.1uF, Capacitor_SMD:C_0402_1005Metric, F.Cu at (15.3, 74.5)
- added C314: 0.1uF, Capacitor_SMD:C_0402_1005Metric, F.Cu at (15.3, 76.5)
- added C315: 0.1uF, Capacitor_SMD:C_0402_1005Metric, F.Cu at (15.3, 78.5)
- added C316: 0.1uF, Capacitor_SMD:C_0402_1005Metric, F.Cu at (15.3, 80.5)
- added C317: 0.1uF, Capacitor_SMD:C_0402_1005Metric, F.Cu at (15.3, 82.4)
- added C318: 0.1uF, Capacitor_SMD:C_0402_1005Metric, F.Cu at (15.3, 84.4)
- added C319: 0.1uF, Capacitor_SMD:C_0402_1005Metric, F.Cu at (15.3, 86.4)
- added C320: 0.1uF, Capacitor_SMD:C_0402_1005Metric, F.Cu at (15.3, 88.3)
- added C321: 0.1uF, Capacitor_SMD:C_0402_1005Metric, F.Cu at (15.3, 90.3)
- added C322: 0.1uF, Capacitor_SMD:C_0402_1005Metric, F.Cu at (15.3, 92.3)
- added C323: 0.1uF, Capacitor_SMD:C_0402_1005Metric, F.Cu at (15.3, 94.2)
- added C324: 0.1uF, Capacitor_SMD:C_0402_1005Metric, F.Cu at (15.3, 96.2)
- added C325: 0.1uF, Capacitor_SMD:C_0402_1005Metric, F.Cu at (15.3, 98.2)
- added C326: 0.1uF, Capacitor_SMD:C_0402_1005Metric, F.Cu at (18.2, 74.5)
- added C327: 0.1uF, Capacitor_SMD:C_0402_1005Metric, F.Cu at (18.2, 76.5)
- added C328: 0.1uF, Capacitor_SMD:C_0402_1005Metric, F.Cu at (18.2, 78.5)
- added C329: 0.1uF, Capacitor_SMD:C_0402_1005Metric, F.Cu at (18.2, 80.5)
- added C330: 0.1uF, Capacitor_SMD:C_0402_1005Metric, F.Cu at (18.2, 82.4)
- added C331: 0.1uF, Capacitor_SMD:C_0402_1005Metric, F.Cu at (18.2, 84.4)
- added C332: 0.1uF, Capacitor_SMD:C_0402_1005Metric, F.Cu at (18.2, 86.4)
- added C333: 0.1uF, Capacitor_SMD:C_0402_1005Metric, F.Cu at (18.2, 88.3)
- added C334: 0.1uF, Capacitor_SMD:C_0402_1005Metric, F.Cu at (18.2, 90.3)
- added C335: 0.1uF, Capacitor_SMD:C_0402_1005Metric, F.Cu at (18.2, 92.3)
- added C336: 0.1uF, Capacitor_SMD:C_0402_1005Metric, F.Cu at (18.2, 94.2)
- added C337: 0.1uF, Capacitor_SMD:C_0402_1005Metric, F.Cu at (40.9, 114.5)
- added C338: 0.1uF, Capacitor_SMD:C_0402_1005Metric, F.Cu at (40.9, 116.5)
- added C339: 1uF, Capacitor_SMD:C_0402_1005Metric, F.Cu at (40.9, 118.5)
- added C340: 0.1uF, Capacitor_SMD:C_0402_1005Metric, F.Cu at (40.9, 120.4)
- added C341: 1uF, Capacitor_SMD:C_0402_1005Metric, F.Cu at (40.9, 122.4)
- added C342: 0.1uF, Capacitor_SMD:C_0402_1005Metric, F.Cu at (40.9, 124.4)
- added C343: 1uF, Capacitor_SMD:C_0402_1005Metric, F.Cu at (40.9, 126.3)
- added C344: 0.1uF, Capacitor_SMD:C_0402_1005Metric, F.Cu at (43.8, 114.5)
- added C345: 1uF, Capacitor_SMD:C_0402_1005Metric, F.Cu at (43.8, 116.5)
- added C346: 0.1uF, Capacitor_SMD:C_0402_1005Metric, F.Cu at (43.8, 118.5)
- added C347: 0.1uF, Capacitor_SMD:C_0402_1005Metric, F.Cu at (43.8, 120.4)
- added C348: 1uF, Capacitor_SMD:C_0402_1005Metric, F.Cu at (43.8, 122.4)
- added C349: 1uF, Capacitor_SMD:C_0402_1005Metric, F.Cu at (43.8, 124.4)
- added C350: 0.1uF, Capacitor_SMD:C_0402_1005Metric, F.Cu at (43.8, 126.3)
- added C351: 0.1uF, Capacitor_SMD:C_0402_1005Metric, F.Cu at (46.7, 114.5)
- added C352: 1uF, Capacitor_SMD:C_0402_1005Metric, F.Cu at (46.7, 116.5)
- added C353: 1uF, Capacitor_SMD:C_0402_1005Metric, F.Cu at (46.7, 118.5)
- added C354: 0.1uF, Capacitor_SMD:C_0402_1005Metric, F.Cu at (46.7, 120.4)
- added C355: 1uF, Capacitor_SMD:C_0402_1005Metric, F.Cu at (46.7, 122.4)
- added C356: 1uF, Capacitor_SMD:C_0402_1005Metric, F.Cu at (46.7, 124.4)
- added C357: 0.1uF, Capacitor_SMD:C_0402_1005Metric, F.Cu at (46.7, 126.3)
- added C358: 0.1uF, Capacitor_SMD:C_0402_1005Metric, F.Cu at (49.5, 114.5)
- added C359: 0.1uF, Capacitor_SMD:C_0402_1005Metric, F.Cu at (49.5, 116.5)
- added C360: 1uF, Capacitor_SMD:C_0402_1005Metric, F.Cu at (49.5, 118.5)
- added D6: LSMB24CAH, Diode_SMD:D_SMC, F.Cu at (73.6, 18.9)
- added D7: SMBJ20A, Diode_SMD:D_SMC, F.Cu at (73.6, 26.6)
- added D8: D_Schottky, Diode_SMD:D_SMC, F.Cu at (73.6, 34.4)
- added D9: D_Schottky, Diode_SMD:D_SMC, F.Cu at (73.6, 42.1)
- added FB2: 120Ω@100MHz, Inductor_SMD:L_01005_0402Metric, F.Cu at (56.6, 46.8)
- added FB3: 120Ω@100MHz, Inductor_SMD:L_01005_0402Metric, F.Cu at (56.6, 48.5)
- added FB4: 120Ω@100MHz, Inductor_SMD:L_01005_0402Metric, F.Cu at (56.6, 50.1)
- added FB5: 120Ω@100MHz, Inductor_SMD:L_01005_0402Metric, F.Cu at (56.6, 51.8)
- added FB6: 120Ω@100MHz, Inductor_SMD:L_01005_0402Metric, F.Cu at (56.6, 53.4)
- added L10: 1uH, Inductor_SMD:L_Bourns_SRP1245A, F.Cu at (54.6, 20.6)
- added L8: 2.2uH,5A, Inductor_SMD:L_Bourns_SRP1245A, F.Cu at (47.4, 79.9)
- added Q2: IPB180P04P4L-02, Package_TO_SOT_SMD:TO-263-7_TabPin8, F.Cu at (95.4, 18.0)
- added R100: 50K, Resistor_SMD:R_0402_1005Metric, F.Cu at (20.1, 36.6)
- added R101: 100k, Resistor_SMD:R_0402_1005Metric, F.Cu at (20.1, 38.5)
- added R102: 10kΩ, Resistor_SMD:R_0402_1005Metric, F.Cu at (106.0, 37.1)
- added R103: 100kΩ, Resistor_SMD:R_0402_1005Metric, F.Cu at (108.9, 25.2)
- added R104: 124k, Resistor_SMD:R_0402_1005Metric, F.Cu at (108.9, 27.2)
- added R105: 10k, Resistor_SMD:R_0402_1005Metric, F.Cu at (108.9, 29.2)
- added R106: 549Ω, Resistor_SMD:R_0402_1005Metric, F.Cu at (108.9, 31.2)
- added R107: 1kΩ, Resistor_SMD:R_0402_1005Metric, F.Cu at (21.0, 80.5)
- added R108: 1kΩ, Resistor_SMD:R_0402_1005Metric, F.Cu at (21.0, 82.5)
- added R109: 240Ω, Resistor_SMD:R_0402_1005Metric, F.Cu at (21.0, 84.5)
- added R110: 10kΩ, Resistor_SMD:R_0402_1005Metric, F.Cu at (52.4, 116.5)
- added R111: 10kΩ, Resistor_SMD:R_0402_1005Metric, F.Cu at (52.4, 118.5)
- added R112: 10kΩ, Resistor_SMD:R_0402_1005Metric, F.Cu at (52.4, 120.5)
- added R113: 10kΩ, Resistor_SMD:R_0402_1005Metric, F.Cu at (52.4, 122.5)
- added R114: 10kΩ, Resistor_SMD:R_0402_1005Metric, F.Cu at (55.3, 114.5)
- added R115: 10kΩ, Resistor_SMD:R_0402_1005Metric, F.Cu at (55.3, 116.5)
- added R116: 22Ω, Resistor_SMD:R_0402_1005Metric, F.Cu at (55.3, 118.5)
- added R117: 22Ω, Resistor_SMD:R_0402_1005Metric, F.Cu at (55.3, 120.5)
- added R118: 10kΩ, Resistor_SMD:R_0402_1005Metric, F.Cu at (55.3, 122.5)
- added R119: 10kΩ, Resistor_SMD:R_0402_1005Metric, F.Cu at (58.3, 114.5)
- added R120: 10kΩ, Resistor_SMD:R_0402_1005Metric, F.Cu at (58.3, 116.5)
- added R121: 10kΩ, Resistor_SMD:R_0402_1005Metric, F.Cu at (58.3, 118.5)
- added R122: 10kΩ, Resistor_SMD:R_0402_1005Metric, F.Cu at (58.3, 120.5)
- added R89: 10kΩ, Resistor_SMD:R_0402_1005Metric, F.Cu at (74.3, 61.8)
- added R90: 100kΩ, Resistor_SMD:R_0402_1005Metric, F.Cu at (74.3, 63.8)
- added R92: 5.9kΩ, Resistor_SMD:R_0402_1005Metric, F.Cu at (106.0, 29.2)
- added R95: 5.1kΩ, Resistor_SMD:R_0402_1005Metric, F.Cu at (106.0, 35.1)
- added R96: 249k, Resistor_SMD:R_0402_1005Metric, F.Cu at (20.1, 30.6)
- added R97: 10kΩ, Resistor_SMD:R_0402_1005Metric, F.Cu at (20.1, 32.6)
- added R98: 1kΩ, Resistor_SMD:R_0402_1005Metric, F.Cu at (74.3, 67.8)
- added R99: 20k, Resistor_SMD:R_0402_1005Metric, F.Cu at (20.1, 34.6)
- added SW1: SW_Push, Button_Switch_SMD:SW_SPST_Omron_B3FS-100xP, F.Cu at (63.8, 90.1)
- added U18: DW06, Devboard_Footprints:SOT-23-6_L2.9-W1.6-P0.95-LS2.8-BL, F.Cu at (46.0, 94.0)
- added U19: TPS61088RHLR, Devboard_Footprints:VQFN-20_L4.6-W3.6-P0.50-BL, F.Cu at (73.2, 73.3)
- added U21: LM66100DCK, Package_TO_SOT_SMD:SOT-363_SC-70-6, F.Cu at (50.1, 93.7)
- added U22: TPS7A4700RGWR, Devboard_Footprints:VQFN-20_L5.0-W5.0-P0.65-TL-EP, F.Cu at (3.46, 45.2)
- added U23: TPS7A4700RGWR, Devboard_Footprints:VQFN-20_L5.0-W5.0-P0.65-TL-EP, F.Cu at (3.46, 52.2)
- added U24: TPS259470ARPWR, Devboard_Footprints:VQFN-10_L2.0-W2.0-P0.45-TL, F.Cu at (98.3, 44.0)
- added U25: TPS54824RNVR, Custom_Footprints:VQFN-18_L3.5-W3.5-P0.50-BL_TPS54824RNVR, F.Cu at (52.9, 46.8)
- added U26: xczu4evfbvb900pkg, Devboard_Footprints:XCZU4EVFBVB900PKG, F.Cu at (95.8, 76.4)
- added U27: RS3112-1.25XSF3, Devboard_Footprints:SOT-23-3_L2.9-W1.3-P0.95-LS2.4-BR, F.Cu at (46.5, 51.7)
- added U32: USB3320C-EZK-TR, Connector_USB:USB3_A_Plug_Wuerth_692112030100_Horizontal, F.Cu at (52.3, 105.9)
- added U33: USBLC6-2SC6, Package_TO_SOT_SMD:SOT-23-6, F.Cu at (65.3, 109.7)
- added U34: CP2102N-Axx-xQFN24, Package_DFN_QFN:QFN-24-1EP_4x4mm_P0.5mm_EP2.6x2.6mm, F.Cu at (54.5, 126.6)
- added U35: TXB0108PW, Package_SO:TSSOP-20_4.4x6.5mm_P0.65mm, F.Cu at (64.5, 126.9)
- added U36: TCA9548APWR, Package_SO:TSSOP-24_4.4x7.8mm_P0.65mm, F.Cu at (64.5, 118.2)
- added U37: PCA9306, Package_SO:VSSOP-8_2.3x2mm_P0.5mm, F.Cu at (42.3, 129.3)
- added U_RAM2: MT40A512M16LY-075:E, Devboard_Footprints:FBGA-96_L13.5-W7.5-R16-C6-P0.80-TL, F.Cu at (4.58, 66.2)
- added U_RAM3: MT40A512M16LY-075:E, Devboard_Footprints:FBGA-96_L13.5-W7.5-R16-C6-P0.80-TL, F.Cu at (14.1, 66.2)
- added U_RAM4: MT40A512M16LY-075:E, Devboard_Footprints:FBGA-96_L13.5-W7.5-R16-C6-P0.80-TL, F.Cu at (23.6, 66.2)
- added U_RAM5: MT40A512M16LY-075:E, Devboard_Footprints:FBGA-96_L13.5-W7.5-R16-C6-P0.80-TL, F.Cu at (33.1, 66.2)
- C100: value 0.1uF -> 10nF
- C101, C98: value 0.1uF -> 22uf 25v; footprint Capacitor_SMD:C_0402_1005Metric -> Capacitor_SMD:C_0805_2012Metric
- C102: value 0.1uF -> 4.7nF 50V
- C103: value 0.1uF -> 100pF
- C104: value 0.1uF -> 22pF
- C105, C107, C109: value 0.1uF -> 0.1uF 25V
- C106, C108, C91, C94: value 0.1uF -> 10uF
- C110: value 330uF -> 10uF
- C111: value 330uF -> 10nF 25V
- C112: value 100uF -> 47uF; footprint Capacitor_SMD:C_0402_1005Metric -> Capacitor_SMD:C_1206_3216Metric
- C113, C115: value 100uF -> 0.1uF 25V
- C114, C116: value 100uF -> 10uF
- C117, C169: value 100uF -> 0.1uF
- C118, C119, C120, C121, C122, C123, C124, C125, C126, C127, C128, C129, C130, C131, C132: value 47uF -> 0.1uF
- C13, C15: value 0.1uF 25V -> 0.1uF 50V
- C150: value 0.1uF -> 47uF; footprint Capacitor_SMD:C_0402_1005Metric -> Capacitor_SMD:C_1210_3225Metric
- C170: footprint Capacitor_SMD:C_0402_1005Metric -> Capacitor_SMD:C_1210_3225Metric
- C171, C172, C185, C191, C194: value 10uF -> 0.1uF
- C184, C187: value 1uF -> 0.1uF
- C188: value 4.7uF -> 0.1uF
- C199, C204, C207, C208: value 22uF -> 0.1uF
- C3, C6, C9: value 100uF 25V -> 100uF 35V
- C38, C39, C40, C41, C42, C70: footprint Capacitor_SMD:C_0402_1005Metric -> Capacitor_SMD:C_1206_3216Metric
- C5: value 330uF -> 2.2uF
- C76, C77: value 100uF -> 1uF; footprint Capacitor_SMD:C_0402_1005Metric -> Capacitor_SMD:C_1210_3225Metric
- C78: value 100uF -> 100nF; footprint Capacitor_SMD:C_0402_1005Metric -> Capacitor_SMD:C_1210_3225Metric
- C79: value 100uF -> 22uF; footprint Capacitor_SMD:C_0402_1005Metric -> Capacitor_SMD:C_0805_2012Metric
- C80, C81, C82: value 47uF -> 100nF
- C83: value 47uF -> 1uF; footprint Capacitor_SMD:C_0402_1005Metric -> Capacitor_SMD:C_1210_3225Metric
- C84, C88, C89: value 47uF -> 1uF; footprint Capacitor_SMD:C_0402_1005Metric -> Capacitor_SMD:C_0805_2012Metric
- C85: value 47uF -> 0.1uF; footprint Capacitor_SMD:C_0402_1005Metric -> Capacitor_SMD:C_0805_2012Metric
- C86, C87: value 47uF -> 10nF; footprint Capacitor_SMD:C_0402_1005Metric -> Capacitor_SMD:C_0805_2012Metric
- C90, C93: value 0.1uF -> 47uF; footprint Capacitor_SMD:C_0402_1005Metric -> Capacitor_SMD:C_1206_3216Metric
- C92, C95: value 0.1uF -> 1uF
- C96, C97: value 0.1uF -> 47uF 6.3V; footprint Capacitor_SMD:C_0402_1005Metric -> Capacitor_SMD:C_1206_3216Metric
- C99: value 0.1uF -> 0.1uF 25v
- D2: value SMCJ36CA -> TP7.OSMD24CA-XC
- L3: value 10uH 3A -> 10uH 12A
- Q1: footprint Devboard_Footprints:TO-263-7_L10.2-W9.2-P1.27-LS15.0-TL -> Package_TO_SOT_SMD:TO-263-7_TabPin8
- R10: value 2.2k -> 29.8k
- R16: value 10k -> 100Ω
- R17: value 357K -> 442k
- R2: value 10kΩ -> 22Ω
- R20: value 10k -> 124k
- R21: value 10k -> 20.5k
- R22: value 357K -> 210k
- R23: value 10k -> 10kΩ
- R24: value 100Ω -> 180Ω
- R3: value 10k -> 240Ω
- R4, R5: value 5.1k -> 240Ω
- R42: value 300kΩ -> 249kΩ
- R49: value 24.9k -> 24.3kΩ
- R67, R70: value 300k -> 249k
- R7: value 549Ω -> 750Ω
- R76: value 33Ω -> 4.7kΩ
- R77: value 4.7k -> 4.7kΩ
- R78, R79: value 10kΩ -> 100k
- R80: value 10kΩ -> 100kΩ
- R81: value 10kΩ -> 1k
- R82: value 10kΩ -> 100
- R84: value 4.7k -> 10kΩ
- R85, R86, R91, R93: value 4.7k -> 100kΩ
- R87: value 33Ω -> 100kΩ
- R88: value 33Ω -> 31.6K
- R9: value 1k -> 750Ω
- R94: value 4.7k -> 5.1kΩ
- U3: value xczu4evfbvb900pkg -> STUSB4500QTR; footprint Devboard_Footprints:XCZU4EVFBVB900PKG -> Package_DFN_QFN:QFN-24-1EP_4x4mm_P0.5mm_EP2.7x2.7mm
- Y1: value ASE-33.333MHz -> 25 MHz; footprint Oscillator:Oscillator_SMD_Abracon_ASE-4Pin_3.2x2.5mm -> Crystal:Crystal_SMD_3225-4Pin_3.2x2.5mm
- Y2: value 32.768 kHz -> 25 MHz; footprint Crystal:Crystal_SMD_3215-2Pin_3.2x1.5mm -> Crystal:Crystal_SMD_3225-4Pin_3.2x2.5mm
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Connections:
- net +20V_MAIN renamed +15V_MAIN
- net /Battery.Charger,Fuel Gauge/BQ_INT_N renamed BQ_INT_N
- net /Battery.Charger,Fuel Gauge/CHG_STAT_N renamed CHG_STAT_N
- net /Battery.Charger,Fuel Gauge/FUEL_GPOUT renamed FUEL_GPOUT
- net /Battery.Charger,Fuel Gauge/I2C_SCL renamed FuelGauge_SCL
- net /Battery.Charger,Fuel Gauge/I2C_SDA renamed FuelGauge_SDA
- net /Battery.Charger,Fuel Gauge/RAW_BAT renamed RAW_BAT
- net /Power Tree/PWR_OV_IN renamed PWR_OV_IN
- net /Power Tree/PWR_UV_IN renamed PWR_UV_IN
- net /Power,Input,Protection/MUX_STATUS renamed MUX_STATUS
- net /Power,Input,Protection/SBU2_SYS renamed SBU2_SYS
- net /Power,Input,Protection/TPD_FLT1 renamed Net-(U2-~{FLT})
- net PWR_FAULT_N renamed PWR_FAULT_N_eF
- net SH renamed /Power,Input,Protection/SH
- C1 pad 2: +3V3 -> VREG_2V7
- C100 pad 1: Net-(C100-Pad1) -> Net-(U25-SS/TRK)
- C101 pad 1: Net-(C101-Pad1) -> +5V_SYS
- C102 pad 1: Net-(C102-Pad1) -> Net-(U25-COMP)
- C102 pad 2: GND -> Net-(C102-Pad2)
- C103 pad 1: Net-(C103-Pad1) -> Net-(C102-Pad2)
- C104 pad 1: Net-(C104-Pad1) -> Net-(U25-FB)
- C105 pad 1: Net-(C105-Pad1) -> +0V9_GTR
- C106 pad 2: Net-(C105-Pad1) -> +0V9_GTR
- C107 pad 1: GND -> +1V2_GTH
- C107 pad 2: Net-(C107-Pad2) -> GND
- C108 pad 2: +0V85_PS -> +1V2_GTH
- C109 pad 1: Net-(C107-Pad2) -> +1V8_MGTRAVTT
- C110 pad 2: +0V9_VCU_GT -> +1V8_MGTRAVTT
- C111 pad 1: GND -> Net-(U24-DVDT)
- C111 pad 2: Net-(C111-Pad2) -> GND
- C112 pad 1: GND -> +1V25
- C112 pad 2: Net-(C112-Pad2) -> GND
- C113 pad 1: GND -> +1V2_PS
- C113 pad 2: Net-(C113-Pad2) -> GND
- C114 pad 2: Net-(C114-Pad2) -> +1V2_PS
- C115 pad 1: GND -> +1V8_VCCADC
- C115 pad 2: Net-(C115-Pad2) -> GND
- C116 pad 2: Net-(C116-Pad2) -> +1V8_VCCADC
- C117 pad 2: Net-(C117-Pad2) -> +0V85
- C131 pad 2: Net-(C131-Pad2) -> +0V85
- C132 pad 2: Net-(C132-Pad2) -> +0V85
- C133 pad 1: +0V9_VCU_GT -> GND
- C133 pad 2: GND -> +0V85
- C134 pad 1: Net-(C111-Pad2) -> GND
- C134 pad 2: GND -> +0V85
- C135 pad 1: Net-(C112-Pad2) -> GND
- C135 pad 2: GND -> +0V85
- C136 pad 1: Net-(C113-Pad2) -> +0V85
- C137 pad 1: Net-(C114-Pad2) -> Net-(C118-Pad2)
- C138 pad 1: Net-(C115-Pad2) -> Net-(C119-Pad2)
- C139 pad 1: Net-(C116-Pad2) -> Net-(C120-Pad2)
- C140 pad 1: Net-(C117-Pad2) -> Net-(C121-Pad2)
- C141 pad 1: Net-(C118-Pad2) -> Net-(C122-Pad2)
- C142 pad 1: Net-(C119-Pad2) -> Net-(C123-Pad2)
- C143 pad 1: Net-(C120-Pad2) -> Net-(C124-Pad2)
- C144 pad 1: Net-(C121-Pad2) -> Net-(C125-Pad2)
- C145 pad 1: Net-(C122-Pad2) -> Net-(C126-Pad2)
- C146 pad 1: Net-(C123-Pad2) -> Net-(C127-Pad2)
- C147 pad 1: Net-(C124-Pad2) -> Net-(C128-Pad2)
- C148 pad 1: Net-(C125-Pad2) -> Net-(C129-Pad2)
- C149 pad 1: Net-(C126-Pad2) -> Net-(C130-Pad2)
- C150 pad 1: Net-(C127-Pad2) -> +0V85
- C151 pad 1: Net-(C128-Pad2) -> +0V85
- C152 pad 1: Net-(C129-Pad2) -> +0V85
- C153 pad 1: Net-(C130-Pad2) -> +0V85
- C154 pad 1: Net-(C131-Pad2) -> +0V85
- C155 pad 1: Net-(C132-Pad2) -> GND
- C155 pad 2: GND -> +0V85_PS
- C156 pad 1: Net-(C156-Pad1) -> GND
- C156 pad 2: GND -> Net-(C156-Pad2)
- C157 pad 1: Net-(C157-Pad1) -> GND
- C157 pad 2: GND -> +0V85_PS
- C158 pad 1: Net-(C158-Pad1) -> GND
- C158 pad 2: GND -> +0V85_PS
- C159 pad 1: Net-(C159-Pad1) -> GND
- C159 pad 2: GND -> Net-(C159-Pad2)
- C160 pad 1: Net-(C160-Pad1) -> GND
- C160 pad 2: GND -> +0V85_PS
- C161 pad 1: Net-(C161-Pad1) -> GND
- C161 pad 2: GND -> +0V85_PS
- C162 pad 2: +0V9_VCU_GT -> +0V9_VCU
- C163 pad 2: Net-(C156-Pad1) -> +0V9_VCU
- C164 pad 2: Net-(C157-Pad1) -> +1V8
- C165 pad 2: Net-(C158-Pad1) -> +1V8
- C166 pad 2: Net-(C159-Pad1) -> +1V8
- C167 pad 2: Net-(C160-Pad1) -> +1V8
- C168 pad 2: Net-(C161-Pad1) -> +0V85_PS
- C169 pad 1: +1V8 -> GND
- C169 pad 2: GND -> +0V85_PS
- C170 pad 1: +1V8 -> +0V85_PS
- C171 pad 1: +1V8 -> GND
- C171 pad 2: GND -> +1V8
- C172 pad 1: +1V8 -> +0V85_PS
- C173 pad 1: +1V8 -> Net-(C156-Pad2)
- C174 pad 1: +1V8 -> +0V85_PS
- C175 pad 1: +1V8 -> +0V85_PS
- C176 pad 1: +1V8 -> Net-(C159-Pad2)
- C177 pad 1: +1V8 -> +0V85_PS
- C178 pad 1: +1V8 -> +0V85_PS
- C179 pad 1: +1V8 -> +0V9_VCU
- C180 pad 1: +1V8 -> +0V9_VCU
- C183 pad 1: +1V8_CLEAN -> +1V8
- C184 pad 1: +1V8_CLEAN -> +1V8
- C185 pad 1: +1V8_CLEAN -> GND
- C185 pad 2: GND -> +1V2
- C186 pad 1: +0V85_PS -> GND
- C186 pad 2: GND -> Net-(C186-Pad2)
- C187 pad 1: +0V85_PS -> GND
- C187 pad 2: GND -> +1V2
- C188 pad 1: +0V85_PS -> Net-(C188-Pad1)
- C188 pad 2: GND -> +0V85_GTR
- C189 pad 1: +0V85_GTR -> GND
- C189 pad 2: GND -> +1V8_CLEAN
- C190 pad 1: +0V85_GTR -> GND
- C190 pad 2: GND -> +1V2_PS
- C191 pad 1: +0V85_GTR -> GND
- C191 pad 2: GND -> +1V2
- C192 pad 1: +0V9_VCU_GT -> GND
- C192 pad 2: GND -> +1V8_CLEAN
- C193 pad 1: +0V9_VCU_GT -> GND
- C193 pad 2: GND -> +1V8_VCCADC
- C194 pad 1: +0V9_VCU_GT -> +1V2
- C195 pad 1: +1V8 -> Net-(C186-Pad2)
- C196 pad 1: +1V8 -> +1V2
- C197 pad 1: +1V8 -> +0V85_GTR
- C197 pad 2: GND -> Net-(C188-Pad1)
- C198 pad 1: +1V8 -> +1V8_CLEAN
- C199 pad 1: +1V8 -> +1V2_PS
- C200 pad 1: +1V2 -> GND
- C200 pad 2: GND -> +0V9_GTR
- C201 pad 1: +1V2 -> GND
- C201 pad 2: GND -> Net-(C201-Pad2)
- C202 pad 1: +1V2 -> GND
- C202 pad 2: GND -> +0V9_GTR
- C203 pad 1: +1V2 -> GND
- C203 pad 2: GND -> +1V2_GTH
- C204 pad 1: +1V2 -> GND
- C204 pad 2: GND -> Net-(C204-Pad2)
- C205 pad 1: /Zynq Core/PS_POR_B -> GND
- C205 pad 2: GND -> Net-(C205-Pad2)
- C206 pad 1: +1V8 -> GND
- C206 pad 2: GND -> Net-(C206-Pad2)
- C207 pad 1: Net-(U3-PS_PADO) -> GND
- C207 pad 2: GND -> +1V2_GTH
- C208 pad 1: Net-(U3-PS_PADI) -> GND
- C208 pad 2: GND -> +1V8
- C5 pad 2: +0V85_PS -> VREG_2V7
- C7 pad 2: /Power,Input,Protection/PWR_CURR_MON -> PWR_CURR_MON_eF
- C76 pad 1: GND -> Net-(U3-VREG_1V2)
- C76 pad 2: Net-(C76-Pad2) -> GND
- C77 pad 1: GND -> VREG_2V7
- C77 pad 2: Net-(C77-Pad2) -> GND
- C78 pad 2: Net-(C78-Pad2) -> VREG_2V7
- C79 pad 1: GND -> BATT_CHG
- C79 pad 2: Net-(C79-Pad2) -> GND
- C80 pad 1: GND -> CELL_B+
- C80 pad 2: Net-(C80-Pad2) -> CELL_B-
- C81 pad 2: Net-(C81-Pad2) -> Net-(U6-QON)
- C82 pad 2: Net-(C82-Pad2) -> VREG_2V7
- C83 pad 1: GND -> VBUS
- C83 pad 2: Net-(C83-Pad2) -> GND
- C84 pad 2: Net-(C84-Pad2) -> Net-(U19-VCC)
- C85 pad 1: GND -> Net-(C85-Pad1)
- C85 pad 2: Net-(C100-Pad1) -> Net-(U19-BOOT)
- C86 pad 2: Net-(C101-Pad1) -> Net-(U19-SS)
- C87 pad 2: Net-(C102-Pad1) -> Net-(C87-Pad2)
- C88 pad 2: Net-(C103-Pad1) -> +5V_BOOST
- C89 pad 2: Net-(C104-Pad1) -> +5V_SYS
- C90 pad 1: +0V85_PS -> +3V3_2
- C91 pad 1: Net-(C76-Pad2) -> +5V_SYS
- C92 pad 1: Net-(C77-Pad2) -> Net-(U22-NR)
- C93 pad 1: Net-(C78-Pad2) -> +2V5
- C94 pad 1: Net-(C79-Pad2) -> +5V_SYS
- C95 pad 1: Net-(C80-Pad2) -> Net-(U23-NR)
- C96 pad 1: Net-(C81-Pad2) -> +0V9_VCU
- C97 pad 1: Net-(C82-Pad2) -> +0V9_VCU
- C98 pad 1: Net-(C83-Pad2) -> +5V_SYS
- C99 pad 1: Net-(C84-Pad2) -> Net-(C99-Pad1)
- C99 pad 2: GND -> Net-(U25-BOOT)
- L1 pad 2: /Battery.Charger,Fuel Gauge/BATT_CHG -> +VSYS
- Q1 pad 8: /Power,Input,Protection/MUX_IN2 -> MUX_IN2_INT
- R12 pad 1: /Power,Input,Protection/PWR_GOOD -> PG_01
- R16 pad 1: MUX_PR1 -> Net-(D1-A)
- R16 pad 2: GND -> Net-(Q2-G)
- R19 pad 1: CP2_MUX -> Net-(U5-OVLO/OVCSEL)
- R2 pad 1: Net-(Y1-EN) -> Net-(U28-C)
- R2 pad 2: +1V8 -> QSPI_SCLK
- R20 pad 1: MUX_PR1 -> Net-(U5-OVLO/OVCSEL)
- R20 pad 2: VBUS -> MUX_OUT
- R23 pad 1: CP2_MUX -> Net-(U4-PR1)
- R23 pad 2: VBUS -> GND
- R3 pad 1: GND -> Net-(U_RAM2-ZQ)
- R3 pad 2: Net-(D1-A) -> GND
- R4 pad 1: CC1 -> Net-(U_RAM3-ZQ)
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Routing:
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
Commit message: Feat : Completed 04d Peripherals
Parts:
- removed U33: USBLC6-2SC6, Package_TO_SOT_SMD:SOT-23-6
- added C361: 0.1uF, Capacitor_SMD:C_0402_1005Metric, F.Cu at (97.2, 32.5)
- added C362: 0.1uF, Capacitor_SMD:C_0402_1005Metric, F.Cu at (97.2, 34.4)
- added C363: 0.1uF, Capacitor_SMD:C_0402_1005Metric, F.Cu at (97.2, 36.4)
- added C364: 1nF, Capacitor_SMD:C_0402_1005Metric, F.Cu at (97.2, 38.4)
- added C365: 1nF, Capacitor_SMD:C_0402_1005Metric, F.Cu at (97.2, 40.3)
- added C366: 1nF, Capacitor_SMD:C_0402_1005Metric, F.Cu at (97.2, 42.3)
- added C367: 0.1uF, Capacitor_SMD:C_0402_1005Metric, F.Cu at (97.2, 44.3)
- added C368: 1nF, Capacitor_SMD:C_0402_1005Metric, F.Cu at (97.2, 46.3)
- added C369: 0.1uF, Capacitor_SMD:C_0402_1005Metric, F.Cu at (100.1, 32.5)
- added C370: 1nF, Capacitor_SMD:C_0402_1005Metric, F.Cu at (100.1, 34.4)
- added C371: 0.1uF, Capacitor_SMD:C_0402_1005Metric, F.Cu at (100.1, 36.4)
- added C372: 1nF, Capacitor_SMD:C_0402_1005Metric, F.Cu at (100.1, 38.4)
- added C373: 0.1uF, Capacitor_SMD:C_0402_1005Metric, F.Cu at (100.1, 40.3)
- added C374: 1nF, Capacitor_SMD:C_0402_1005Metric, F.Cu at (100.1, 42.3)
- added C375: 22uF, Capacitor_SMD:C_0402_1005Metric, F.Cu at (100.1, 44.3)
- added C376: 22uF, Capacitor_SMD:C_0402_1005Metric, F.Cu at (100.1, 46.3)
- added C377: 0.1uF, Capacitor_SMD:C_0402_1005Metric, F.Cu at (102.9, 32.5)
- added C378: 0.1uF, Capacitor_SMD:C_0402_1005Metric, F.Cu at (102.9, 34.4)
- added C379: 22uF, Capacitor_SMD:C_0402_1005Metric, F.Cu at (102.9, 36.4)
- added C380: 22uF, Capacitor_SMD:C_0402_1005Metric, F.Cu at (102.9, 38.4)
- added C381: 0.1uF, Capacitor_SMD:C_0402_1005Metric, F.Cu at (102.9, 40.3)
- added C382: 0.1uF, Capacitor_SMD:C_0402_1005Metric, F.Cu at (102.9, 42.3)
- added C383: 0.1uF, Capacitor_SMD:C_0402_1005Metric, F.Cu at (102.9, 44.3)
- added C384: 0.1uF, Capacitor_SMD:C_0402_1005Metric, F.Cu at (102.9, 46.3)
- added Card1: TF-01A, Devboard_Footprints:TF-SMD_TF-01A, F.Cu at (96.0, 21.3)
- added J1: HR911105A_C12074, Devboard_Footprints:RJ45-TH_HR911105A, F.Cu at (77.7, 24.2)
- added R123: 22Ω, Resistor_SMD:R_0402_1005Metric, F.Cu at (112.1, 19.8)
- added R124: 22Ω, Resistor_SMD:R_0402_1005Metric, F.Cu at (112.1, 21.8)
- added R125: 22Ω, Resistor_SMD:R_0402_1005Metric, F.Cu at (112.1, 23.8)
- added R126: 22Ω, Resistor_SMD:R_0402_1005Metric, F.Cu at (112.1, 25.8)
- added R127: 22Ω, Resistor_SMD:R_0402_1005Metric, F.Cu at (115.0, 15.8)
- added R128: 22Ω, Resistor_SMD:R_0402_1005Metric, F.Cu at (115.0, 17.8)
- added R129: 22Ω, Resistor_SMD:R_0402_1005Metric, F.Cu at (115.0, 19.8)
- added R130: 22Ω, Resistor_SMD:R_0402_1005Metric, F.Cu at (115.0, 21.8)
- added R131: 10kΩ, Resistor_SMD:R_0402_1005Metric, F.Cu at (115.0, 23.8)
- added R132: 10kΩ, Resistor_SMD:R_0402_1005Metric, F.Cu at (115.0, 25.8)
- added R133: 2.49kΩ, Resistor_SMD:R_0402_1005Metric, F.Cu at (118.0, 15.8)
- added R134: 10kΩ, Resistor_SMD:R_0402_1005Metric, F.Cu at (118.0, 17.8)
- added R135: 2.49kΩ, Resistor_SMD:R_0402_1005Metric, F.Cu at (118.0, 19.8)
- added R136: 11kΩ, Resistor_SMD:R_0402_1005Metric, F.Cu at (118.0, 21.8)
- added R137: 470Ω, Resistor_SMD:R_0402_1005Metric, F.Cu at (118.0, 23.8)
- added R138: 470Ω, Resistor_SMD:R_0402_1005Metric, F.Cu at (118.0, 25.8)
- added U28: MT25QU256ABA8ESF-0SIT TR, Devboard_Footprints:SOP-16_L10.3-W7.5-P1.27-LS10.4-BL, F.Cu at (97.5, 6.15)
- added U29: FEMDNN032G-A3A55, Devboard_Footprints:FBGA-153_L13.0-W11.5-P0.50_KLMAG1JETD-B041, F.Cu at (111.2, 39.0)
- added U30: TXS02612RTWR, Devboard_Footprints:WQFN-24_L4.0-W4.0-P0.50-TL-EP2.5, F.Cu at (106.5, 11.8)
- added U31: DP83867IRRGZR, Devboard_Footprints:VQFN-48_L7.0-W7.0-P0.50-TL-EP4.1, F.Cu at (73.0, 42.1)
- added U38: TPD4E05U06DQA, Package_SON:USON-10_2.5x1.0mm_P0.5mm, F.Cu at (111.9, 29.0)
- moved U34 130.2 mm to (115.8, 11.7)
- moved U36 122.0 mm to (107.9, 4.17)
- moved U37 119.9 mm to (107.7, 28.7)
- moved R121 115.9 mm to (112.1, 15.8)
- moved R122 115.9 mm to (112.1, 17.8)
- moved R115 114.2 mm to (109.2, 15.8)
- moved R116 114.2 mm to (109.2, 17.8)
- moved R118 114.2 mm to (109.2, 21.8)
- moved R117 114.2 mm to (109.2, 19.8)
- moved R110 112.4 mm to (106.3, 17.8)
- moved R111 112.4 mm to (106.3, 19.8)
- moved R112 112.4 mm to (106.3, 21.8)
- moved R113 112.4 mm to (106.3, 23.8)
- moved R2 112.4 mm to (106.3, 15.8)
- moved Y1 110.5 mm to (114.9, 1.77)
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Connections:
- U26 pad C23: unconnected-(U26-PS_MIO38-PadC23) -> GEM_RST
- U34 pad 2: Net-(U34-GND-Pad2) -> GND
- U34 pad 25: Net-(U34-GND-Pad2) -> GND
- U34 pad 8: unconnected-(U34-VBUS-Pad8) -> VBUS
- U35 pad 11: unconnected-(U35-GND-Pad11) -> GND
- U37 pad 1: unconnected-(U37-GND-Pad1) -> GND
- Y1 pad 1: unconnected-(Y1-Pad1) -> Net-(U31-X_I)
- Y1 pad 2: Net-(Y1-G-Pad2) -> GND
- Y1 pad 3: unconnected-(Y1-Pad3) -> Net-(U31-X_O)
- Y1 pad 4: Net-(Y1-G-Pad2) -> GND
- Y2 pad 1: unconnected-(Y2-Pad1) -> Net-(C380-Pad2)
- Y2 pad 2: Net-(Y2-G-Pad2) -> GND
- Y2 pad 3: unconnected-(Y2-Pad3) -> Net-(C379-Pad2)
- Y2 pad 4: Net-(Y2-G-Pad2) -> GND
Other:
- board outline added: 133.4 x 151 mm
