File: PCB/Devboard.kicad_pcb (KiCad board)
At the start: 2 copper layers, 174.2 x 169.9 mm, 875 parts, among them CN1 1-2199230-6, J1 HR911105A_C12074, J10 Conn_02x07_Odd_Even, J11 Conn_01x04_Pin, J12 SFP+, J13 Conn_01x22, J14 Conn_01x10, J15 Conn_01x10, J16 Conn_01x10, J2 Conn_01x03_Pin, J3 USB3_B, J4 Conn_01x02_Pin, J5 Conn_01x02_Pin, J6 3.3V_I2C, J7 Conn_01x10, J8 Conn_01x09_Pin, J9 Conn_Coaxial, Q1 IPB180P04P4L-02, Q2 IPB180P04P4L-02, SW1 SW_Push, SW2 SW_SPDT, U1 TPD6S300ARUKR, U10 BQ27441DRZR-G1A, U11 LM66100DCK, U12 TPS61088RHLR, U13 TPS548A20RVER, U14 TPS62130RGTR, U15 TPS54824RNVR, U16 TPS62823DLCR, U17 TPS62822DLCR, U18 TPS7A4700RGWR, U19 TPS3700DSET, U2 STUSB4500QTR, U20 TPS54824RNVR, U21 TPS54824RNVR, U22 TPS7A4700RGWR, U23 TPS7A4700RGWR, U24 RS3112-1.25XSF3, U25 TPS54824RNVR, U26 TPS7A4700RGWR, U27 xczu4evfbvb900pkg, U28 TXS02612RTWR, U29 MT25QU256ABA8ESF-0SIT TR, U3 TVS2201DRBR, U30 FEMDNN032G-A3A55, U31 DP83867IRRGZR, U32 CP2102N-A02-GQFN24, U33 USB3320C-EZK-TR, U34 TPD4E05U06DQA, U35 TCA9548APWR, U36 TXB0108PW, U37 PCA9306, U38 USB2514B_Bi, U39 TPD4E05U06DQA, U4 TPS259470ARPWR, U40 TXS0102DQE, U41 SI5341A-D12636-GM, U42 REF5025AD, U43 LMX2594RHAR, U44 ADS131M08IPBS, U45 ADS4245IRGCT, U46 AD9744ARUZRL7, U47 THS4509RGTT, U48 ADL8100ACPZN, U49 BPF-A355, U5 TPS2121RUXR, U50 TMP117DRVR, U51 ICM-42688-P, U52 MMC5983MA, U53 TCA9548APWR, U54 BMP581, U55 MAX-M10S-00B, U56 ATECC608B-MAHDA, U57 OPTIGA TPM SLB 9673 FW26, U58 BQ25570, U59 STM32G0B1RBT6, U6 TPS259470ARPWR, U7 XT60, U8 DW06, U9 BQ25895RTWR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

Commit message: Refactor : Repo
Parts:
- U33: footprint Devboard_Footprints:RJ45-TH_HR911105A -> Devboard_Footprints:QFN-32_L5.0-W5.0-P0.50-BL-EP3.4
- moved J1 7.17 mm to (2.24, 71.4)

Commit message: Feat : Finished four sections of Placement
Parts:
- added ?: , , F.Cu at (528.5, 337.1)
- added REF**: MountingHole_6.4mm_M6_ISO7380, MountingHole:MountingHole_6.4mm_M6_ISO7380, F.Cu at (527.0, 151.9)
- added REF**: MountingHole_2.7mm_M2.5, MountingHole:MountingHole_2.7mm_M2.5, F.Cu at (369.4, 236.3)
- added REF**: MountingHole_6.4mm_M6_ISO7380, MountingHole:MountingHole_6.4mm_M6_ISO7380, F.Cu at (243.5, 151.3)
- added REF**: MountingHole_2.7mm_M2.5, MountingHole:MountingHole_2.7mm_M2.5, F.Cu at (419.8, 287.8)
- added REF**: MountingHole_2.7mm_M2.5, MountingHole:MountingHole_2.7mm_M2.5, F.Cu at (419.8, 236.9)
- added REF**: MountingHole_6.4mm_M6_ISO7380, MountingHole:MountingHole_6.4mm_M6_ISO7380, F.Cu at (245.0, 336.5)
- added REF**: MountingHole_2.7mm_M2.5, MountingHole:MountingHole_2.7mm_M2.5, F.Cu at (369.4, 287.3)
- C1, C2, C3, C4: footprint Capacitor_SMD:C_1210_3225Metric -> Capacitor_SMD:C_0402_1005Metric
- moved C406 1072.7 mm to (-844.6, 739.5)
- moved C407 1072.7 mm to (-844.6, 741.5)
- moved J6 1072.7 mm to (-801.9, 708.1)
- moved R154 1072.7 mm to (-830.1, 737.6)
- moved R156 1072.7 mm to (-830.1, 741.6)
- moved R157 1072.7 mm to (-830.1, 743.6)
- moved R159 1072.7 mm to (-830.1, 747.6)
- moved R160 1072.7 mm to (-827.2, 729.6)
- moved U37 1072.7 mm to (-831.1, 762.6)
- moved R198 984.5 mm to (-715.1, 734.6)
- moved R199 984.5 mm to (-715.1, 736.6)
- moved R200 984.5 mm to (-715.1, 738.6)
- moved U53 984.5 mm to (-696.5, 709.5)
- moved C504 984.5 mm to (-732.6, 750.3)
- moved C397 971.6 mm to (-808.6, 623.7)
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Connections:
- net /Analog | RF/ADC_INM_A renamed /Analog_RF/ADC_INM_A
- net /Analog | RF/ADC_INM_B renamed /Analog_RF/ADC_INM_B
- net /Analog | RF/ADC_INP_A renamed /Analog_RF/ADC_INP_A
- net /Analog | RF/ADC_INP_B renamed /Analog_RF/ADC_INP_B
- net /Analog | RF/ADC_VCM renamed /Analog_RF/ADC_VCM
- net /Analog | RF/CLKM renamed /Analog_RF/CLKM
- net /Analog | RF/CLKP renamed /Analog_RF/CLKP
- net /Analog | RF/CPout renamed /Analog_RF/CPout
- net /Analog | RF/OSCinM renamed /Analog_RF/OSCinM
- net /Analog | RF/OSCinP renamed /Analog_RF/OSCinP
- net /Analog | RF/RF_IN renamed /Analog_RF/RF_IN
- net /Analog | RF/RF_LNA_OUT renamed /Analog_RF/RF_LNA_OUT
- net /Analog | RF/RF_RX renamed /Analog_RF/RF_RX
- net /Analog | RF/RF_RX_FILT renamed /Analog_RF/RF_RX_FILT
- net /Analog | RF/RF_TX renamed /Analog_RF/RF_TX
- net /Analog | RF/SMA_RF_OUT renamed /Analog_RF/SMA_RF_OUT
- net /Analog | RF/TCX0_OUT renamed /Analog_RF/TCX0_OUT
- net /Analog | RF/THS_IN_N renamed /Analog_RF/THS_IN_N
- net /Analog | RF/THS_IN_P renamed /Analog_RF/THS_IN_P
- net /Analog | RF/THS_OUT+ renamed /Analog_RF/THS_OUT+
- net /Analog | RF/THS_OUT- renamed /Analog_RF/THS_OUT-
- net /Analog | RF/Vtune renamed /Analog_RF/Vtune
Other:
- board size 174.2 x 169.9 mm -> 300 x 200 mm
- board text added: "U27"
