File: PCB/schematics/01_Power/Power_Input_Protection.kicad_sch (KiCad schematic)
At the start: 65 parts, among them Q1 IPB180P04P4L-02, Q2 IPB180P04P4L-02, U1 TVS2201DRBR, U2 TPD6S300ARUKR, U3 STUSB4500QTR, U4 TPS2121RUXR, U5 TPS259470ARPWR

Commit message: Fix Section 1
Parts:
- R76, R77: value 100k -> 4.7kΩ
Connections:
- net +5V_SYS: no longer names the net of C4.2, U2.3 (VBIAS)
Other:
- moved on the sheet: C2
Changed lines of the file:
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@@
 	)
 	(junction
-		(at 353.06 116.84)
-		(diameter 0)
-		(color 0 0 0 0)
-	)
-	(junction
 		(at 381 72.39)
 		(diameter 0)
@@
 	(symbol
 		(lib_id "power:+3V3")
-		(at 300.99 99.06 90)
+		(at 298.45 99.06 90)
 		(unit 1)
 		(body_style 1)
@@
 		(fields_autoplaced yes)
 		(property "Reference" "#PWR0160"
-			(at 304.8 99.06 0)
+			(at 302.26 99.06 0)
 			(hide yes)
 			(show_name no)
@@
 		)
 		(property "Value" "+3V3"
-			(at 297.18 99.0599 90)
+			(at 294.64 99.0599 90)
 			(show_name no)
 			(do_not_autoplace no)
@@
 		)
 		(property "Footprint" ""
-			(at 300.99 99.06 0)
+			(at 298.45 99.06 0)
 			(hide yes)
 			(show_name no)
@@
 		)
 		(property "Datasheet" ""
-			(at 300.99 99.06 0)
+			(at 298.45 99.06 0)
 			(hide yes)
 			(show_name no)
@@
 		)
 		(property "Description" "Power symbol creates a global label with name \"+3V3\""
-			(at 300.99 99.06 0)
+			(at 298.45 99.06 0)
 			(hide yes)
 			(show_name no)
@@
 	(symbol
 		(lib_id "power:GND")
-		(at 300.99 91.44 270)
+		(at 298.45 91.44 270)
 		(unit 1)
 		(body_style 1)
@@
 		(fields_autoplaced yes)
 		(property "Reference" "#PWR077"
-			(at 294.64 91.44 0)
+			(at 292.1 91.44 0)
 			(hide yes)
 			(show_name no)
@@
 		)
 		(property "Value" "GND"
-			(at 295.91 91.44 0)
+			(at 293.37 91.44 0)
 			(show_name no)
 			(do_not_autoplace no)
@@
 		)
 		(property "Footprint" ""
-			(at 300.99 91.44 0)
+			(at 298.45 91.44 0)
 			(hide yes)
 			(show_name no)
@@
 		)
 		(property "Datasheet" ""
-			(at 300.99 91.44 0)
+			(at 298.45 91.44 0)
 			(hide yes)
 			(show_name no)
@@
 		)
 		(property "Description" "Power symbol creates a global label with name \"GND\" , ground"
-			(at 300.99 91.44 0)
+			(at 298.45 91.44 0)
 			(hide yes)
 			(show_name no)
@@
 			)
 		)
-		(property "Value" "100k"
+		(property "Value" "4.7kΩ"
 			(at 167.894 101.6 90)
 			(show_name no)
@@
 			(effects
 				(font
-					(size 1.27 1.27)
+					(size 1 1)
 				)
 				(justify left)
@@
 	(symbol
 		(lib_id "Device:C")
-		(at 300.99 95.25 0)
+		(at 298.45 95.25 0)
 		(unit 1)
 		(body_style 1)
@@
 		(fields_autoplaced yes)
 		(property "Reference" "C2"
-			(at 304.8 93.9799 0)
+			(at 302.26 93.9799 0)
 			(show_name no)
 			(do_not_autoplace no)
@@
 		)
 		(property "Value" "1uF 25V"
-			(at 304.8 96.5199 0)
+			(at 302.26 96.5199 0)
 			(show_name no)
 			(do_not_autoplace no)
@@
 		)
 		(property "Footprint" "Capacitor_SMD:C_0402_1005Metric"
-			(at 301.9552 99.06 0)
+			(at 299.4152 99.06 0)
 			(hide yes)
 			(show_name no)
@@
 		)
 		(property "Datasheet" ""
-			(at 300.99 95.25 0)
+			(at 298.45 95.25 0)
 			(hide yes)
 			(show_name no)
@@
 		)
 		(property "Description" "Unpolarized capacitor"
-			(at 300.99 95.25 0)
+			(at 298.45 95.25 0)
 			(hide yes)
 			(show_name no)
@@
 			)
 		)
-		(property "Value" "100k"
+		(property "Value" "4.7kΩ"
 			(at 167.894 104.14 90)
 			(show_name no)
@@
 			(effects
 				(font
-					(size 1.27 1.27)
+					(size 1 1)
 				)
 				(justify left)
@@
 	)
 	(symbol
-		(lib_id "power:+3V3")
-		(at 353.06 116.84 270)
-		(unit 1)
-		(body_style 1)
-		(exclude_from_sim no)
-		(in_bom yes)
-		(on_board yes)
-		(in_pos_files yes)
-		(dnp no)
-		(property "Reference" "#PWR0284"
-			(at 349.25 116.84 0)
-			(hide yes)
-			(show_name no)
-			(do_not_autoplace no)
-			(effects
-				(font
-					(size 1.27 1.27)
-				)
-			)
-		)
-		(property "Value" "+5V_SYS"
-			(at 356.87 111.76 0)
-			(show_name no)
-			(do_not_autoplace no)
-			(effects
-				(font
-					(size 1.27 1.27)
-				)
-				(justify left)
-			)
-		)
-		(property "Footprint" ""
-			(at 353.06 116.84 0)
-			(hide yes)
-			(show_name no)
-			(do_not_autoplace no)
-			(effects
-				(font
-					(size 1.27 1.27)
-				)
-			)
-		)
-		(property "Datasheet" ""
-			(at 353.06 116.84 0)
-			(hide yes)
-			(show_name no)
-			(do_not_autoplace no)
-			(effects
-				(font
-					(size 1.27 1.27)
-				)
-			)
-		)
-		(property "Description" "Power symbol creates a global label with name \"+3V3\""
-			(at 353.06 116.84 0)
-			(hide yes)
-			(show_name no)
-			(do_not_autoplace no)
-			(effects
-				(font
-					(size 1.27 1.27)
-				)
-			)
-		)
-		(pin "1"
-		)
-		(instances
-			(project "Devboard"
-				(path "/f4f7837f-dd80-4f77-b150-4534de1c10d6/880a94ed-a974-4da2-b4ca-cb72436ddb06"
-					(reference "#PWR0284")
-					(unit 1)
-				)
-			)
-		)
-	)
-	(symbol
 		(lib_id "power:GND")
 		(at 217.17 243.84 90)
@@
 		(dnp no)
 		(property "Reference" "C4"
-			(at 347.472 120.904 90)
+			(at 362.966 128.778 0)
 			(show_name no)
 			(do_not_autoplace no)
@@
 		)
 		(property "Value" "0.1uF 50V X7R"
-			(at 349.504 120.396 90)
+			(at 362.458 126.746 0)
 			(show_name no)
 			(do_not_autoplace no)

Commit message: Journal Update
Parts:
- added C111: 10nF 25V, Capacitor_SMD:C_0402_1005Metric, symbol Device:C
- added R102: 10kΩ, Resistor_SMD:R_0402_1005Metric, symbol Device:R
- added R103: 100kΩ, Resistor_SMD:R_0402_1005Metric, symbol Device:R
- added R104: 124k, Resistor_SMD:R_0402_1005Metric, symbol Device:R
- added R105: 10k, Resistor_SMD:R_0402_1005Metric, symbol Device:R
- added R106: 549Ω, Resistor_SMD:R_0402_1005Metric, symbol Device:R
- added R9: 750Ω, Resistor_SMD:R_0402_1005Metric, symbol Device:R
- added U24: TPS259470ARPWR, easyeda2kicad:VQFN-10_L2.0-W2.0-P0.45-TL, symbol Devboard_Symbols:TPS259470ARPWR
Connections:
- net GND: now also C111.2, R102.2, R105.2, R106.2, R9.2, U24.8 (GND)
- net VBUS: now also R103.2, R104.2, U24.5 (IN); no longer U1.1 (IN), U1.2 (IN), U1.3 (IN), U1.4 (IN)
- net U5_ILM: no longer names the net of R7.1, U5.9 (ILM)
- new net: R102.1, R103.1, U24.1 (EN/UVLO)
- new net: R9.1, U24.9 (ILM)
- new net: R104.1, R105.1, U24.2 (OVLO/OVCSEL)
- new net: R106.1, U24.10 (ITIMER)
- new net: C111.1, U24.7 (DVDT)
- new net OUT_VBUS: U1.1 (IN), U1.2 (IN), U1.3 (IN), U1.4 (IN), U24.6 (OUT)
- no-connect marks 17 -> 19
Other:
- moved on the sheet: C6, D7, R7, R94, R95, U1

Commit message: Feat: Added zynq decoupling caps
Parts:
- U24: footprint easyeda2kicad:VQFN-10_L2.0-W2.0-P0.45-TL -> Devboard_Footprints:VQFN-10_L2.0-W2.0-P0.45-TL
Changed lines of the file:
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@@
 			)
 		)
-		(property "Footprint" "easyeda2kicad:VQFN-10_L2.0-W2.0-P0.45-TL"
+		(property "Footprint" "Devboard_Footprints:VQFN-10_L2.0-W2.0-P0.45-TL"
 			(at 54.61 132.08 0)
 			(hide yes)

Commit message: Feat : Schematics Complete
Parts:
- renumbered C76 to C1, C2 to C10, C4 to C11, C111 to C12, C7 to C13, C8 to C14, C9 to C15, C10 to C16, C11 to C17, C12 to C18, C13 to C19, C6 to C2, C14 to C20, C15 to C21, C77 to C3, C78 to C4, C1 to C5, C5 to C6, C82 to C7, C83 to C8, C3 to C9, D7 to D1, D1 to D2, D2 to D3, D6 to D4, D3 to D5, D4 to D6, D8 to D7, D9 to D8, R94 to R1, R102 to R10, R78 to R11, R79 to R12, R103 to R13, R106 to R14, R9 to R15, R6 to R16, R8 to R17, R10 to R18, R11 to R19, R93 to R2, R19 to R20, R12 to R21, R13 to R22, R14 to R23, R15 to R24, R20 to R25, R7 to R26, R23 to R27, R92 to R28, R18 to R29, R95 to R3, R17 to R30, R22 to R31, R21 to R32, R1 to R4, R16 to R5, R76 to R6, R105 to R7, R77 to R8, R104 to R9, U2 to U1, U3 to U2, U1 to U3, U24 to U4, U4 to U5, U5 to U6

Commit message: Refactor : Repo
Changed lines of the file:
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@@
 		(stroke
 			(width 0)
-			(type default)
+			(type solid)
 		)
 		(fill
-			(type none)
+			(type color)
+			(color 255 229 191 1)
 		)
 	)
@@
 	(text "SECTION 1 : POWER, INPUT, PROTECTION"
 		(exclude_from_sim no)
-		(at 279.908 32.258 0)
+		(at 299.212 32.512 0)
 		(effects
 			(font

Commit message: Feat : Finished four sections of Placement
Parts:
- C1, C2, C3, C4: footprint Capacitor_SMD:C_1210_3225Metric -> Capacitor_SMD:C_0402_1005Metric
