File: PCB/schematics/02_Battery/Battery_Charger_FuelGauge.kicad_sch (KiCad schematic)
At the start: 53 parts, among them SW1 SW_Push, U18 DW06, U19 TPS61088RHLR, U21 LM66100DCK, U6 BQ25895RTWR, U7 BQ27441DRZR-G1A, U9 XT60

Commit message: Journal Update
Connections:
- net +5V_SYS: no longer U6.1 (VBUS)
- new net OUT_VBUS: U6.1 (VBUS)
Changed lines of the file:
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@@
 		)
 	)
+	(global_label "OUT_VBUS"
+		(shape input)
+		(at 166.37 104.14 180)
+		(fields_autoplaced yes)
+		(effects
+			(font
+				(size 1.27 1.27)
+			)
+			(justify right)
+		)
+		(property "Intersheetrefs" "${INTERSHEET_REFS}"
+			(at 153.89 104.14 0)
+			(hide yes)
+			(show_name no)
+			(do_not_autoplace no)
+			(effects
+				(font
+					(size 1.27 1.27)
+				)
+				(justify right)
+			)
+		)
+	)
 	(global_label "BATT_CHG"
 		(shape input)
@@
 					(unit 1)
 				)
-			)
-		)
-	)
-	(symbol
-		(lib_id "power:+1V0")
-		(at 166.37 104.14 90)
-		(unit 1)
-		(body_style 1)
-		(exclude_from_sim no)
-		(in_bom yes)
-		(on_board yes)
-		(in_pos_files yes)
-		(dnp no)
-		(fields_autoplaced yes)
-		(property "Reference" "#PWR075"
-			(at 170.18 104.14 0)
-			(hide yes)
-			(show_name no)
-			(do_not_autoplace no)
-			(effects
-				(font
-					(size 1.27 1.27)
-				)
-			)
-		)
-		(property "Value" "+5V_SYS"
-			(at 162.56 104.1399 90)
-			(show_name no)
-			(do_not_autoplace no)
-			(effects
-				(font
-					(size 1.27 1.27)
-				)
-				(justify left)
-			)
-		)
-		(property "Footprint" ""
-			(at 166.37 104.14 0)
-			(hide yes)
-			(show_name no)
-			(do_not_autoplace no)
-			(effects
-				(font
-					(size 1.27 1.27)
-				)
-			)
-		)
-		(property "Datasheet" ""
-			(at 166.37 104.14 0)
-			(hide yes)
-			(show_name no)
-			(do_not_autoplace no)
-			(effects
-				(font
-					(size 1.27 1.27)
-				)
-			)
-		)
-		(property "Description" "Power symbol creates a global label with name \"+1V0\""
-			(at 166.37 104.14 0)
-			(hide yes)
-			(show_name no)
-			(do_not_autoplace no)
-			(effects
-				(font
-					(size 1.27 1.27)
-				)
-			)
-		)
-		(pin "1"
-		)
-		(instances
-			(project "Devboard"
-				(path "/f4f7837f-dd80-4f77-b150-4534de1c10d6/58c0d1bc-f1af-47a1-8444-9b0b37a445d5"
-					(reference "#PWR075")
-					(unit 1)
-				)

Commit message: Feat : Schematics Complete
Parts:
- R33: renamed from R31; footprint Resistor_SMD:R_2512_6332Metric -> Resistor_SMD:R_Shunt_Isabellenhuette_BVR4026
- renumbered C16 to C22, C25 to C23, C26 to C24, C18 to C25, C80 to C26, C17 to C27, C79 to C28, C20 to C29, C21 to C30, C81 to C31, C84 to C32, C88 to C33, C23 to C34, C87 to C35, C22 to C36, C89 to C37, C85 to C38, C86 to C39, D5 to D9, L8 to L2, R35 to R34, R30 to R35, R27 to R36, R32 to R37, R81 to R38, R82 to R39, R24 to R40, R85 to R41, R33 to R42, R28 to R43, R29 to R44, R25 to R45, R34 to R46, R26 to R47, R98 to R48, R80 to R49, R90 to R50, R83 to R51, R86 to R52, R89 to R53, R87 to R54, R88 to R55, R91 to R56, U7 to U10, U21 to U11, U19 to U12, U9 to U7, U18 to U8, U6 to U9
