File: PCB/schematics/03_Power_Tree/03_Power_Tree.kicad_sch (KiCad schematic)
At the start: 145 parts, among them U10 TPS62822DLCR, U11 TPS62823DLCR, U12 TPS548A20RVER, U13 TPS7A4700RGWR, U14 TPS3700DSET, U15 TPS54824RNVR, U16 TPS54824RNVR, U17 TPS7A4700RGWR, U20 TPS54824RNVR, U22 TPS7A4700RGWR, U23 TPS7A4700RGWR, U25 TPS54824RNVR, U8 TPS62130RGTR

Commit message: Feat: Added zynq decoupling caps
Parts:
- added C112: 47uF, Capacitor_SMD:C_1206_3216Metric, symbol Device:C
- added C113, C115: 0.1uF 25V, Capacitor_SMD:C_0402_1005Metric, symbol Device:C
- added C114, C116: 10uF, Capacitor_SMD:C_0402_1005Metric, symbol Device:C
- added FB5, FB6: 120Ω@100MHz, Inductor_SMD:L_01005_0402Metric, symbol Device:FerriteBead
- added U27: RS3112-1.25XSF3, Devboard_Footprints:SOT-23-3_L2.9-W1.3-P0.95-LS2.4-BR, symbol Devboard_Symbols:RS3112-1.25XSF3
Connections:
- net +1V2: now also FB5.2
- net +1V8: now also FB6.2
- net +3V3_ANA: now also U27.1 (VIN)
- net GND: now also C112.2, C113.2, C114.1, C115.2, C116.1, U27.3 (GND)
- new net +1V25: C112.1, U27.2 (OUT)
- new net +1V2_PS: C113.1, C114.2, FB5.1
- new net +1V8_VCCADC: C115.1, C116.2, FB6.1
Other:
- moved on the sheet: C105, C106, C109, C110, C93, C94, C95, FB2, FB4, U23

Commit message: Feat : Schematics Complete
Parts:
- removed C90: 47uF, Capacitor_SMD:C_1206_3216Metric, symbol Device:C
- removed C91: 10uF, Capacitor_SMD:C_0402_1005Metric, symbol Device:C
- removed C92: 1uF, Capacitor_SMD:C_0402_1005Metric, symbol Device:C
- removed U22: TPS7A4700RGWR, Devboard_Footprints:VQFN-20_L5.0-W5.0-P0.65-TL-EP, symbol Custom_Symbols:TPS7A4700RGWR
- added C105, C70: 0.1uF 25V, Capacitor_SMD:C_0402_1005Metric, symbol Device:C
- added C106, C108, C71: 10uF, Capacitor_SMD:C_0402_1005Metric, symbol Device:C
- added C107: 47uF, Capacitor_SMD:C_1206_3216Metric, symbol Device:C
- added C117: 1uF, Capacitor_SMD:C_0402_1005Metric, symbol Device:C
- added FB3, FB7: 120Ω@100MHz, Inductor_SMD:L_01005_0402Metric, symbol Device:FerriteBead
- added U26: TPS7A4700RGWR, Devboard_Footprints:VQFN-20_L5.0-W5.0-P0.65-TL-EP, symbol Custom_Symbols:TPS7A4700RGWR
- renumbered C71 to C100, C95 to C101, C72 to C102, C73 to C103, C99 to C104, C100 to C109, C98 to C110, C102 to C111, C103 to C112, C112 to C113, C104 to C114, C96 to C115, C97 to C116, C101 to C118, C105 to C119, C106 to C120, C36 to C40, C43 to C41, C34 to C42, C46 to C43, C32 to C44, C48 to C45, C33 to C46, C35 to C47, C44 to C48, C31 to C49, C30 to C50, C47 to C51, C29 to C52, C39 to C53, C40 to C54, C41 to C55, C42 to C56, C38 to C57, C37 to C58, C28 to C59, C27 to C60, C51 to C61, C49 to C62, C19 to C63, C24 to C64, C52 to C65, C107 to C66, C108 to C67, C113 to C68, C114 to C69, C109 to C72, C110 to C73, C115 to C74, C116 to C75, C64 to C76, C50 to C77, C55 to C78, C65 to C79, C63 to C80, C67 to C81, C68 to C82, C60 to C83, C53 to C84, C45 to C85, C59 to C86, C69 to C87, C58 to C88, C61 to C89, C62 to C90, C66 to C91, C56 to C92, C57 to C93, C75 to C94, C74 to C95, C54 to C96, C93 to C97, C94 to C98, C70 to C99, FB3 to FB1, FB5 to FB2, FB6 to FB5, FB1 to FB6, FB2 to FB8, L2 to L3, L3 to L5, L5 to L7, L9 to L8, L7 to L9, R96 to R102, R38 to R57, R50 to R58, R39 to R59, R51 to R60, R48 to R61, R43 to R62, R47 to R63, R49 to R64, R36 to R65, R40 to R66, R52 to R67, R37 to R68, R41 to R69, R45 to R70, R42 to R71, R44 to R72, R58 to R73, R56 to R74, R55 to R75, R57 to R76, R53 to R77, R54 to R78, R68 to R79, R69 to R80, R63 to R81, R62 to R82, R71 to R83, R66 to R84, R72 to R85, R73 to R86, R65 to R87, R59 to R88, R46 to R89, R74 to R90, R70 to R91, R64 to R92, R67 to R93, R60 to R94, R61 to R95, R75 to R96, R84 to R97, R97 to R98, U12 to U13, U8 to U14, U11 to U16, U10 to U17, U13 to U18, U14 to U19, U16 to U21, U23 to U22, U17 to U23, U27 to U24
Connections:
- net +3V3_ANA: now also FB3.2, U26.3 (SENSE/FB)
- net +5V_SYS: now also C108.1, U26.13 (EN), U26.15 (IN), U26.16 (IN)
- net GND: now also C105.2, C106.1, C107.2, C108.2, C117.2, C70.2, C71.1, U26.10 (0P4V), U26.21 (EP), U26.6 (3P2V), U26.7 (GND)
- new net: C107.1, FB7.2, U26.1 (OUT), U26.20 (OUT)
- new net: C117.1, U26.14 (NR)
- new net +3V3_LMX: C70.1, C71.2, FB3.1
- new net +5V_ANA: C105.1, C106.2, FB7.1
- no-connect marks 43 -> 44
Other:
- moved on the sheet: C104, C109, C110, C111, C112, C113, C114, C115, C116, C118, C119, C120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

Commit message: Refactor : Repo
Other:
- note added: "+0V85"
- note added: "+0V85_PS, +0V85_GTR"
- note added: "+0V9_VCU, +0V9_GTR"
- note added: "+0V9_VCU_GT"
- note added: "+1V2. +1V2_PS, +1V2_GTH"
- note added: "+1V25"
- note added: "+1V8"
- note added: "+1V8_CLEAN"
- note added: "+2V5"
- note added: "+3V3"
- note added: "+3V3_ANA, +3V3_LMX"
- note added: "+5V_ANA"
- note added: "+5V_SYS"
- moved on the sheet: C105, C106, C107, C108, C117, FB7, U26

Commit message: Feat : Finished four sections of Placement
Other:
- moved on the sheet: C59, C60, C61, C66, C67, C68, C69, FB1, FB2, L6, R73, R74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
