File: PCB/schematics/12_Expansion/12_Expansion.kicad_sch (KiCad schematic)
At the start: 4 parts, among them J14 Conn_01x10, J15 Conn_01x10, J16 Conn_01x10, J7 Conn_01x10

Commit message: Refactor : Repo
Other:
- moved on the sheet: J14, J15, J16, J7
